File: mechanical-mock.sch (KiCad schematic (older format))
At the start: 13 parts, among them J1 DF40HC(3.0)-100DS-0.4v, J2 DF40HC(3.0)-100DS-0.4v, U1 SiFive-U74, U2 MT53E256M32D2, U3 MT53E256M32D2, U4 S25FL128SAGNFI000, U5 TPS65086100, U6 TDA19988BHN_C1,557, U7 KSZ9031RNXCA

Commit message: Connected interfaces to VIC to visualise its ball locations (wip, mock purposes)
Parts:
- removed J1, J2: DF40HC(3.0)-100DS-0.4v, riscv-u74-som-footprints:DF40HC(3.0)-100DS-0.4v, symbol riscv-u74-som:DF40HC(3.0)-100DS-0.4v
- added J1, J2: DF40C-100DP-0.4V(51), antmicro-footprints:HRS_DF40C-100DP-0.4V(51), symbol antmicroRectangularConnectorsHeadersMalePins:DF40C-100DP-0.4V(51)
Changed lines of the file:
@@
 $Descr A3 16535 11693
 encoding utf-8
-Sheet 3 4
+Sheet 3 11
 Title ""
 Date ""
@@
 Comment4 ""
 $EndDescr
-$Comp
-L riscv-u74-som:DF40HC(3.0)-100DS-0.4v J1
-U 1 1 60535B3F
-P 1950 3650
-F 0 "J1" H 1950 6317 50  0000 C CNN
-F 1 "DF40HC(3.0)-100DS-0.4v" H 1950 6226 50  0000 C CNN
-F 2 "riscv-u74-som-footprints:DF40HC(3.0)-100DS-0.4v" H 1950 3650 50  0001 L BNN
-F 3 "" H 1950 3650 50  0001 L BNN
-F 4 "HRS" H 1950 3650 50  0001 L BNN "Manufacturer"
-	1    1950 3650
-	1    0    0    -1
-$EndComp
-$Comp
-L riscv-u74-som:DF40HC(3.0)-100DS-0.4v J2
-U 1 1 60537500
-P 3475 3750
-F 0 "J2" H 3475 6417 50  0000 C CNN
-F 1 "DF40HC(3.0)-100DS-0.4v" H 3475 6326 50  0000 C CNN
-F 2 "riscv-u74-som-footprints:DF40HC(3.0)-100DS-0.4v" H 3475 3750 50  0001 L BNN
-F 3 "" H 3475 3750 50  0001 L BNN
-F 4 "HRS" H 3475 3750 50  0001 L BNN "Manufacturer"
-	1    3475 3750
-	1    0    0    -1
-$EndComp
 $Comp
 L riscv-u74-som:SiFive-U74 U1
@@
 	1    0    0    -1
 $EndComp
+$Comp
+L antmicroRectangularConnectorsHeadersMalePins:DF40C-100DP-0.4V(51) J1
+U 1 1 6100E05C
+P 1950 3275
+F 0 "J1" H 1950 6032 50  0000 C CNN
+F 1 "DF40C-100DP-0.4V(51)" H 1950 5941 50  0000 C CNN
+F 2 "antmicro-footprints:HRS_DF40C-100DP-0.4V(51)" H 1950 3275 50  0001 L BNN
+F 3 "" H 1950 3275 50  0001 L BNN
+F 4 "HRS" H 1950 3275 50  0001 L BNN "Manufacturer"
+F 5 "DF40C-100DP-0.4V(51)" H 1950 5850 50  0000 C CNN "MPN"
+	1    1950 3275
+	1    0    0    -1
+$EndComp
+$Comp
+L antmicroRectangularConnectorsHeadersMalePins:DF40C-100DP-0.4V(51) J2
+U 1 1 6100F52A
+P 3350 3250
+F 0 "J2" H 3350 6007 50  0000 C CNN
+F 1 "DF40C-100DP-0.4V(51)" H 3350 5916 50  0000 C CNN
+F 2 "antmicro-footprints:HRS_DF40C-100DP-0.4V(51)" H 3350 3250 50  0001 L BNN
+F 3 "" H 3350 3250 50  0001 L BNN
+F 4 "HRS" H 3350 3250 50  0001 L BNN "Manufacturer"
+F 5 "DF40C-100DP-0.4V(51)" H 3350 5825 50  0000 C CNN "MPN"
+	1    3350 3250
+	1    0    0    -1
+$EndComp

Commit message: Renamed design files
Parts:
- SP1, SP2, SP3, SP4: footprint riscv-u74-som-footprints:9774030151 -> arv-som-footprints:9774030151; symbol riscv-u74-som:9774030151 -> arv-som:9774030151
- U1: footprint riscv-u74-som-footprints:SiFive-U74 -> arv-som-footprints:SiFive-U74; symbol riscv-u74-som:SiFive-U74 -> arv-som:SiFive-U74
- U2, U3: footprint riscv-u74-som-footprints:BGA-200_10.0x14.5mm_Layout12x22_P0.80x0.65mm -> arv-som-footprints:BGA-200_10.0x14.5mm_Layout12x22_P0.80x0.65mm; symbol riscv-u74-som:MT53E256M32D2 -> arv-som:MT53E256M32D2
- U4: footprint riscv-u74-som-footprints:S25FL128SAGNFI000 -> arv-som-footprints:S25FL128SAGNFI000; symbol riscv-u74-som:S25FL128SAGNFI000 -> arv-som:S25FL128SAGNFI000
- U5: footprint riscv-u74-som-footprints:QFN50P900X900X80-65N -> arv-som-footprints:QFN50P900X900X80-65N; symbol riscv-u74-som:TPS65086100 -> arv-som:TPS65086100
- U6: footprint riscv-u74-som-footprints:QFN50P900X900X100-65N -> arv-som-footprints:QFN50P900X900X100-65N; symbol riscv-u74-som:TDA19988BHN_C1,557 -> arv-som:TDA19988BHN_C1,557
- U7: footprint riscv-u74-som-footprints:QFN-48-Microchip-QFN77-48LD-PL-2 -> arv-som-footprints:QFN-48-Microchip-QFN77-48LD-PL-2; symbol riscv-u74-som:KSZ9031RNXCA -> arv-som:KSZ9031RNXCA
Changed lines of the file:
@@
 $EndDescr
 $Comp
-L riscv-u74-som:SiFive-U74 U1
+L arv-som:SiFive-U74 U1
 U 1 1 6053879C
 P 5125 1250
 F 0 "U1" H 5303 1171 50  0000 L CNN
 F 1 "SiFive-U74" H 5303 1080 50  0000 L CNN
-F 2 "riscv-u74-som-footprints:SiFive-U74" H 5125 1250 50  0001 C CNN
+F 2 "arv-som-footprints:SiFive-U74" H 5125 1250 50  0001 C CNN
 F 3 "" H 5125 1250 50  0001 C CNN
 	1    5125 1250
@@
 $EndComp
 $Comp
-L riscv-u74-som:MT53E256M32D2 U2
+L arv-som:MT53E256M32D2 U2
 U 1 1 6053A199
 P 7250 1875
 F 0 "U2" H 7250 286 50  0000 C CNN
 F 1 "MT53E256M32D2" H 7250 195 50  0000 C CNN
-F 2 "riscv-u74-som-footprints:BGA-200_10.0x14.5mm_Layout12x22_P0.80x0.65mm" H 7300 -25 50  0001 C CNN
+F 2 "arv-som-footprints:BGA-200_10.0x14.5mm_Layout12x22_P0.80x0.65mm" H 7300 -25 50  0001 C CNN
 F 3 "" H 7150 675 50  0001 C CNN
 	1    7250 1875
@@
 $EndComp
 $Comp
-L riscv-u74-som:MT53E256M32D2 U2
+L arv-som:MT53E256M32D2 U2
 U 2 1 6053CBCD
 P 9125 1875
 F 0 "U2" H 9125 286 50  0000 C CNN
 F 1 "MT53E256M32D2" H 9125 195 50  0000 C CNN
-F 2 "riscv-u74-som-footprints:BGA-200_10.0x14.5mm_Layout12x22_P0.80x0.65mm" H 9175 -25 50  0001 C CNN
+F 2 "arv-som-footprints:BGA-200_10.0x14.5mm_Layout12x22_P0.80x0.65mm" H 9175 -25 50  0001 C CNN
 F 3 "" H 9025 675 50  0001 C CNN
 	2    9125 1875
@@
 $EndComp
 $Comp
-L riscv-u74-som:MT53E256M32D2 U3
+L arv-som:MT53E256M32D2 U3
 U 1 1 60550D6A
 P 7225 5150
 F 0 "U3" H 7225 3561 50  0000 C CNN
 F 1 "MT53E256M32D2" H 7225 3470 50  0000 C CNN
-F 2 "riscv-u74-som-footprints:BGA-200_10.0x14.5mm_Layout12x22_P0.80x0.65mm" H 7275 3250 50  0001 C CNN
+F 2 "arv-som-footprints:BGA-200_10.0x14.5mm_Layout12x22_P0.80x0.65mm" H 7275 3250 50  0001 C CNN
 F 3 "" H 7125 3950 50  0001 C CNN
 	1    7225 5150
@@
 $EndComp
 $Comp
-L riscv-u74-som:MT53E256M32D2 U3
+L arv-som:MT53E256M32D2 U3
 U 2 1 60550D70
 P 9100 5150
 F 0 "U3" H 9100 3561 50  0000 C CNN
 F 1 "MT53E256M32D2" H 9100 3470 50  0000 C CNN
-F 2 "riscv-u74-som-footprints:BGA-200_10.0x14.5mm_Layout12x22_P0.80x0.65mm" H 9150 3250 50  0001 C CNN
+F 2 "arv-som-footprints:BGA-200_10.0x14.5mm_Layout12x22_P0.80x0.65mm" H 9150 3250 50  0001 C CNN
 F 3 "" H 9000 3950 50  0001 C CNN
 	2    9100 5150
@@
 $EndComp
 $Comp
-L riscv-u74-som:S25FL128SAGNFI000 U4
+L arv-som:S25FL128SAGNFI000 U4
 U 1 1 60559440
 P 11025 1500
 F 0 "U4" H 11725 1787 60  0000 C CNN
 F 1 "S25FL128SAGNFI000" H 11725 1681 60  0000 C CNN
-F 2 "riscv-u74-som-footprints:S25FL128SAGNFI000" H 12025 1740 60  0001 C CNN
+F 2 "arv-som-footprints:S25FL128SAGNFI000" H 12025 1740 60  0001 C CNN
 F 3 "" H 11025 1500 60  0000 C CNN
 	1    11025 1500
@@
 $EndComp
 $Comp
-L riscv-u74-som:TPS65086100 U5
+L arv-som:TPS65086100 U5
 U 1 1 605606CE
 P 12950 1600
 F 0 "U5" H 13078 1546 50  0000 L CNN
 F 1 "TPS65086100" H 13078 1455 50  0000 L CNN
-F 2 "riscv-u74-som-footprints:QFN50P900X900X80-65N" H 12950 1600 50  0001 C CNN
+F 2 "arv-som-footprints:QFN50P900X900X80-65N" H 12950 1600 50  0001 C CNN
 F 3 "" H 12950 1600 50  0001 C CNN
 	1    12950 1600
@@
 $EndComp
 $Comp
-L riscv-u74-som:TDA19988BHN_C1,557 U6
+L arv-som:TDA19988BHN_C1,557 U6
 U 1 1 605671A3
 P 12500 5550
 F 0 "U6" H 12500 8217 50  0000 C CNN
 F 1 "TDA19988BHN_C1,557" H 12500 8126 50  0000 C CNN
-F 2 "riscv-u74-som-footprints:QFN50P900X900X100-65N" H 12500 5550 50  0001 L BNN
+F 2 "arv-som-footprints:QFN50P900X900X100-65N" H 12500 5550 50  0001 L BNN
 F 3 "" H 12500 5550 50  0001 L BNN
 F 4 "NXP Semiconductors" H 12500 5550 50  0001 L BNN "MANUFACTURER"
@@
 $EndComp
 $Comp
-L riscv-u74-som:KSZ9031RNXCA U7
+L arv-som:KSZ9031RNXCA U7
 U 1 1 6058304D
 P 7825 7600
 F 0 "U7" H 8925 4511 50  0000 C CNN
 F 1 "KSZ9031RNXCA" H 8925 4420 50  0000 C CNN
-F 2 "riscv-u74-som-footprints:QFN-48-Microchip-QFN77-48LD-PL-2" H 7825 8100 50  0001 L CNN
+F 2 "arv-som-footprints:QFN-48-Microchip-QFN77-48LD-PL-2" H 7825 8100 50  0001 L CNN
 F 3 "http://ww1.microchip.com/downloads/en/DeviceDoc/00002117F.pdf" H 7825 8100 50  0001 L CNN
 F 4 "Microchip" H 7825 7900 50  0001 L CNN "Manufacturer"
@@
 $EndComp
 $Comp
-L riscv-u74-som:9774030151 SP1
+L arv-som:9774030151 SP1
 U 1 1 6059CEA0
 P 15175 1075
 F 0 "SP1" H 15305 1128 60  0000 L CNN
 F 1 "9774030151" H 15305 1022 60  0000 L CNN
-F 2 "riscv-u74-som-footprints:9774030151" H 15175 1075 60  0001 C CNN
+F 2 "arv-som-footprints:9774030151" H 15175 1075 60  0001 C CNN
 F 3 "https://www.we-online.com/catalog/datasheet/9774030151.pdf" H 15175 1075 60  0001 C CNN
 F 4 "Wurth Elektronik" H 15175 1075 50  0001 C CNN "Manufacturer"
@@
 $EndComp
 $Comp
-L riscv-u74-som:9774030151 SP2
+L arv-som:9774030151 SP2
 U 1 1 6059EA55
 P 15175 1350
 F 0 "SP2" H 15305 1403 60  0000 L CNN
 F 1 "9774030151" H 15305 1297 60  0000 L CNN
-F 2 "riscv-u74-som-footprints:9774030151" H 15175 1350 60  0001 C CNN
+F 2 "arv-som-footprints:9774030151" H 15175 1350 60  0001 C CNN
 F 3 "https://www.we-online.com/catalog/datasheet/9774030151.pdf" H 15175 1350 60  0001 C CNN
 F 4 "Wurth Elektronik" H 15175 1350 50  0001 C CNN "Manufacturer"
@@
 $EndComp
 $Comp
-L riscv-u74-som:9774030151 SP3
+L arv-som:9774030151 SP3
 U 1 1 6059ECA8
 P 15175 1625
 F 0 "SP3" H 15305 1678 60  0000 L CNN
 F 1 "9774030151" H 15305 1572 60  0000 L CNN
-F 2 "riscv-u74-som-footprints:9774030151" H 15175 1625 60  0001 C CNN
+F 2 "arv-som-footprints:9774030151" H 15175 1625 60  0001 C CNN
 F 3 "https://www.we-online.com/catalog/datasheet/9774030151.pdf" H 15175 1625 60  0001 C CNN
 F 4 "Wurth Elektronik" H 15175 1625 50  0001 C CNN "Manufacturer"
@@
 $EndComp
 $Comp
-L riscv-u74-som:9774030151 SP4
+L arv-som:9774030151 SP4
 U 1 1 6059EE21
 P 15175 1900
 F 0 "SP4" H 15305 1953 60  0000 L CNN
 F 1 "9774030151" H 15305 1847 60  0000 L CNN
-F 2 "riscv-u74-som-footprints:9774030151" H 15175 1900 60  0001 C CNN
+F 2 "arv-som-footprints:9774030151" H 15175 1900 60  0001 C CNN
 F 3 "https://www.we-online.com/catalog/datasheet/9774030151.pdf" H 15175 1900 60  0001 C CNN
 F 4 "Wurth Elektronik" H 15175 1900 50  0001 C CNN "Manufacturer"
