File: PMIC.sch (KiCad schematic (older format))
At the start: 70 parts

Commit message: Connected interfaces to VIC to visualise its ball locations (wip, mock purposes)
Parts:
- gave numbers to parts that had none: 70
Connections:
- net labels added: I2C0_SCL, I2C0_SDA, VDD2PEN
- net labels removed: FNSH028_VDD2PEN, FNSH055_I2C0_SDA, FNSH056_I2C0_SCL

Commit message: Updated interfaces, CPU and B2B connector connections
Other:
- note added: "TODO: find valid replacement for \nCSD87381P"
Changed lines of the file:
@@
 $Descr A3 16535 11693
 encoding utf-8
-Sheet 2 11
+Sheet 2 10
 Title ""
 Date ""
@@
 Wire Wire Line
 	4200 5975 4375 5975
+Text Notes 8825 3700 0    50   ~ 0
+TODO: find valid replacement for \nCSD87381P
+Text Notes 9750 5925 0    50   ~ 0
+TODO: find valid replacement for \nCSD87381P
 $EndSCHEMATC

Commit message: Schematic cleanup, added logotypes
Other:
- note added: "5V8 boost regulator"
