File: PMIC.sch (KiCad schematic (older format))
At the start: 70 parts, among them Q1 BSS138AKA, Q2 BSS138AKA, Q3 BSS138AKA, Q4 BSS138AKA, U5 LMR62014XMF_NOPB, U8 TPS65086100

Commit message: PMIC fixed and cleaned
Parts:
- removed C12: C_1n_0603, antmicro-footprints:0603-cap, symbol antmicroCapacitors0603:C_1n_0603
- removed C3, C4, C8: C_2u2_0402, antmicro-footprints:0402-cap, symbol antmicroCapacitors0402:C_2u2_0402
- removed Q1, Q2, Q3, Q4: BSS138AKA, antmicro-footprints:SOT-23-3, symbol antmicroTransistorsFETsMOSFETsSingle:BSS138AKA
- removed R1: R_1M_0603, antmicro-footprints:0603-res, symbol antmicroResistors0603:R_1M_0603
- removed R8: R_549k_0603, antmicro-footprints:0603-res, symbol antmicroResistors0603:R_549k_0603
- removed R9: R_13k3_0603, antmicro-footprints:0603-res, symbol antmicroResistors0603:R_13k3_0603
- removed S1: B3F-1000, antmicro-footprints:Switch_Tactile_THT_B3F-1xxx, symbol antmicroTactileSwitches:B3F-1000
- added C12: C_1n0_0402, antmicro-footprints:0402-cap, symbol antmicroCapacitors0402:C_1n0_0402
- added C3, C4, C8: C_10u_0402, antmicro-footprints:0402-cap, symbol antmicroCapacitors0402:C_10u_0402
- added C?: C_100n_0402_16V, antmicro-footprints:0402-cap, symbol antmicroCapacitorsmisc:C_100n_0402_16V
- added R1: R_1M0_0402, antmicro-footprints:0402-res, symbol antmicroResistors0402:R_1M0_0402
- added R8: R_49k9_0402, antmicro-footprints:0402-res, symbol antmicroResistors0402:R_49k9_0402
- added R9: R_13k3_0402, antmicro-footprints:0402-res, symbol antmicroResistors0402:R_13k3_0402
- added R?: R_10k_0402, antmicro-footprints:0402-res, symbol antmicroResistors0402:R_10k_0402
- added S1: B3U-3000PM, antmicro-footprints:B3U-3000P, symbol antmicroPushbuttonSwitches:B3U-3000PM
- added U? (x2): CSD86330Q3D, antmicro-footprints:CSD86330Q3D, symbol antmicroTransistorsFETsMOSFETsArrays:CSD86330Q3D
Connections:
- net labels added: U5FB
- net labels removed: FB
- wire segments 226 -> 254
Other:
- note added: "ARV SoM - Power Mangement"
- note added: "PMIC OTP"
- note removed: "TODO: find valid replacement for \nCSD87381P"
- note removed: "TODO: replace with 49k9 resistor"

Commit message: Added title block settings
Parts:
- removed C12: C_1n0_0402, antmicro-footprints:0402-cap, symbol antmicroCapacitors0402:C_1n0_0402
- removed C3, C4, C8: C_10u_0402, antmicro-footprints:0402-cap, symbol antmicroCapacitors0402:C_10u_0402
- removed C?: C_100n_0402_16V, antmicro-footprints:0402-cap, symbol antmicroCapacitorsmisc:C_100n_0402_16V
- removed R1: R_1M0_0402, antmicro-footprints:0402-res, symbol antmicroResistors0402:R_1M0_0402
- removed R8: R_49k9_0402, antmicro-footprints:0402-res, symbol antmicroResistors0402:R_49k9_0402
- removed R9: R_13k3_0402, antmicro-footprints:0402-res, symbol antmicroResistors0402:R_13k3_0402
- removed R?: R_10k_0402, antmicro-footprints:0402-res, symbol antmicroResistors0402:R_10k_0402
- removed S1: B3U-3000PM, antmicro-footprints:B3U-3000P, symbol antmicroPushbuttonSwitches:B3U-3000PM
- removed U? (x2): CSD86330Q3D, antmicro-footprints:CSD86330Q3D, symbol antmicroTransistorsFETsMOSFETsArrays:CSD86330Q3D
- added C12: C_1n_0603, antmicro-footprints:0603-cap, symbol antmicroCapacitors0603:C_1n_0603
- added C3, C4, C8: C_2u2_0402, antmicro-footprints:0402-cap, symbol antmicroCapacitors0402:C_2u2_0402
- added Q1, Q2, Q3, Q4: BSS138AKA, antmicro-footprints:SOT-23-3, symbol antmicroTransistorsFETsMOSFETsSingle:BSS138AKA
- added R1: R_1M_0603, antmicro-footprints:0603-res, symbol antmicroResistors0603:R_1M_0603
- added R8: R_549k_0603, antmicro-footprints:0603-res, symbol antmicroResistors0603:R_549k_0603
- added R9: R_13k3_0603, antmicro-footprints:0603-res, symbol antmicroResistors0603:R_13k3_0603
- added S1: B3F-1000, antmicro-footprints:Switch_Tactile_THT_B3F-1xxx, symbol antmicroTactileSwitches:B3F-1000
Connections:
- net labels added: FB
- net labels removed: U5FB
- wire segments 254 -> 226
Other:
- note added: "TODO: find valid replacement for \nCSD87381P"
- note added: "TODO: replace with 49k9 resistor"
- note removed: "ARV SoM - Power Mangement"
- note removed: "PMIC OTP"

Commit message: PMIC restored
Parts:
- removed C12: C_1n_0603, antmicro-footprints:0603-cap, symbol antmicroCapacitors0603:C_1n_0603
- removed C3, C4, C8: C_2u2_0402, antmicro-footprints:0402-cap, symbol antmicroCapacitors0402:C_2u2_0402
- removed Q1, Q2, Q3, Q4: BSS138AKA, antmicro-footprints:SOT-23-3, symbol antmicroTransistorsFETsMOSFETsSingle:BSS138AKA
- removed R1: R_1M_0603, antmicro-footprints:0603-res, symbol antmicroResistors0603:R_1M_0603
- removed R8: R_549k_0603, antmicro-footprints:0603-res, symbol antmicroResistors0603:R_549k_0603
- removed R9: R_13k3_0603, antmicro-footprints:0603-res, symbol antmicroResistors0603:R_13k3_0603
- removed S1: B3F-1000, antmicro-footprints:Switch_Tactile_THT_B3F-1xxx, symbol antmicroTactileSwitches:B3F-1000
- added C12: C_1n0_0402, antmicro-footprints:0402-cap, symbol antmicroCapacitors0402:C_1n0_0402
- added C242: C_100n_0402_16V, antmicro-footprints:0402-cap, symbol antmicroCapacitorsmisc:C_100n_0402_16V
- added C3, C4, C8: C_10u_0402, antmicro-footprints:0402-cap, symbol antmicroCapacitors0402:C_10u_0402
- added R1: R_1M0_0402, antmicro-footprints:0402-res, symbol antmicroResistors0402:R_1M0_0402
- added R121: R_10k_0402, antmicro-footprints:0402-res, symbol antmicroResistors0402:R_10k_0402
- added R8: R_49k9_0402, antmicro-footprints:0402-res, symbol antmicroResistors0402:R_49k9_0402
- added R9: R_13k3_0402, antmicro-footprints:0402-res, symbol antmicroResistors0402:R_13k3_0402
- added S1: B3U-3000PM, antmicro-footprints:B3U-3000P, symbol antmicroPushbuttonSwitches:B3U-3000PM
- added U4, U6: CSD86330Q3D, antmicro-footprints:CSD86330Q3D, symbol antmicroTransistorsFETsMOSFETsArrays:CSD86330Q3D
Connections:
- net labels added: PWR_OFF, U5FB
- net labels removed: FB
- wire segments 226 -> 254
Other:
- note added: "ARV SoM - Power Mangement"
- note added: "PMIC OTP"
- note removed: "TODO: find valid replacement for \nCSD87381P"
- note removed: "TODO: replace with 49k9 resistor"

Commit message: Added local libraries
Parts:
- C1, C16, C27, C28: footprint antmicro-footprints:0603-cap -> arv-som-footprints:0603-cap; symbol antmicroCapacitors0603:C_10u_0603 -> arv-som:C_10u_0603
- C10, C13, C17, C18, C242: footprint antmicro-footprints:0402-cap -> arv-som-footprints:0402-cap; symbol antmicroCapacitorsmisc:C_100n_0402_16V -> arv-som:C_100n_0402_16V
- C11, C14, C6: footprint antmicro-footprints:0402-cap -> arv-som-footprints:0402-cap; symbol antmicroCapacitors0402:C_4u7_0402 -> arv-som:C_4u7_0402
- C12: footprint antmicro-footprints:0402-cap -> arv-som-footprints:0402-cap; symbol antmicroCapacitors0402:C_1n0_0402 -> arv-som:C_1n0_0402
- C15, C2, C5, C7, C9: footprint antmicro-footprints:0402-cap -> arv-som-footprints:0402-cap; symbol antmicroCapacitors0402:C_2u2_0402 -> arv-som:C_2u2_0402
- C19, C20, C21, C22, C29, C30, C31, C32, C33, C34: footprint antmicro-footprints:0603-cap -> arv-som-footprints:0603-cap; symbol antmicroCapacitors0603:C_22u_0603 -> arv-som:C_22u_0603
- C23, C24, C25, C26: footprint antmicro-footprints:0805-cap -> arv-som-footprints:0805-cap; symbol antmicroCapacitorsmisc:C_100u_0805 -> arv-som:C_100u_0805
- C3, C4, C8: footprint antmicro-footprints:0402-cap -> arv-som-footprints:0402-cap; symbol antmicroCapacitors0402:C_10u_0402 -> arv-som:C_10u_0402
- D1: footprint antmicro-footprints:PGB1010603MR -> arv-som-footprints:PGB1010603MR; symbol antmicroTVSDiodes:PGB1010603MR -> arv-som:PGB1010603MR
- D2: footprint antmicro-footprints:SOD-123 -> arv-som-footprints:SOD-123; symbol antmicroDiodesRectifiersSingle:1N4148W-TP -> arv-som:1N4148W-TP
- L1: footprint antmicro-footprints:0805-res -> arv-som-footprints:0805-res; symbol antmicroFixedInductors:10uH -> arv-som:10uH
- L2, L3, L4: footprint antmicro-footprints:IND_LQH32PN1R0NN0L -> arv-som-footprints:IND_LQH32PN1R0NN0L; symbol antmicroFixedInductors:LQH32PN1R0NN0L -> arv-som:LQH32PN1R0NN0L
- L5: footprint antmicro-footprints:MPX1D0520LR47 -> arv-som-footprints:MPX1D0520LR47; symbol antmicroFixedInductors:MPX1D0520LR47 -> arv-som:MPX1D0520LR47
- L6: footprint antmicro-footprints:IHLP4040DZERR56M01 -> arv-som-footprints:IHLP4040DZERR56M01; symbol antmicroFixedInductors:IHLP4040DZERR56M01 -> arv-som:IHLP4040DZERR56M01
- R1: footprint antmicro-footprints:0402-res -> arv-som-footprints:0402-res; symbol antmicroResistors0402:R_1M0_0402 -> arv-som:R_1M0_0402
- R10, R11, R12, R14, R15, R16, R5, R6: footprint antmicro-footprints:0402-res -> arv-som-footprints:0402-res; symbol antmicroResistors0402:R_0R_0402 -> arv-som:R_0R_0402
- R121, R2, R3, R4: footprint antmicro-footprints:0402-res -> arv-som-footprints:0402-res; symbol antmicroResistors0402:R_10k_0402 -> arv-som:R_10k_0402
- R13, R17: footprint antmicro-footprints:0402-res -> arv-som-footprints:0402-res; symbol antmicroResistors0402:R_4k7_0402 -> arv-som:R_4k7_0402
- R7: footprint antmicro-footprints:0402-res -> arv-som-footprints:0402-res; symbol antmicroResistors0402:R_2k2_0402 -> arv-som:R_2k2_0402
- R8: footprint antmicro-footprints:0402-res -> arv-som-footprints:0402-res; symbol antmicroResistors0402:R_49k9_0402 -> arv-som:R_49k9_0402
- R9: footprint antmicro-footprints:0402-res -> arv-som-footprints:0402-res; symbol antmicroResistors0402:R_13k3_0402 -> arv-som:R_13k3_0402
- S1: footprint antmicro-footprints:B3U-3000P -> arv-som-footprints:B3U-3000P; symbol antmicroPushbuttonSwitches:B3U-3000PM -> arv-som:B3U-3000PM
- TP1, TP2, TP3, TP4: footprint antmicro-footprints:Testpoint_smd_1mm -> arv-som-footprints:Testpoint_smd_1mm; symbol antmicroTestPoints:TP_SMD1MM -> arv-som:TP_SMD1MM
- U4, U6: footprint antmicro-footprints:CSD86330Q3D -> arv-som-footprints:CSD86330Q3D; symbol antmicroTransistorsFETsMOSFETsArrays:CSD86330Q3D -> arv-som:CSD86330Q3D
- U5: footprint antmicro-footprints:SOT95P280X145-5N -> arv-som-footprints:SOT95P280X145-5N; symbol antmicroPMICVoltageRegulatorsLinear:LMR62014XMF_NOPB -> arv-som:LMR62014XMF_NOPB
- U8: footprint antmicro-footprints:QFN50P900X900X80-65N -> arv-som-footprints:QFN50P900X900X80-65N; symbol antmicroPMICBatteryManagement:TPS65086100 -> arv-som:TPS65086100

Commit message: Update naming convention
Parts:
- C1, C16, C27, C28: footprint arv-som-footprints:0603-cap -> arvsom-footprints:0603-cap; symbol arv-som:C_10u_0603 -> arvsom:C_10u_0603
- C10, C13, C17, C18, C242: footprint arv-som-footprints:0402-cap -> arvsom-footprints:0402-cap; symbol arv-som:C_100n_0402_16V -> arvsom:C_100n_0402_16V
- C11, C14, C6: footprint arv-som-footprints:0402-cap -> arvsom-footprints:0402-cap; symbol arv-som:C_4u7_0402 -> arvsom:C_4u7_0402
- C12: footprint arv-som-footprints:0402-cap -> arvsom-footprints:0402-cap; symbol arv-som:C_1n0_0402 -> arvsom:C_1n0_0402
- C15, C2, C5, C7, C9: footprint arv-som-footprints:0402-cap -> arvsom-footprints:0402-cap; symbol arv-som:C_2u2_0402 -> arvsom:C_2u2_0402
- C19, C20, C21, C22, C29, C30, C31, C32, C33, C34: footprint arv-som-footprints:0603-cap -> arvsom-footprints:0603-cap; symbol arv-som:C_22u_0603 -> arvsom:C_22u_0603
- C23, C24, C25, C26: footprint arv-som-footprints:0805-cap -> arvsom-footprints:0805-cap; symbol arv-som:C_100u_0805 -> arvsom:C_100u_0805
- C3, C4, C8: footprint arv-som-footprints:0402-cap -> arvsom-footprints:0402-cap; symbol arv-som:C_10u_0402 -> arvsom:C_10u_0402
- D1: footprint arv-som-footprints:PGB1010603MR -> arvsom-footprints:PGB1010603MR; symbol arv-som:PGB1010603MR -> arvsom:PGB1010603MR
- D2: footprint arv-som-footprints:SOD-123 -> arvsom-footprints:SOD-123; symbol arv-som:1N4148W-TP -> arvsom:1N4148W-TP
- L1: footprint arv-som-footprints:0805-res -> arvsom-footprints:0805-res; symbol arv-som:10uH -> arvsom:10uH
- L2, L3, L4: footprint arv-som-footprints:IND_LQH32PN1R0NN0L -> arvsom-footprints:IND_LQH32PN1R0NN0L; symbol arv-som:LQH32PN1R0NN0L -> arvsom:LQH32PN1R0NN0L
- L5: footprint arv-som-footprints:MPX1D0520LR47 -> arvsom-footprints:MPX1D0520LR47; symbol arv-som:MPX1D0520LR47 -> arvsom:MPX1D0520LR47
- L6: footprint arv-som-footprints:IHLP4040DZERR56M01 -> arvsom-footprints:IHLP4040DZERR56M01; symbol arv-som:IHLP4040DZERR56M01 -> arvsom:IHLP4040DZERR56M01
- R1: footprint arv-som-footprints:0402-res -> arvsom-footprints:0402-res; symbol arv-som:R_1M0_0402 -> arvsom:R_1M0_0402
- R10, R11, R12, R14, R15, R16, R5, R6: footprint arv-som-footprints:0402-res -> arvsom-footprints:0402-res; symbol arv-som:R_0R_0402 -> arvsom:R_0R_0402
- R121, R2, R3, R4: footprint arv-som-footprints:0402-res -> arvsom-footprints:0402-res; symbol arv-som:R_10k_0402 -> arvsom:R_10k_0402
- R13, R17: footprint arv-som-footprints:0402-res -> arvsom-footprints:0402-res; symbol arv-som:R_4k7_0402 -> arvsom:R_4k7_0402
- R7: footprint arv-som-footprints:0402-res -> arvsom-footprints:0402-res; symbol arv-som:R_2k2_0402 -> arvsom:R_2k2_0402
- R8: footprint arv-som-footprints:0402-res -> arvsom-footprints:0402-res; symbol arv-som:R_49k9_0402 -> arvsom:R_49k9_0402
- R9: footprint arv-som-footprints:0402-res -> arvsom-footprints:0402-res; symbol arv-som:R_13k3_0402 -> arvsom:R_13k3_0402
- S1: footprint arv-som-footprints:B3U-3000P -> arvsom-footprints:B3U-3000P; symbol arv-som:B3U-3000PM -> arvsom:B3U-3000PM
- TP1, TP2, TP3, TP4: footprint arv-som-footprints:Testpoint_smd_1mm -> arvsom-footprints:Testpoint_smd_1mm; symbol arv-som:TP_SMD1MM -> arvsom:TP_SMD1MM
- U4, U6: footprint arv-som-footprints:CSD86330Q3D -> arvsom-footprints:CSD86330Q3D; symbol arv-som:CSD86330Q3D -> arvsom:CSD86330Q3D
- U5: footprint arv-som-footprints:SOT95P280X145-5N -> arvsom-footprints:SOT95P280X145-5N; symbol arv-som:LMR62014XMF_NOPB -> arvsom:LMR62014XMF_NOPB
- U8: footprint arv-som-footprints:QFN50P900X900X80-65N -> arvsom-footprints:QFN50P900X900X80-65N; symbol arv-som:TPS65086100 -> arvsom:TPS65086100
