File: PMIC.sch (KiCad schematic (older format))
At the start: 70 parts, among them U4 CSD86330Q3D, U5 LMR62014XMF_NOPB, U6 CSD86330Q3D, U8 TPS65086100

Commit message: Updated PMIC to match B0.9
Parts:
- removed R121: R_10k_0402, arvsom-footprints:0402-res, symbol arvsom:R_10k_0402
- removed R13: R_4k7_0402, arvsom-footprints:0402-res, symbol arvsom:R_4k7_0402
- added R121: R_1k_0402, antmicro-footprints:0402-res, symbol antmicroResistors0402:R_1k_0402
- added R123: R_0R_0402, antmicro-footprints:0402-res, symbol antmicroResistors0402:R_0R_0402
- added R13: R_12k1_0402, antmicro-footprints:0402-res, symbol antmicroResistors0402:R_12k1_0402
Connections:
- wire segments 254 -> 256
Other:
- moved on the sheet: C242, C6, D1, S1
Changed lines of the file:
@@
 	5900 3275 5900 2500
 Text GLabel 5900 2500 1    50   Input ~ 0
-VCC_1V1
+VCC_0V9
 Wire Wire Line
 	5400 3125 5400 2625
@@
 	1    0    0    -1
 $EndComp
-Text GLabel 4650 5575 0    50   Input ~ 0
+Text GLabel 4125 5575 0    50   Input ~ 0
 SYS_RSTN
 NoConn ~ 6125 5225
@@
 L arvsom:C_4u7_0402 C6
 U 1 1 6078F3CE
-P 4900 5925
-F 0 "C6" H 5000 6000 60  0000 L CNN
-F 1 "C_4u7_0402" H 4900 5775 60  0001 C CNN
-F 2 "arvsom-footprints:0402-cap" H 5100 6125 60  0001 L CNN
-F 3 "" H 4900 5925 50  0001 C CNN
-F 4 "MURATA" H 5100 6325 60  0001 L CNN "Manufacturer"
-F 5 "GRM155R61A475MEAAD" H 5100 6225 60  0001 L CNN "MPN"
-F 6 "4u7" H 4950 5825 50  0000 L CNN "Val"
-	1    4900 5925
+P 5325 5925
+F 0 "C6" H 5050 5975 60  0000 L CNN
+F 1 "C_4u7_0402" H 5325 5775 60  0001 C CNN
+F 2 "arvsom-footprints:0402-cap" H 5525 6125 60  0001 L CNN
+F 3 "" H 5325 5925 50  0001 C CNN
+F 4 "MURATA" H 5525 6325 60  0001 L CNN "Manufacturer"
+F 5 "GRM155R61A475MEAAD" H 5525 6225 60  0001 L CNN "MPN"
+F 6 "4u7" H 5050 5900 50  0000 L CNN "Val"
+	1    5325 5925
 	1    0    0    -1
 $EndComp
@@
 Wire Wire Line
 	8125 4075 8350 4075
-$Comp
-L arvsom:R_4k7_0402 R13
-U 1 1 608C48A7
-P 8500 4475
-F 0 "R13" H 8275 4525 60  0000 C CNN
-F 1 "R_4k7_0402" H 8500 4325 60  0001 C CNN
-F 2 "arvsom-footprints:0402-res" H 8700 4675 60  0001 L CNN
-F 3 "" H 8500 4475 50  0001 C CNN
-F 4 "PANASONIC_ELECTRONIC_COMPONENTS" H 8700 4875 60  0001 L CNN "Manufacturer"
-F 5 "ERJ2GEJ472X" H 8700 4775 60  0001 L CNN "MPN"
-F 6 "4k7" H 8275 4425 50  0000 C CNN "Val"
-	1    8500 4475
-	1    0    0    -1
-$EndComp
 Wire Wire Line
 	8125 4475 8350 4475
@@
 VCC_5V0
 Text GLabel 12875 3775 2    50   Input ~ 0
-VCC_0V9
+VCC_1V1
 $Comp
 L arvsom:C_100u_0805 C24
@@
 VCC_5V0
 Text GLabel 12875 6075 2    50   Input ~ 0
-VCC_1V1
+VCC_0V9
 Wire Wire Line
 	9000 6775 11375 6775
@@
 L arvsom:GND #PWR0129
 U 1 1 60A44B2E
-P 3500 5325
-F 0 "#PWR0129" H 3500 5075 50  0001 C CNN
-F 1 "GND" H 3505 5152 50  0000 C CNN
-F 2 "" H 3500 5325 50  0001 C CNN
-F 3 "" H 3500 5325 50  0001 C CNN
-	1    3500 5325
+P 3500 5050
+F 0 "#PWR0129" H 3500 4800 50  0001 C CNN
+F 1 "GND" H 3505 4877 50  0000 C CNN
+F 2 "" H 3500 5050 50  0001 C CNN
+F 3 "" H 3500 5050 50  0001 C CNN
+	1    3500 5050
 	1    0    0    -1
 $EndComp
@@
 L arvsom:B3U-3000PM S1
 U 1 1 608A76FB
-P 3500 5125
-F 0 "S1" V 3575 5325 50  0000 C CNN
-F 1 "B3U-3000PM" H 3450 5000 50  0000 C CNN
-F 2 "arvsom-footprints:B3U-3000P" H 3700 5325 50  0001 L CNN
-F 3 "http://www.farnell.com/datasheets/2610940.pdf" H 3700 5425 60  0001 L CNN
-F 4 "B3U-3000PM" H 3696 5518 60  0001 L CNN "MPN"
-F 5 "OMRON" H 3700 5597 60  0001 L CNN "Manufacturer"
-	1    3500 5125
+P 3500 4850
+F 0 "S1" V 3575 5050 50  0000 C CNN
+F 1 "B3U-3000PM" H 3450 4725 50  0000 C CNN
+F 2 "arvsom-footprints:B3U-3000P" H 3700 5050 50  0001 L CNN
+F 3 "http://www.farnell.com/datasheets/2610940.pdf" H 3700 5150 60  0001 L CNN
+F 4 "B3U-3000PM" H 3696 5243 60  0001 L CNN "MPN"
+F 5 "OMRON" H 3700 5322 60  0001 L CNN "Manufacturer"
+	1    3500 4850
 	0    -1   -1   0
 $EndComp
@@
 	5825 4225 6125 4225
 Wire Wire Line
-	4650 5575 4900 5575
+	4125 5575 4900 5575
 Wire Wire Line
 	5900 5575 5900 5125
@@
 Connection ~ 4900 5575
 Wire Wire Line
-	4900 5575 5900 5575
+	4900 5575 5275 5575
 Wire Notes Line
 	5650 4200 5650 5200
@@
 	4125 6125 4425 6125
 Connection ~ 4425 6125
-Connection ~ 4900 5775
-Wire Wire Line
-	4900 5775 6125 5775
 Wire Wire Line
-	4900 6175 4900 6075
-Wire Wire Line
-	4125 5775 4900 5775
+	5325 6175 5325 6075
 Wire Wire Line
 	8525 3225 8325 3225
@@
 Connection ~ 9875 6575
 $Comp
-L arvsom:GND #PWR0127
-U 1 1 609E6360
-P 8375 3725
-F 0 "#PWR0127" H 8375 3475 50  0001 C CNN
-F 1 "GND" H 8375 3575 50  0000 C CNN
-F 2 "" H 8375 3725 50  0001 C CNN
-F 3 "" H 8375 3725 50  0001 C CNN
-	1    8375 3725
-	1    0    0    -1
-$EndComp
-$Comp
 L arvsom:C_22u_0603 C21
 U 1 1 609E6351
@@
 Wire Wire Line
 	12675 5125 12875 5125
-$Comp
-L arvsom:R_10k_0402 R121
-U 1 1 615719DA
-P 3650 3750
-F 0 "R121" V 3605 3820 60  0000 L CNN
-F 1 "R_10k_0402" H 3650 3600 60  0001 C CNN
-F 2 "arvsom-footprints:0402-res" H 3850 3950 60  0001 L CNN
-F 3 "" H 3650 3750 50  0001 C CNN
-F 4 "VISHAY" H 3850 4150 60  0001 L CNN "Manufacturer"
-F 5 "CRCW040210K0FKEDHP" H 3850 4050 60  0001 L CNN "MPN"
-F 6 "10k" V 3703 3820 50  0000 L CNN "Val"
-	1    3650 3750
-	0    1    1    0
-$EndComp
 Connection ~ 3925 4325
 Wire Wire Line
@@
 L arvsom:C_100n_0402_16V C242
 U 1 1 616769CC
-P 3650 4525
-F 0 "C242" H 3375 4500 60  0000 L CNN
-F 1 "C_100n_0402_16V" H 3650 4375 60  0001 C CNN
-F 2 "arvsom-footprints:0402-cap" H 3850 4725 60  0001 L CNN
-F 3 "" H 3650 4525 50  0001 C CNN
-F 4 "MULTICOMP" H 3850 4925 60  0001 L CNN "Manufacturer"
-F 5 "MC0402B104K160CT" H 3850 4825 60  0001 L CNN "MPN"
-F 6 "100n" H 3375 4425 50  0000 L CNN "Val"
-	1    3650 4525
-	1    0    0    -1
-$EndComp
-$Comp
-L arvsom:GND #PWR014
-U 1 1 6167B2DA
-P 3650 4675
-F 0 "#PWR014" H 3650 4425 50  0001 C CNN
-F 1 "GND" H 3800 4600 50  0000 C CNN
-F 2 "" H 3650 4675 50  0001 C CNN
-F 3 "" H 3650 4675 50  0001 C CNN
-	1    3650 4675
+P 4900 5950
+F 0 "C242" H 4550 6000 60  0000 L CNN
+F 1 "C_100n_0402_16V" H 4900 5800 60  0001 C CNN
+F 2 "arvsom-footprints:0402-cap" H 5100 6150 60  0001 L CNN
+F 3 "" H 4900 5950 50  0001 C CNN
+F 4 "MULTICOMP" H 5100 6350 60  0001 L CNN "Manufacturer"
+F 5 "MC0402B104K160CT" H 5100 6250 60  0001 L CNN "MPN"
+F 6 "100n" H 4550 5925 50  0000 L CNN "Val"
+	1    4900 5950
 	1    0    0    -1
 $EndComp
-Wire Wire Line
-	3650 4375 3650 4125
 $Comp
 L arvsom:GND #PWR0130
 U 1 1 60A9AEF8
-P 3925 5325
-F 0 "#PWR0130" H 3925 5075 50  0001 C CNN
-F 1 "GND" H 3930 5152 50  0000 C CNN
-F 2 "" H 3925 5325 50  0001 C CNN
-F 3 "" H 3925 5325 50  0001 C CNN
-	1    3925 5325
+P 3925 5050
+F 0 "#PWR0130" H 3925 4800 50  0001 C CNN
+F 1 "GND" H 3930 4877 50  0000 C CNN
+F 2 "" H 3925 5050 50  0001 C CNN
+F 3 "" H 3925 5050 50  0001 C CNN
+	1    3925 5050
 	1    0    0    -1
 $EndComp
 Wire Wire Line
-	3925 4925 3925 4875
+	3925 4650 3925 4600
 $Comp
 L arvsom:PGB1010603MR D1
 U 1 1 60A9081E
-P 3925 5125
-F 0 "D1" V 4025 5350 60  0000 R CNN
-F 1 "PGB1010603MR" H 4300 5000 60  0000 R CNN
-F 2 "arvsom-footprints:PGB1010603MR" H 4125 5325 60  0001 L CNN
-F 3 "https://www.littelfuse.com/data/en/data_sheets/littelfuse_pulseguard-esd_pgb1.pdf" H 4125 5425 60  0001 L CNN
-F 4 "Littelfuse Inc." H 4125 6225 60  0001 L CNN "Manufacturer"
-F 5 "PGB1010603MR" H 4125 5625 60  0001 L CNN "MPN"
-	1    3925 5125
+P 3925 4850
+F 0 "D1" V 4025 5075 60  0000 R CNN
+F 1 "PGB1010603MR" H 4300 4725 60  0000 R CNN
+F 2 "arvsom-footprints:PGB1010603MR" H 4125 5050 60  0001 L CNN
+F 3 "https://www.littelfuse.com/data/en/data_sheets/littelfuse_pulseguard-esd_pgb1.pdf" H 4125 5150 60  0001 L CNN
+F 4 "Littelfuse Inc." H 4125 5950 60  0001 L CNN "Manufacturer"
+F 5 "PGB1010603MR" H 4125 5350 60  0001 L CNN "MPN"
+	1    3925 4850
 	0    -1   -1   0
 $EndComp
 Wire Wire Line
-	3500 5275 3500 5325
-Wire Wire Line
-	3500 4975 3500 4875
+	3500 5000 3500 5050
 Wire Wire Line
-	3500 4875 3925 4875
-Connection ~ 3925 4875
+	3500 4700 3500 4600
 Wire Wire Line
-	3925 4875 3925 4325
+	3500 4600 3925 4600
 $Comp
 L arvsom:R_1M0_0402 R1
@@
 Wire Wire Line
 	11025 6075 11375 6075
+$Comp
+L antmicroResistors0402:R_1k_0402 R121
+U 1 1 60BEDFDF
+P 3650 3750
+F 0 "R121" V 3700 4050 60  0000 R CNN
+F 1 "R_1k_0402" H 3650 3600 60  0001 C CNN
+F 2 "antmicro-footprints:0402-res" H 3850 3950 60  0001 L CNN
+F 3 "" H 3650 3750 50  0001 C CNN
+F 4 "BOURNS" H 3850 4150 60  0001 L CNN "Manufacturer"
+F 5 "CR0402-FX-1001GLF" H 3850 4050 60  0001 L CNN "MPN"
+F 6 "1k" V 3600 4050 50  0000 R CNN "Val"
+	1    3650 3750
+	0    -1   -1   0
+$EndComp
+Wire Wire Line
+	3925 4600 3925 4325
+Connection ~ 3925 4600
+$Comp
+L antmicroResistors0402:R_0R_0402 R123
+U 1 1 60C2519F
+P 5425 5575
+F 0 "R123" H 5375 5700 60  0000 C CNN
+F 1 "R_0R_0402" H 5425 5425 60  0001 C CNN
+F 2 "antmicro-footprints:0402-res" H 5625 5775 60  0001 L CNN
+F 3 "" H 5425 5575 50  0001 C CNN
+F 4 "PANASONIC" H 5625 5975 60  0001 L CNN "Manufacturer"
+F 5 "ERJ2GE0R00X" H 5625 5875 60  0001 L CNN "MPN"
+F 6 "0R" H 5525 5675 50  0000 C CNN "Val"
+	1    5425 5575
+	1    0    0    -1
+$EndComp
+Connection ~ 5325 5775
+Wire Wire Line
+	5325 5775 6125 5775
+Wire Wire Line
+	4125 5775 5325 5775
+$Comp
+L arvsom:GND #PWR0116
+U 1 1 60C37C76
+P 5325 6175
+F 0 "#PWR0116" H 5325 5925 50  0001 C CNN
+F 1 "GND" H 5330 6002 50  0000 C CNN
+F 2 "" H 5325 6175 50  0001 C CNN
+F 3 "" H 5325 6175 50  0001 C CNN
+	1    5325 6175
+	1    0    0    -1
+$EndComp
+Wire Wire Line
+	4900 5800 4900 5575
+Wire Wire Line
+	4900 6100 4900 6175
+Wire Wire Line
+	5575 5575 5900 5575
+$Comp
+L antmicroResistors0402:R_12k1_0402 R13
+U 1 1 60C62589
+P 8500 4475
+F 0 "R13" H 8275 4525 60  0000 C CNN
+F 1 "R_12k1_0402" H 8500 4325 60  0001 C CNN
+F 2 "antmicro-footprints:0402-res" H 8700 4675 60  0001 L CNN
+F 3 "" H 8500 4475 50  0001 C CNN
+F 4 "MULTICOMP" H 8700 4875 60  0001 L CNN "Manufacturer"
+F 5 "MCWR04X1212FTL" H 8700 4775 60  0001 L CNN "MPN"
+F 6 "12k1" H 8275 4425 50  0000 C CNN "Val"
+	1    8500 4475
+	1    0    0    -1
+$EndComp
 $EndSCHEMATC
