File: decoupling.sch (KiCad schematic (older format))
At the start: 101 parts

Commit message: Added processor and B2B sheets
Parts:
- removed C? (x5): C_1u_0402, antmicro-footprints:0402-cap, symbol antmicroCapacitors0402:C_1u_0402
- removed C? (x44): C_100n_0201, antmicro-footprints:0201-res, symbol antmicroCapacitorsmisc:C_100n_0201
- removed C? (x5): C_22u_0603, antmicro-footprints:0603-cap, symbol antmicroCapacitors0603:C_22u_0603
- removed C? (x7): C_10u_0402, antmicro-footprints:0402-cap, symbol antmicroCapacitors0402:C_10u_0402
- removed C? (x4): C_1n_0402, antmicro-footprints:0402-res, symbol antmicroCapacitors0402:C_1n_0402
- removed FB?: BLM15PD121SN1D, antmicro-footprints:0402-res, symbol antmicroFerriteBeadsandChips:BLM15PD121SN1D
Connections:
- net labels removed: AVDD09_PLL, VCC_1V1
- wire segments 396 -> 141
Other:
- note removed: "VDDPLL_DDR0"
- note removed: "VDDPLL_DDR1"
- note removed: "VDDQCK_DDR0"
- note removed: "VDDQCK_DDR1"

Commit message: Connected interfaces to VIC to visualise its ball locations (wip, mock purposes)
Parts:
- removed C? (x2): C_10u_0402, antmicro-footprints:0402-cap, symbol antmicroCapacitors0402:C_10u_0402
- removed C? (x11): C_1u_0402, antmicro-footprints:0402-cap, symbol antmicroCapacitors0402:C_1u_0402
- removed C? (x21): C_100n_0201, antmicro-footprints:0201-res, symbol antmicroCapacitorsmisc:C_100n_0201
- removed FB?: BLM15PD121SN1D, antmicro-footprints:0402-res, symbol antmicroFerriteBeadsandChips:BLM15PD121SN1D
Connections:
- net labels removed: AVDD3V3_USB, GND, VCC_0V9, VCC_1V8, VCC_3V3
- wire segments 141 -> 0
Other:
- note removed: "MIPI&USB"
- note removed: "VDD3318_GMII"
- note removed: "VDD3318_SENSOR"
- note removed: "VIC 3V3 GPIO"
- note removed: "VIC LCD&RGMII"
- note removed: "VIC MIPI&USB"
