File: VIC7100-interfaces.sch (KiCad schematic (older format))
At the start: 38 parts

Commit message: Connected interfaces to VIC to visualise its ball locations (wip, mock purposes)
Parts:
- added C173, C174, C175, C183, C185, C186, C187, C189, C198, C199, C202: C_1u_0402, antmicro-footprints:0402-cap, symbol antmicroCapacitors0402:C_1u_0402
- added C176, C177, C178, C179, C180, C181, C188, C190, C191, C192, C193, C194, C195, C196, C197, C200, C201, C203, C204, C205, C206: C_100n_0201, antmicro-footprints:0201-res, symbol antmicroCapacitorsmisc:C_100n_0201
- added C182, C184: C_10u_0402, antmicro-footprints:0402-cap, symbol antmicroCapacitors0402:C_10u_0402
- added FB6: BLM15PD121SN1D, antmicro-footprints:0402-res, symbol antmicroFerriteBeadsandChips:BLM15PD121SN1D
- gave numbers to parts that had none: 34
Connections:
- net labels added: ETH_MDC, ETH_MDIO, RGMII_REF_CLK, RGMII_RXD0, RGMII_RXD1, RGMII_RXD2, RGMII_RXD3, RGMII_RX_CLK, RGMII_RX_DV, RGMII_TXD0, RGMII_TXD1, RGMII_TXD2, RGMII_TXD3, RGMII_TX_CLK, RGMII_TX_DV
- net labels removed: GMAC_GTXCLK, GMAC_MDC, GMAC_MDIO, GMAC_RXCLK, GMAC_RXD0, GMAC_RXD1, GMAC_RXD2, GMAC_RXD3, GMAC_RXDV, GMAC_TXD0, GMAC_TXD1, GMAC_TXD2, GMAC_TXD3
- wire segments 64 -> 218
Other:
- note added: "MIPI&USB"
- note added: "VDD3318_GMII"
- note added: "VDD3318_SENSOR"
- note added: "VIC 3V3 GPIO"
- note added: "VIC LCD&RGMII"
- note added: "VIC MIPI&USB"

Commit message: Updated interfaces, CPU and B2B connector connections
Connections:
- net labels added: RGMII_GTXCLK, RGMII_MDC, RGMII_MDIO, RGMII_RXCLK, RGMII_RXDV, RGMII_TXEN
- net labels removed: ETH_MDC, ETH_MDIO, GMAC_TXEN, RGMII_REF_CLK, RGMII_RX_CLK, RGMII_RX_DV, RGMII_TX_CLK, RGMII_TX_DV
- wire segments 218 -> 219
Other:
- note added: "not on B2B connector?"
Changed lines of the file:
@@
 $Descr A3 16535 11693
 encoding utf-8
-Sheet 9 11
+Sheet 9 10
 Title ""
 Date ""
@@
 NoConn ~ 5625 7375
 NoConn ~ 5625 7475
-Text GLabel 5625 5275 0    50   Input ~ 0
-GMAC_TXEN
+Text GLabel 5025 5275 0    50   Input ~ 0
+RGMII_TXEN
 Text GLabel 8700 1350 0    50   Input ~ 0
 VCC_0V9
@@
 Text Notes 11400 5800 0    118  ~ 24
 VIC MIPI&USB
-Text GLabel 5075 4900 0    50   Output ~ 0
-RGMII_REF_CLK
 Text GLabel 5025 6275 0    50   Output ~ 0
-RGMII_RX_CLK
+RGMII_RXCLK
 Text GLabel 5025 6875 0    50   Output ~ 0
 RGMII_RXD3
@@
 RGMII_RXD0
 Text GLabel 5050 5075 0    50   Input ~ 0
-RGMII_TX_CLK
+RGMII_GTXCLK
 Text GLabel 5025 5775 0    50   Input ~ 0
 RGMII_TXD3
@@
 Text GLabel 5025 5475 0    50   Input ~ 0
 RGMII_TXD0
-Text GLabel 5050 5175 0    50   Input ~ 0
-RGMII_TX_DV
 Text GLabel 5025 7675 0    50   BiDi ~ 0
-ETH_MDIO
+RGMII_MDIO
 Text GLabel 5025 7575 0    50   Input ~ 0
-ETH_MDC
+RGMII_MDC
 Text GLabel 5025 6375 0    50   Output ~ 0
-RGMII_RX_DV
+RGMII_RXDV
 Wire Wire Line
 	12925 6500 13250 6500
@@
 Wire Wire Line
 	5625 5075 5050 5075
+Wire Wire Line
+	5025 5275 5625 5275
+Text Notes 1600 6300 2    50   ~ 0
+not on B2B connector?
 $EndSCHEMATC

Commit message: Schematic cleanup, added logotypes
Connections:
- wire segments 219 -> 217
Other:
- note added: "TODO: connect resistors before VIC"
- note added: "VIC7100 interfaces"

Commit message: Marked BT, WiFi, DAC pins as NC, added ACK LED
Parts:
- added D?: KP-1608CGCK, antmicro-footprints:LED_0603, symbol antmicroLEDIndicationDiscrete:KP-1608CGCK
- added Q?: BSS138AKA, antmicro-footprints:SOT-23-3, symbol antmicroTransistorsFETsMOSFETsSingle:BSS138AKA
- added R?: R_1k_0402, antmicro-footprints:0402-res, symbol antmicroResistors0402:R_1k_0402
- added R?: R_33R_0402, antmicro-footprints:0402-res, symbol antmicroResistors0402:R_33R_0402
Connections:
- net labels removed: BT_RSTN, BT_UART_CTS, BT_UART_RTS, BT_UART_RXD, BT_UART_TXD, BT_WAKE, DAC_PWML, DAC_PWMR, WIFI_EN, WIFI_SDIO1_CLK, WIFI_SDIO1_CMD, WIFI_SDIO1_D0, WIFI_SDIO1_D1, WIFI_SDIO1_D2, WIFI_SDIO1_D3
- wire segments 217 -> 222
- no-connect marks 36 -> 51
Other:
- note added: "ACK LED"
- note added: "BT_RSTN"
- note added: "BT_UART_CTS"
- note added: "BT_UART_RTS"
- note added: "BT_UART_RXD"
- note added: "BT_UART_TXD"
- note added: "BT_WAKE"
- note added: "DAC_PWML"
- note added: "DAC_PWMR"
- note added: "TODO:\nadd on/off logic connection\nto PWR_OFF pin"
- note added: "WIFI_EN"
- note added: "WIFI_SDIO1_CLK"
- note added: "WIFI_SDIO1_CMD"
- note added: "WIFI_SDIO1_D0"
- note added: "WIFI_SDIO1_D1"
- note added: "WIFI_SDIO1_D2"
- note added: "WIFI_SDIO1_D3"
- note removed: "not on B2B connector?"
Changed lines of the file:
@@
 Text GLabel 2125 4075 0    50   Input ~ 0
 VDD2PEN
-Text GLabel 2125 4175 0    50   Input ~ 0
-WIFI_SDIO1_CMD
-Text GLabel 2125 4275 0    50   Input ~ 0
-WIFI_SDIO1_D1
-Text GLabel 2125 4375 0    50   Input ~ 0
-WIFI_SDIO1_D3
-Text GLabel 2125 4475 0    50   Input ~ 0
-BT_WAKE
-Text GLabel 2125 4575 0    50   Input ~ 0
-WIFI_SDIO1_CLK
-Text GLabel 2125 4675 0    50   Input ~ 0
-WIFI_SDIO1_D2
 Text GLabel 2125 4775 0    50   Input ~ 0
 LED
-Text GLabel 2125 4875 0    50   Input ~ 0
-WIFI_SDIO1_D0
 Text GLabel 2125 4975 0    50   Input ~ 0
 PWR_OFF
-Text GLabel 2125 5075 0    50   Input ~ 0
-BT_UART_CTS
-Text GLabel 2125 5175 0    50   Input ~ 0
-BT_UART_RXD
-Text GLabel 2125 5275 0    50   Input ~ 0
-BT_UART_TXD
-Text GLabel 2125 5375 0    50   Input ~ 0
-BT_UART_RTS
-Text GLabel 2125 5475 0    50   Input ~ 0
-WIFI_EN
-Text GLabel 2125 5575 0    50   Input ~ 0
-BT_RSTN
 Text GLabel 2125 5675 0    50   Input ~ 0
 SDIO0_D0
@@
 Text GLabel 2125 6875 0    50   Input ~ 0
 I2C0_SCL
-Text GLabel 2125 6975 0    50   Input ~ 0
-DAC_PWML
-Text GLabel 2125 7075 0    50   Input ~ 0
-DAC_PWMR
 Text GLabel 1325 7175 0    50   Input ~ 0
 HDMI_I2STX0
@@
 Wire Wire Line
 	5025 5275 5625 5275
-Text Notes 1600 6300 2    50   ~ 0
-not on B2B connector?
 $Bitmap
 Pos 1500 10693
@@
 Text Notes 4025 1175 0    50   ~ 0
 TODO: connect resistors before VIC
+Text Notes 1275 4200 0    50   ~ 0
+WIFI_SDIO1_CMD
+Text Notes 1275 4325 0    50   ~ 0
+WIFI_SDIO1_D1
+Text Notes 1275 4425 0    50   ~ 0
+WIFI_SDIO1_D3
+Text Notes 1275 4525 0    50   ~ 0
+BT_WAKE
+Text Notes 1275 4625 0    50   ~ 0
+WIFI_SDIO1_CLK
+Text Notes 1275 4725 0    50   ~ 0
+WIFI_SDIO1_D2
+Text Notes 1275 4925 0    50   ~ 0
+WIFI_SDIO1_D0
+Text Notes 1275 5125 0    50   ~ 0
+BT_UART_CTS
+Text Notes 1275 5225 0    50   ~ 0
+BT_UART_RXD
+Text Notes 1275 5325 0    50   ~ 0
+BT_UART_TXD
+Text Notes 1275 5425 0    50   ~ 0
+BT_UART_RTS
+Text Notes 1275 5525 0    50   ~ 0
+WIFI_EN
+Text Notes 1275 5625 0    50   ~ 0
+BT_RSTN
+NoConn ~ 2125 4175
+NoConn ~ 2125 4275
+NoConn ~ 2125 4375
+NoConn ~ 2125 4475
+NoConn ~ 2125 4575
+NoConn ~ 2125 4675
+NoConn ~ 2125 4875
+NoConn ~ 2125 5075
+NoConn ~ 2125 5175
+NoConn ~ 2125 5275
+NoConn ~ 2125 5375
+NoConn ~ 2125 5475
+NoConn ~ 2125 5575
+Text GLabel 8325 9750 0    50   Input ~ 0
+LED
+$Comp
+L antmicroResistors0402:R_1k_0402 R?
+U 1 1 630B1A75
+P 9200 8925
+F 0 "R?" V 9155 8995 60  0000 L CNN
+F 1 "R_1k_0402" H 9200 8775 60  0001 C CNN
+F 2 "antmicro-footprints:0402-res" H 9400 9125 60  0001 L CNN
+F 3 "" H 9200 8925 50  0001 C CNN
+F 4 "BOURNS" H 9400 9325 60  0001 L CNN "Manufacturer"
+F 5 "CR0402-FX-1001GLF" H 9400 9225 60  0001 L CNN "MPN"
+F 6 "1k" V 9253 8995 50  0000 L CNN "Val"
+	1    9200 8925
+	0    1    1    0
+$EndComp
+$Comp
+L antmicroLEDIndicationDiscrete:KP-1608CGCK D?
+U 1 1 630B453C
+P 9200 9350
+F 0 "D?" V 9097 9528 60  0000 L CNN
+F 1 "KP-1608CGCK" V 9203 9528 60  0000 L CNN
+F 2 "antmicro-footprints:LED_0603" H 9400 9550 60  0001 L CNN
+F 3 "http://www.farnell.com/datasheets/2045956.pdf" H 9400 9650 60  0001 L CNN
+F 4 "KP-1608CGCK" H 9400 9850 60  0001 L CNN "MPN"
+F 5 "KINGBRIGHT" H 9410 9970 60  0001 L CNN "Manufacturer"
+	1    9200 9350
+	0    1    1    0
+$EndComp
+Wire Wire Line
+	9200 9075 9200 9150
+Text GLabel 9200 8675 1    50   Input ~ 0
+VCC_3V3
+Wire Wire Line
+	9200 8675 9200 8775
+$Comp
+L antmicroTransistorsFETsMOSFETsSingle:BSS138AKA Q?
+U 1 1 631064ED
+P 9200 9650
+F 0 "Q?" H 9308 9703 60  0000 L CNN
+F 1 "BSS138AKA" H 9308 9597 60  0000 L CNN
+F 2 "antmicro-footprints:SOT-23-3" H 9400 9850 60  0001 L CNN
+F 3 "https://www.onsemi.com/pub/Collateral/BSS138-D.PDF" H 9400 9950 60  0001 L CNN
+F 4 "BSS138AKAR" H 9400 10150 60  0001 L CNN "MPN"
+F 5 "ON Semiconductor" H 9400 10750 60  0001 L CNN "Manufacturer"
+	1    9200 9650
+	1    0    0    -1
+$EndComp
+Wire Wire Line
+	9200 9850 9200 9950
+$Comp
+L power:GND #PWR?
+U 1 1 63136436
+P 9200 9950
+AR Path="/607683D6/63136436" Ref="#PWR?"  Part="1"
+AR Path="/60805CEC/63136436" Ref="#PWR?"  Part="1"
+F 0 "#PWR?" H 9200 9700 50  0001 C CNN
+F 1 "GND" H 9205 9777 50  0000 C CNN
+F 2 "" H 9200 9950 50  0001 C CNN
+F 3 "" H 9200 9950 50  0001 C CNN
+	1    9200 9950
+	1    0    0    -1
+$EndComp
+$Comp
+L antmicroResistors0402:R_33R_0402 R?
+U 1 1 63153957
+P 8650 9750
+F 0 "R?" H 8650 9963 60  0000 C CNN
+F 1 "R_33R_0402" H 8650 9600 60  0001 C CNN
+F 2 "antmicro-footprints:0402-res" H 8850 9950 60  0001 L CNN
+F 3 "" H 8650 9750 50  0001 C CNN
+F 4 "Vishay" H 8850 10150 60  0001 L CNN "Manufacturer"
+F 5 "CRCW040233R0FKED" H 8850 10050 60  0001 L CNN "MPN"
+F 6 "33R" H 8650 9865 50  0000 C CNN "Val"
+	1    8650 9750
+	1    0    0    -1
+$EndComp
+Wire Wire Line
+	8800 9750 8900 9750
+Wire Wire Line
+	8500 9750 8325 9750
+Text Notes 8825 8050 0    118  ~ 24
+ACK LED
+Text Notes 3250 4750 0    50   ~ 0
+TODO:\nadd on/off logic connection\nto PWR_OFF pin
+Text Notes 1325 6975 0    50   ~ 0
+DAC_PWML
+Text Notes 1325 7075 0    50   ~ 0
+DAC_PWMR
+NoConn ~ 2125 6975
+NoConn ~ 2125 7075
 $EndSCHEMATC

Commit message: Added I2C0 pullups, minor interfaces changes
Parts:
- added R117, R118: R_2k_0402, antmicro-footprints:0402-res, symbol antmicroResistors0402:R_2k_0402
- gave numbers to parts that had none: 4
Connections:
- net labels removed: USB_SSRXA1, USB_SSRXA2, USB_SSRXB1, USB_SSRXB2, USB_SSTXA1, USB_SSTXA2, USB_SSTXB1, USB_SSTXB2
- wire segments 222 -> 260
- no-connect marks 51 -> 59
Other:
- note added: "TBD: put PCIe interface here"
- note added: "USB_SSRXA1"
- note added: "USB_SSRXA2"
- note added: "USB_SSRXB1"
- note added: "USB_SSRXB2"
- note added: "USB_SSTXA1"
- note added: "USB_SSTXA2"
- note added: "USB_SSTXB1"
- note added: "USB_SSTXB2"
- note removed: "TODO: connect resistors before VIC"

Commit message: Added SDIO CD pulldown
Parts:
- added R?: R_10k_0402, antmicro-footprints:0402-res, symbol antmicroResistors0402:R_10k_0402
Connections:
- wire segments 260 -> 263
Changed lines of the file:
@@
 Text GLabel 2125 6175 0    50   Input ~ 0
 SDIO0_CLK
-Text GLabel 2125 6275 0    50   Input ~ 0
-SDIO0_CD
 Text GLabel 2125 6375 0    50   Input ~ 0
 CSI1_PWDN
@@
 Wire Wire Line
 	1325 6125 1325 6025
+Text GLabel 2125 6275 0    50   Input ~ 0
+SDIO0_CD
+Text GLabel 1700 9000 2    50   Input ~ 0
+SDIO0_CD
+$Comp
+L antmicroResistors0402:R_10k_0402 R?
+U 1 1 611FAF4E
+P 1400 9000
+F 0 "R?" H 1400 9305 60  0000 C CNN
+F 1 "R_10k_0402" H 1400 8850 60  0001 C CNN
+F 2 "antmicro-footprints:0402-res" H 1600 9200 60  0001 L CNN
+F 3 "" H 1400 9000 50  0001 C CNN
+F 4 "VISHAY" H 1600 9400 60  0001 L CNN "Manufacturer"
+F 5 "CRCW040210K0FKEDHP" H 1600 9300 60  0001 L CNN "MPN"
+F 6 "10k" H 1400 9207 50  0000 C CNN "Val"
+F 7 "DNP" H 1400 9116 50  0000 C CNN "Populate"
+	1    1400 9000
+	1    0    0    -1
+$EndComp
+Wire Wire Line
+	1550 9000 1700 9000
+Wire Wire Line
+	1250 9000 1025 9000
+Wire Wire Line
+	1025 9000 1025 9175
+$Comp
+L power:GND #PWR?
+U 1 1 6123BF63
+P 1025 9175
+AR Path="/607683D6/6123BF63" Ref="#PWR?"  Part="1"
+AR Path="/60805CEC/6123BF63" Ref="#PWR?"  Part="1"
+F 0 "#PWR?" H 1025 8925 50  0001 C CNN
+F 1 "GND" H 1030 9002 50  0000 C CNN
+F 2 "" H 1025 9175 50  0001 C CNN
+F 3 "" H 1025 9175 50  0001 C CNN
+	1    1025 9175
+	1    0    0    -1
+$EndComp
 $EndSCHEMATC

Commit message: Added local libraries
Parts:
- C173, C174, C175, C183, C185, C186, C187, C189, C198, C199, C202: footprint antmicro-footprints:0402-cap -> arv-som-footprints:0402-cap; symbol antmicroCapacitors0402:C_1u_0402 -> arv-som:C_1u_0402
- C176, C177, C178, C179, C180, C181, C188, C190, C191, C192, C193, C194, C195, C196, C197, C200, C201, C203, C204, C205, C206: footprint antmicro-footprints:0201-res -> arv-som-footprints:0201-res; symbol antmicroCapacitorsmisc:C_100n_0201 -> arv-som:C_100n_0201
- C182, C184: footprint antmicro-footprints:0402-cap -> arv-som-footprints:0402-cap; symbol antmicroCapacitors0402:C_10u_0402 -> arv-som:C_10u_0402
- D4: footprint antmicro-footprints:LED_0603 -> arv-som-footprints:LED_0603; symbol antmicroLEDIndicationDiscrete:KP-1608CGCK -> arv-som:KP-1608CGCK
- FB6: footprint antmicro-footprints:0402-res -> arv-som-footprints:0402-res; symbol antmicroFerriteBeadsandChips:BLM15PD121SN1D -> arv-som:BLM15PD121SN1D
- Q5: footprint antmicro-footprints:SOT-23-3 -> arv-som-footprints:SOT-23-3; symbol antmicroTransistorsFETsMOSFETsSingle:BSS138AKA -> arv-som:BSS138AKA
- R117, R118: footprint antmicro-footprints:0402-res -> arv-som-footprints:0402-res; symbol antmicroResistors0402:R_2k_0402 -> arv-som:R_2k_0402
- R119, R55, R56, R57, R58, R59: footprint antmicro-footprints:0402-res -> arv-som-footprints:0402-res; symbol antmicroResistors0402:R_33R_0402 -> arv-som:R_33R_0402
- R120: footprint antmicro-footprints:0402-res -> arv-som-footprints:0402-res; symbol antmicroResistors0402:R_1k_0402 -> arv-som:R_1k_0402
- R122: renamed from R?; footprint antmicro-footprints:0402-res -> arv-som-footprints:0402-res; symbol antmicroResistors0402:R_10k_0402 -> arv-som:R_10k_0402
- R60, R61, R62, R63, R64, R65, R66, R67, R68, R69, R70, R71, R72, R73, R74, R75, R76, R77, R78, R79, R80, R81, R82, R83, R84, R85, R86, R87: footprint antmicro-footprints:0201-res -> arv-som-footprints:0201-res; symbol antmicroResistorsmisc:R_33R_0201 -> arv-som:R_33R_0201
- U13: footprint antmicro-footprints:vic7100 -> arv-som-footprints:vic7100; symbol antmicroMicrocontrollers:VIC7100 -> arv-som:VIC7100
