File: interfaces.sch (KiCad schematic (older format))
At the start: 26 parts

Commit message: Connected interfaces to VIC to visualise its ball locations (wip, mock purposes)
Parts:
- gave numbers to parts that had none: 26

Commit message: Updated interfaces, CPU and B2B connector connections
Connections:
- net labels added: HDMI_12MHZ, HDMI_BCLK, HDMI_I2S_TX0, HDMI_INT, HDMI_LRCLK, I2C0_SCL, I2C0_SDA
- net labels removed: FNSH025_HDMI_12MHZ, FNSH026_HDMI_BCLK, FNSH027_HDMI_I2S_LRCLK, FNSH028_HDMI_I2S_TX0, FNSH032_HDMI_INT, FNSH061_I2C0_SDA, FNSH062_I2C0_SCL
Changed lines of the file:
@@
 $Descr A3 16535 11693
 encoding utf-8
-Sheet 4 11
+Sheet 4 10
 Title ""
 Date ""
@@
 	2775 6125 2350 6125
 Text GLabel 2350 6125 0    50   Input ~ 0
-FNSH026_HDMI_BCLK
+HDMI_BCLK
 NoConn ~ 2775 7025
 Wire Wire Line
 	2775 6925 2350 6925
 Text GLabel 2350 6925 0    50   Input ~ 0
-FNSH028_HDMI_I2S_TX0
+HDMI_I2S_TX0
 Wire Wire Line
 	2775 6825 2350 6825
 Text GLabel 2350 6825 0    50   Input ~ 0
-FNSH027_HDMI_I2S_LRCLK
+HDMI_LRCLK
 Wire Wire Line
 	2775 5925 2675 5925
@@
 	2775 7125 2350 7125
 Text GLabel 2350 7125 0    50   Input ~ 0
-FNSH025_HDMI_12MHZ
+HDMI_12MHZ
 NoConn ~ 2775 7225
 Wire Wire Line
@@
 $EndComp
 Text GLabel 4775 8525 2    50   Input ~ 0
-FNSH062_I2C0_SCL
+I2C0_SCL
 Text GLabel 4775 8625 2    50   Input ~ 0
-FNSH061_I2C0_SDA
+I2C0_SDA
 Wire Wire Line
 	5725 8475 5725 8925
@@
 VCC_3V3
 Text GLabel 4775 9125 2    50   Input ~ 0
-FNSH032_HDMI_INT
+HDMI_INT
 Wire Wire Line
 	4775 9725 4925 9725

Commit message: Schematic cleanup, added logotypes
Parts:
- removed C35: C_1u_0402, antmicro-footprints:0402-cap, symbol antmicroCapacitors0402:C_1u_0402
- removed C36: C_100n_0201, antmicro-footprints:0201-res, symbol antmicroCapacitorsmisc:C_100n_0201
- removed R18, R19, R20, R22, R23, R24: R_33R_0402, antmicro-footprints:0402-res, symbol antmicroResistors0402:R_33R_0402
- removed R21: R_4k7_0402, antmicro-footprints:0402-res, symbol antmicroResistors0402:R_4k7_0402
- removed U9: GD25LQ256DWIGR, antmicro-footprints:8-WSON-6x5, symbol antmicroMemory:GD25LQ256DWIGR
Connections:
- net labels removed: QSPI_CLK, QSPI_CS0_N, QSPI_D0, QSPI_D1, QSPI_D2, QSPI_D3
- wire segments 103 -> 85
Other:
- note added: "HDMI transmitter"
- note removed: "LCD to HDMI"
- note removed: "NOR Flash"
- note removed: "TODO: replace 33R with 0201 package"

Commit message: Added I2C0 pullups, minor interfaces changes
Parts:
- removed F1: 0ZCM0002FF2G, antmicro-footprints:0603-res, symbol antmicroFuses:0ZCM0002FF2G
- added FB7: BLM15PD121SN1D, antmicro-footprints:0402-res, symbol antmicroFerriteBeadsandChips:BLM15PD121SN1D
Connections:
- wire segments 85 -> 83
Changed lines of the file:
@@
 U 1 1 608F44D4
 P 9025 6125
-F 0 "R26" V 8980 6195 60  0000 L CNN
+F 0 "R26" H 8950 6225 60  0000 L CNN
 F 1 "R_1k_0402" H 9025 5975 60  0001 C CNN
 F 2 "antmicro-footprints:0402-res" H 9225 6325 60  0001 L CNN
@@
 F 4 "BOURNS" H 9225 6525 60  0001 L CNN "Manufacturer"
 F 5 "CR0402-FX-1001GLF" H 9225 6425 60  0001 L CNN "MPN"
-F 6 "1k" V 9078 6195 50  0000 L CNN "Val"
+F 6 "1k" H 8975 6125 50  0000 L CNN "Val"
 	1    9025 6125
 	0    1    1    0
@@
 U 1 1 608F47DE
 P 9275 6125
-F 0 "R27" V 9230 6195 60  0000 L CNN
+F 0 "R27" H 9200 6225 60  0000 L CNN
 F 1 "R_1k_0402" H 9275 5975 60  0001 C CNN
 F 2 "antmicro-footprints:0402-res" H 9475 6325 60  0001 L CNN
@@
 F 4 "BOURNS" H 9475 6525 60  0001 L CNN "Manufacturer"
 F 5 "CR0402-FX-1001GLF" H 9475 6425 60  0001 L CNN "MPN"
-F 6 "1k" V 9328 6195 50  0000 L CNN "Val"
+F 6 "1k" H 9225 6125 50  0000 L CNN "Val"
 	1    9275 6125
 	0    1    1    0
@@
 Wire Wire Line
 	9275 6625 9425 6625
-$Comp
-L antmicroFuses:0ZCM0002FF2G F1
-U 1 1 60918CF5
-P 9025 5675
-F 0 "F1" V 9071 5545 50  0000 R CNN
-F 1 "0ZCM0002FF2G" V 8980 5545 50  0000 R CNN
-F 2 "antmicro-footprints:0603-res" H 9075 5450 50  0001 C CNN
-F 3 "https://www.belfuse.com/resources/datasheets/circuitprotection/ds-cp-0zcm-series.pdf" H 9025 5525 50  0001 C CNN
-F 4 "0ZCM0002FF2G" H 9050 5375 50  0001 C CNN "MPN"
-F 5 "BEL FUSE" H 9075 5300 50  0001 C CNN "Manufacturer"
-	1    9025 5675
-	0    -1   -1   0
-$EndComp
-Text GLabel 9025 5425 1    50   Input ~ 0
+Text GLabel 9025 5500 1    50   Input ~ 0
 VCC_5V0
 Wire Wire Line
-	9025 5425 9025 5525
-Wire Wire Line
-	9025 5825 9025 5900
-Wire Wire Line
 	9025 5900 9275 5900
 Wire Wire Line
 	9275 5900 9275 5975
-Connection ~ 9025 5900
 Wire Wire Line
 	9025 5900 9025 5975
@@
 EndData
 $EndBitmap
+$Comp
+L antmicroFerriteBeadsandChips:BLM15PD121SN1D FB7
+U 1 1 60D6E8D3
+P 9025 5700
+F 0 "FB7" H 9025 5987 60  0000 C CNN
+F 1 "BLM15PD121SN1D" H 9025 5881 60  0000 C CNN
+F 2 "antmicro-footprints:0402-res" H 9225 5900 60  0001 L CNN
+F 3 "" H 9225 6000 60  0001 L CNN
+F 4 "BLM15PD121SN1D" H 9225 6200 60  0001 L CNN "MPN"
+F 5 "Murata" H 9225 6800 60  0001 L CNN "Manufacturer"
+	1    9025 5700
+	0    -1   -1   0
+$EndComp
+Connection ~ 9025 5900
 $EndSCHEMATC

Commit message: Added local libraries
Parts:
- C37, C39, C41, C43: footprint antmicro-footprints:0402-cap -> arv-som-footprints:0402-cap; symbol antmicroCapacitors0402:C_2u2_0402 -> arv-som:C_2u2_0402
- C38, C40, C42, C44: footprint antmicro-footprints:0201-res -> arv-som-footprints:0201-res; symbol antmicroCapacitorsmisc:C_100n_0201 -> arv-som:C_100n_0201
- D3: footprint antmicro-footprints:SOD-323F -> arv-som-footprints:SOD-323F; symbol antmicroDiodesRectifiersSingle:1N4148WS -> arv-som:1N4148WS
- FB1, FB7: footprint antmicro-footprints:0402-res -> arv-som-footprints:0402-res; symbol antmicroFerriteBeadsandChips:BLM15PD121SN1D -> arv-som:BLM15PD121SN1D
- R25: footprint antmicro-footprints:0402-res -> arv-som-footprints:0402-res; symbol antmicroResistors0402:R_10k_0402 -> arv-som:R_10k_0402
- R26, R27: footprint antmicro-footprints:0402-res -> arv-som-footprints:0402-res; symbol antmicroResistors0402:R_1k_0402 -> arv-som:R_1k_0402
- R28: footprint antmicro-footprints:0402-res -> arv-som-footprints:0402-res; symbol antmicroResistors0402:R_27k_0402 -> arv-som:R_27k_0402
- U10: footprint antmicro-footprints:QFN50P900X900X100-65N -> arv-som-footprints:QFN50P900X900X100-65N; symbol antmicroInterfaceControllers:TDA19988BHN_C1,557 -> arv-som:TDA19988BHN_C1,557
Changed lines of the file:
@@
 $EndDescr
 $Comp
-L antmicroInterfaceControllers:TDA19988BHN_C1,557 U10
+L arv-som:TDA19988BHN_C1,557 U10
 U 1 1 607A5735
 P 7075 5525
 F 0 "U10" H 7075 8192 50  0000 C CNN
 F 1 "TDA19988BHN_C1,557" H 7075 8101 50  0000 C CNN
-F 2 "antmicro-footprints:QFN50P900X900X100-65N" H 7075 5525 50  0001 L BNN
+F 2 "arv-som-footprints:QFN50P900X900X100-65N" H 7075 5525 50  0001 L BNN
 F 3 "" H 7075 5525 50  0001 L BNN
 F 4 "NXP Semiconductors" H 7075 5525 50  0001 L BNN "MANUFACTURER"
@@
 Connection ~ 5975 3725
 $Comp
-L power:GND #PWR0137
+L arv-som:GND #PWR0137
 U 1 1 607C5297
 P 5975 8125
@@
 Connection ~ 8375 3425
 $Comp
-L antmicroCapacitors0402:C_2u2_0402 C37
+L arv-som:C_2u2_0402 C37
 U 1 1 607E47D0
 P 9125 3000
 F 0 "C37" H 9240 3045 60  0000 L CNN
 F 1 "C_2u2_0402" H 9125 2850 60  0001 C CNN
-F 2 "antmicro-footprints:0402-cap" H 9325 3200 60  0001 L CNN
+F 2 "arv-som-footprints:0402-cap" H 9325 3200 60  0001 L CNN
 F 3 "" H 9125 3000 50  0001 C CNN
 F 4 "TDK" H 9325 3400 60  0001 L CNN "Manufacturer"
@@
 $EndComp
 $Comp
-L antmicroCapacitors0402:C_2u2_0402 C39
+L arv-som:C_2u2_0402 C39
 U 1 1 607E4C5F
 P 9900 3000
 F 0 "C39" H 10015 3045 60  0000 L CNN
 F 1 "C_2u2_0402" H 9900 2850 60  0001 C CNN
-F 2 "antmicro-footprints:0402-cap" H 10100 3200 60  0001 L CNN
+F 2 "arv-som-footprints:0402-cap" H 10100 3200 60  0001 L CNN
 F 3 "" H 9900 3000 50  0001 C CNN
 F 4 "TDK" H 10100 3400 60  0001 L CNN "Manufacturer"
@@
 HDMI_1V8
 $Comp
-L power:GND #PWR0138
+L arv-som:GND #PWR0138
 U 1 1 607E87FB
 P 9125 3150
@@
 HDMI_1V8
 $Comp
-L power:GND #PWR0139
+L arv-som:GND #PWR0139
 U 1 1 607EFCC2
 P 9900 3150
@@
 $EndComp
 $Comp
-L antmicroCapacitors0402:C_2u2_0402 C41
+L arv-som:C_2u2_0402 C41
 U 1 1 607F1ECB
 P 10625 3000
 F 0 "C41" H 10740 3045 60  0000 L CNN
 F 1 "C_2u2_0402" H 10625 2850 60  0001 C CNN
-F 2 "antmicro-footprints:0402-cap" H 10825 3200 60  0001 L CNN
+F 2 "arv-som-footprints:0402-cap" H 10825 3200 60  0001 L CNN
 F 3 "" H 10625 3000 50  0001 C CNN
 F 4 "TDK" H 10825 3400 60  0001 L CNN "Manufacturer"
@@
 HDMI_1V8
 $Comp
-L power:GND #PWR0140
+L arv-som:GND #PWR0140
 U 1 1 607F1ED2
 P 10625 3150
@@
 $EndComp
 $Comp
-L antmicroCapacitors0402:C_2u2_0402 C43
+L arv-som:C_2u2_0402 C43
 U 1 1 607F4B71
 P 11375 3000
 F 0 "C43" H 11490 3045 60  0000 L CNN
 F 1 "C_2u2_0402" H 11375 2850 60  0001 C CNN
-F 2 "antmicro-footprints:0402-cap" H 11575 3200 60  0001 L CNN
+F 2 "arv-som-footprints:0402-cap" H 11575 3200 60  0001 L CNN
 F 3 "" H 11375 3000 50  0001 C CNN
 F 4 "TDK" H 11575 3400 60  0001 L CNN "Manufacturer"
@@
 HDMI_1V8
 $Comp
-L power:GND #PWR0141
+L arv-som:GND #PWR0141
 U 1 1 607F4B78
 P 11375 3150
@@
 $EndComp
 $Comp
-L antmicroCapacitorsmisc:C_100n_0201 C38
+L arv-som:C_100n_0201 C38
 U 1 1 607F7307
 P 9500 3000
 F 0 "C38" H 9615 3045 60  0000 L CNN
 F 1 "C_100n_0201" H 9500 2850 60  0001 C CNN
-F 2 "antmicro-footprints:0201-res" H 9700 3200 60  0001 L CNN
+F 2 "arv-som-footprints:0201-res" H 9700 3200 60  0001 L CNN
 F 3 "" H 9500 3000 50  0001 C CNN
 F 4 "YAGEO" H 9700 3400 60  0001 L CNN "Manufacturer"
@@
 HDMI_1V8
 $Comp
-L power:GND #PWR0142
+L arv-som:GND #PWR0142
 U 1 1 607F77A7
 P 9500 3150
@@
 $EndComp
 $Comp
-L antmicroCapacitorsmisc:C_100n_0201 C40
+L arv-som:C_100n_0201 C40
 U 1 1 607F8E18
 P 10275 3000
 F 0 "C40" H 10390 3045 60  0000 L CNN
 F 1 "C_100n_0201" H 10275 2850 60  0001 C CNN
-F 2 "antmicro-footprints:0201-res" H 10475 3200 60  0001 L CNN
+F 2 "arv-som-footprints:0201-res" H 10475 3200 60  0001 L CNN
 F 3 "" H 10275 3000 50  0001 C CNN
 F 4 "YAGEO" H 10475 3400 60  0001 L CNN "Manufacturer"
@@
 HDMI_1V8
 $Comp
-L power:GND #PWR0143
+L arv-som:GND #PWR0143
 U 1 1 607F8E1F
 P 10275 3150
@@
 $EndComp
 $Comp
-L antmicroCapacitorsmisc:C_100n_0201 C42
+L arv-som:C_100n_0201 C42
 U 1 1 607FB340
 P 11000 3000
 F 0 "C42" H 11115 3045 60  0000 L CNN
 F 1 "C_100n_0201" H 11000 2850 60  0001 C CNN
-F 2 "antmicro-footprints:0201-res" H 11200 3200 60  0001 L CNN
+F 2 "arv-som-footprints:0201-res" H 11200 3200 60  0001 L CNN
 F 3 "" H 11000 3000 50  0001 C CNN
 F 4 "YAGEO" H 11200 3400 60  0001 L CNN "Manufacturer"
@@
 HDMI_1V8
 $Comp
-L power:GND #PWR0144
+L arv-som:GND #PWR0144
 U 1 1 607FB347
 P 11000 3150
@@
 $EndComp
 $Comp
-L antmicroCapacitorsmisc:C_100n_0201 C44
+L arv-som:C_100n_0201 C44
 U 1 1 607FD800
 P 11750 3000
 F 0 "C44" H 11865 3045 60  0000 L CNN
 F 1 "C_100n_0201" H 11750 2850 60  0001 C CNN
-F 2 "antmicro-footprints:0201-res" H 11950 3200 60  0001 L CNN
+F 2 "arv-som-footprints:0201-res" H 11950 3200 60  0001 L CNN
 F 3 "" H 11750 3000 50  0001 C CNN
 F 4 "YAGEO" H 11950 3400 60  0001 L CNN "Manufacturer"
@@
 HDMI_1V8
 $Comp
-L power:GND #PWR0145
+L arv-som:GND #PWR0145
 U 1 1 607FD807
 P 11750 3150
@@
 TODO: 2u2 with 0201 package
 $Comp
-L antmicroFerriteBeadsandChips:BLM15PD121SN1D FB1
+L arv-som:BLM15PD121SN1D FB1
 U 1 1 6086D39A
 P 11325 2175
 F 0 "FB1" H 11325 2462 60  0000 C CNN
 F 1 "BLM15PD121SN1D" H 11325 2356 60  0000 C CNN
-F 2 "antmicro-footprints:0402-res" H 11525 2375 60  0001 L CNN
+F 2 "arv-som-footprints:0402-res" H 11525 2375 60  0001 L CNN
 F 3 "" H 11525 2475 60  0001 L CNN
 F 4 "BLM15PD121SN1D" H 11525 2675 60  0001 L CNN "MPN"
@@
 	8550 3725 8650 3725
 $Comp
-L antmicroResistors0402:R_10k_0402 R25
+L arv-som:R_10k_0402 R25
 U 1 1 608924F4
 P 8800 3725
 F 0 "R25" H 8800 3938 60  0000 C CNN
 F 1 "R_10k_0402" H 8800 3575 60  0001 C CNN
-F 2 "antmicro-footprints:0402-res" H 9000 3925 60  0001 L CNN
+F 2 "arv-som-footprints:0402-res" H 9000 3925 60  0001 L CNN
 F 3 "" H 8800 3725 50  0001 C CNN
 F 4 "VISHAY" H 9000 4125 60  0001 L CNN "Manufacturer"
@@
 $EndComp
 $Comp
-L power:GND #PWR0146
+L arv-som:GND #PWR0146
 U 1 1 60893600
 P 9050 3725
@@
 HDMI_DSDA
 $Comp
-L antmicroResistors0402:R_1k_0402 R26
+L arv-som:R_1k_0402 R26
 U 1 1 608F44D4
 P 9025 6125
 F 0 "R26" H 8950 6225 60  0000 L CNN
 F 1 "R_1k_0402" H 9025 5975 60  0001 C CNN
-F 2 "antmicro-footprints:0402-res" H 9225 6325 60  0001 L CNN
+F 2 "arv-som-footprints:0402-res" H 9225 6325 60  0001 L CNN
 F 3 "" H 9025 6125 50  0001 C CNN
 F 4 "BOURNS" H 9225 6525 60  0001 L CNN "Manufacturer"
@@
 $EndComp
 $Comp
-L antmicroResistors0402:R_1k_0402 R27
+L arv-som:R_1k_0402 R27
 U 1 1 608F47DE
 P 9275 6125
 F 0 "R27" H 9200 6225 60  0000 L CNN
 F 1 "R_1k_0402" H 9275 5975 60  0001 C CNN
-F 2 "antmicro-footprints:0402-res" H 9475 6325 60  0001 L CNN
+F 2 "arv-som-footprints:0402-res" H 9475 6325 60  0001 L CNN
 F 3 "" H 9275 6125 50  0001 C CNN
 F 4 "BOURNS" H 9475 6525 60  0001 L CNN "Manufacturer"
@@
 HDMI_HPD
 $Comp
-L antmicroDiodesRectifiersSingle:1N4148WS D3
+L arv-som:1N4148WS D3
 U 1 1 60934FA2
 P 9225 6950
 F 0 "D3" H 9025 6900 60  0000 C CNN
 F 1 "1N4148WS" H 9575 6900 60  0000 C CNN
-F 2 "antmicro-footprints:SOD-323F" H 9425 7150 60  0001 L CNN
+F 2 "arv-som-footprints:SOD-323F" H 9425 7150 60  0001 L CNN
 F 3 "https://www.onsemi.com/pub/Collateral/1N914BWS-D.pdf" H 9425 7250 60  0001 L CNN
 F 4 "1N4148WS" H 9425 7450 60  0001 L CNN "MPN"
@@
 	8950 7125 9425 7125
 $Comp
-L antmicroResistors0402:R_27k_0402 R28
+L arv-som:R_27k_0402 R28
 U 1 1 6093E329
 P 9700 6950
 F 0 "R28" H 9700 7050 60  0000 C CNN
 F 1 "R_27k_0402" H 9700 6800 60  0001 C CNN
-F 2 "antmicro-footprints:0402-res" H 9900 7150 60  0001 L CNN
+F 2 "arv-som-footprints:0402-res" H 9900 7150 60  0001 L CNN
 F 3 "" H 9700 6950 50  0001 C CNN
 F 4 "PANASONIC_ELECTRONIC_COMPONENTS" H 9900 7350 60  0001 L CNN "Manufacturer"
@@
 	8225 7825 8225 7925
 $Comp
-L power:GND #PWR0147
+L arv-som:GND #PWR0147
 U 1 1 6095A132
 P 8225 8125
@@
 $EndBitmap
 $Comp
-L antmicroFerriteBeadsandChips:BLM15PD121SN1D FB7
+L arv-som:BLM15PD121SN1D FB7
 U 1 1 60D6E8D3
 P 9025 5700
 F 0 "FB7" H 9025 5987 60  0000 C CNN
 F 1 "BLM15PD121SN1D" H 9025 5881 60  0000 C CNN
-F 2 "antmicro-footprints:0402-res" H 9225 5900 60  0001 L CNN
+F 2 "arv-som-footprints:0402-res" H 9225 5900 60  0001 L CNN
 F 3 "" H 9225 6000 60  0001 L CNN
 F 4 "BLM15PD121SN1D" H 9225 6200 60  0001 L CNN "MPN"
