File: B2B-connectors.sch (KiCad schematic (older format))
At the start: 2 parts

Commit message: Updated B2B connectors sheet
Parts:
- removed J? (x2): QSE-020-01-F-D, antmicro-footprints:QSE-020-01-XXX-D-A, symbol antmicroRectangularConnectorsHeadersFemalePins:QSE-020-01-F-D
- added J? (x2): DF40C-100DS-0.4V(51), antmicro-footprints:DF40C-100DS-0.4V_51_, symbol antmicroRectangularConnectorsHeadersMalePins:DF40C-100DS-0.4V(51)
Connections:
- net labels added: 1V8_OUT, 3V3_OUT, 5V0_IN, AIN0, AIN1, BT_nDis, CAM0_C_N, CAM0_C_P, CAM0_D0_N, CAM0_D0_P, CAM0_D1_N, CAM0_D1_P, CAM1_C_N, CAM1_C_P, CAM1_D0_N, CAM1_D0_P, CAM1_D1_N, CAM1_D1_P, CAM1_D2_N, CAM1_D2_P, CAM1_D3_N, CAM1_D3_P, CAM_GPIO, DSI0_C_N, DSI0_C_P, DSI0_D0_N, DSI0_D0_P, DSI0_D1_N, DSI0_D1_P, DSI1_C_N, DSI1_C_P, DSI1_D0_N, DSI1_D0_P, DSI1_D1_N, DSI1_D1_P, DSI1_D3_N, DSI1_D3_P, DSI2_D1_N, DSI2_D1_P, EEPROM_nWP, ETH_LEDG, ETH_LEDY, ETH_nLED1, GLOBAL_EN, GPIO10, GPIO11, GPIO12, GPIO13, GPIO14, GPIO15, GPIO16, GPIO17, GPIO19, GPIO2, GPIO20, GPIO21, GPIO22, GPIO23, GPIO27, GPIO3, GPIO4, GPIO5, GPIO6, GPIO9, GPIO_VREF, ID_SC, ID_SD, PCIE_CLK_N, PCIE_CLK_P, PCIE_CLK_nREQ, PCIE_RX_N, PCIE_RX_P, PCIE_TX_N, PCIE_TX_P, PI_nLED_ACT, PSCIE_nRST, RESERVED, RUN_PG, SD_CLK, SD_CMD, SD_DAT0, SD_DAT1, SD_DAT2, SD_DAT3, SD_DAT4, SD_DAT5, SD_DAT7, SD_PWR_ON, SD_VDD_OVRD, SYNC_IN, SYNC_OUT, TRD0_N, TRD0_P, TRD1_N, TRD1_P, TRD2_N, TRD2_P, TRD3_N, TRD3_P, TV_OUT, USB2_N, USB2_P, USBOTG_ID, WL_nDis, nEXTRST, nPWR_LED, nRPIBOOT
- net labels removed: 3V3_RPi, 3V3_SSD, Adapter_RXD, Adapter_TXD, Adapter_USB_N, Adapter_USB_P, VCC5V0
- wire segments 108 -> 251
Other:
- note added: "Ethernet_nLED2"
- note added: "Ethernet_nLED3"
- note added: "Pi_nLED_Activity"
- note added: "RPi_RXD"
- note added: "RPi_TXD"
- note removed: "QSE connector current rating:\n2A per pin (2 pins powered)"
- note removed: "TODO: replace with QTE-020-01-F-D"

Commit message: Changed B2B connectors to headers
Parts:
- removed J? (x2): DF40C-100DS-0.4V(51), antmicro-footprints:DF40C-100DS-0.4V_51_, symbol antmicroRectangularConnectorsHeadersMalePins:DF40C-100DS-0.4V(51)
- added J? (x2): DF40C-100DP-0.4V(51), antmicro-footprints:HRS_DF40C-100DP-0.4V(51), symbol antmicroRectangularConnectorsHeadersMalePins:DF40C-100DP-0.4V(51)
Connections:
- wire segments 251 -> 247
Changed lines of the file:
@@
 $Descr A3 16535 11693
 encoding utf-8
-Sheet 12 12
+Sheet 11 11
 Title ""
 Date ""
@@
 GPIO15
 $Comp
-L antmicroRectangularConnectorsHeadersMalePins:DF40C-100DS-0.4V(51) J?
-U 1 1 60803D5D
-P 4300 5000
-F 0 "J?" H 4300 7667 50  0000 C CNN
-F 1 "DF40C-100DS-0.4V(51)" H 4300 7576 50  0000 C CNN
-F 2 "antmicro-footprints:DF40C-100DS-0.4V_51_" H 4300 5000 50  0001 L BNN
-F 3 "" H 4300 5000 50  0001 L BNN
-F 4 "HRS" H 4300 5000 50  0001 L BNN "Manufacturer"
-	1    4300 5000
-	-1   0    0    -1
-$EndComp
-Connection ~ 3800 6700
-Connection ~ 3800 6900
-$Comp
-L antmicroRectangularConnectorsHeadersMalePins:DF40C-100DS-0.4V(51) J?
-U 1 1 60807468
-P 8300 5000
-F 0 "J?" H 8300 7667 50  0000 C CNN
-F 1 "DF40C-100DS-0.4V(51)" H 8300 7576 50  0000 C CNN
-F 2 "antmicro-footprints:DF40C-100DS-0.4V_51_" H 8300 5000 50  0001 L BNN
-F 3 "" H 8300 5000 50  0001 L BNN
-F 4 "HRS" H 8300 5000 50  0001 L BNN "Manufacturer"
-	1    8300 5000
-	-1   0    0    -1
-$EndComp
-$Comp
 L power:GND #PWR?
 U 1 1 6083430C
@@
 Text GLabel 5250 6400 2    50   Input ~ 0
 5V0_IN
-Connection ~ 4800 6400
-Connection ~ 4800 6500
-Wire Wire Line
-	4800 6500 4800 6400
-Connection ~ 4800 6600
-Wire Wire Line
-	4800 6600 4800 6500
-Wire Wire Line
-	4800 6600 4800 6700
-Wire Wire Line
-	4800 6700 4800 6800
-Connection ~ 4800 6700
-Connection ~ 4800 6800
-Wire Wire Line
-	4800 6800 4800 6900
 Wire Wire Line
 	4800 7200 5250 7200
@@
 Text GLabel 7350 2800 0    50   Input ~ 0
 RESERVED
+$Comp
+L antmicroRectangularConnectorsHeadersMalePins:DF40C-100DP-0.4V(51) J?
+U 1 1 60FEF31E
+P 4300 5000
+F 0 "J?" H 4300 7757 50  0000 C CNN
+F 1 "DF40C-100DP-0.4V(51)" H 4300 7666 50  0000 C CNN
+F 2 "antmicro-footprints:HRS_DF40C-100DP-0.4V(51)" H 4300 5000 50  0001 L BNN
+F 3 "" H 4300 5000 50  0001 L BNN
+F 4 "HRS" H 4300 5000 50  0001 L BNN "Manufacturer"
+F 5 "DF40C-100DP-0.4V(51)" H 4300 7575 50  0000 C CNN "MPN"
+	1    4300 5000
+	-1   0    0    -1
+$EndComp
+Wire Wire Line
+	4800 6800 4800 6900
+Connection ~ 3800 6700
+Connection ~ 3800 6900
+$Comp
+L antmicroRectangularConnectorsHeadersMalePins:DF40C-100DP-0.4V(51) J?
+U 1 1 60FFB551
+P 8300 5000
+F 0 "J?" H 8300 7757 50  0000 C CNN
+F 1 "DF40C-100DP-0.4V(51)" H 8300 7666 50  0000 C CNN
+F 2 "antmicro-footprints:HRS_DF40C-100DP-0.4V(51)" H 8300 5000 50  0001 L BNN
+F 3 "" H 8300 5000 50  0001 L BNN
+F 4 "HRS" H 8300 5000 50  0001 L BNN "Manufacturer"
+F 5 "DF40C-100DP-0.4V(51)" H 8300 7575 50  0000 C CNN "MPN"
+	1    8300 5000
+	-1   0    0    -1
+$EndComp
 $EndSCHEMATC

Commit message: Connected interfaces to VIC to visualise its ball locations (wip, mock purposes)
Parts:
- gave numbers to parts that had none: 2
Connections:
- net labels added: CDTX_DSI_D0_N, CDTX_DSI_D0_P, CDTX_DSI_D1_N, CDTX_DSI_D1_P, CDTX_DSI_D2_N, CDTX_DSI_D2_P, CDTX_DSI_D3_N, CDTX_DSI_D3_P, CDTX_DSI_D4_N, CDTX_DSI_D4_P, CSI0_PWDN, CSI1RX_CLK_N, CSI1RX_CLK_P, CSI1RX_D0_N, CSI1RX_D0_P, CSI1RX_D1_N, CSI1RX_D1_P, CSI1_PWDN, CSI2RX_CLK_N, CSI2RX_CLK_P, CSI2RX_D0_N, CSI2RX_D0_P, CSI2RX_D1_N, CSI2RX_D1_P, ETH0_N, ETH0_P, ETH1_N, ETH1_P, ETH2_N, ETH2_P, ETH3_N, ETH3_P, ETH_LED1, ETH_LED2, HDMI_CEC, HDMI_DSCL, HDMI_DSDA, HDMI_HPD, HDMI_TX0_N, HDMI_TX0_P, HDMI_TX1_N, HDMI_TX1_P, HDMI_TX2_N, HDMI_TX2_P, HDMI_TXC_N, HDMI_TXC_P, I2C0_SCL, I2C0_SDA, I2C2_SCL, I2C2_SDA, RPI_GPIO10, RPI_GPIO11, RPI_GPIO12, RPI_GPIO13, RPI_GPIO14, RPI_GPIO15, RPI_GPIO16, RPI_GPIO17, RPI_GPIO18, RPI_GPIO19, RPI_GPIO2, RPI_GPIO20, RPI_GPIO21, RPI_GPIO22, RPI_GPIO23, RPI_GPIO24, RPI_GPIO25, RPI_GPIO26, RPI_GPIO27, RPI_GPIO3, RPI_GPIO4, RPI_GPIO5, RPI_GPIO6, RPI_GPIO7, RPI_GPIO8, RPI_GPIO9, RPI_ID_SC, RPI_ID_SD, SDIO0_CD, SDIO0_CLK, SDIO0_CMD, SDIO0_D0, SDIO0_D1, SDIO0_D2, SDIO0_D3, USBDM_N, USBDP_P
- net labels removed: CAM0_C_N, CAM0_C_P, CAM0_D0_N, CAM0_D0_P, CAM0_D1_N, CAM0_D1_P, CAM1_C_N, CAM1_C_P, CAM1_D0_N, CAM1_D0_P, CAM1_D1_N, CAM1_D1_P, ETH_LEDG, ETH_LEDY, GPIO10, GPIO11, GPIO12, GPIO13, GPIO14, GPIO15, GPIO16, GPIO17, GPIO18, GPIO19, GPIO2, GPIO20, GPIO21, GPIO22, GPIO23, GPIO24, GPIO25, GPIO26, GPIO27, GPIO3, GPIO4, GPIO5, GPIO6, GPIO7, GPIO8, GPIO9, HDMI0_CEC, HDMI0_CK_N, HDMI0_CK_P, HDMI0_D0_N, HDMI0_D0_P, HDMI0_D1_N, HDMI0_D1_P, HDMI0_D2_N, HDMI0_D2_P, HDMI0_HOTPLUG, HDMI0_SCL, HDMI0_SDA, ID_SC, ID_SD, SCL0, SDA0, SD_CLK, SD_CMD, SD_DAT0, SD_DAT1, SD_DAT3, TRD0_N, TRD0_P, TRD1_N, TRD1_P, TRD2_N, TRD2_P, TRD3_N, TRD3_P, USB2_N, USB2_P
- wire segments 247 -> 251

Commit message: Updated interfaces, CPU and B2B connector connections
Connections:
- net labels removed: DSI0_C_N, DSI0_C_P, DSI0_D0_N, DSI0_D0_P, DSI0_D1_N, DSI0_D1_P, ETH_nLED1, I2C2_SCL, I2C2_SDA, SYNC_IN, SYNC_OUT
Other:
- note added: "Analog inputs of CM4's PMIC\n(Type C power connector)"
- note added: "DSI0_C_N"
- note added: "DSI0_C_P"
- note added: "Drive low to power off CM4"
- note added: "ETH_nLED1"
- note added: "LED replicating status LED from RPi4B"
- note added: "Low: resets CM4\nOutput: signals Power good (10k pullup)"
- note added: "Power On LED output (AL), needs to be buffered"
- note added: "SDCARD/eMMC \navailable only on CM4Lite"
- note added: "SD_CLK"
- note added: "SD_CMD"
- note added: "SD_DAT0"
- note added: "SD_DAT1"
- note added: "SD_DAT2"
- note added: "SD_DAT3"
- note added: "SYNC_IN"
- note added: "SYNC_OUT"
- note added: "Signals provided by CM4's PHY (BCM54210PE)"
- note added: "TBD:"
- note added: "TBD: connect to any free GPIO?"
- note added: "TBD: connect to any free GPIO? (float if not used)"
- note added: "Write protection TBD"
- note added: "force SD/eMMC interface to 1.8V, otherwise NC"
- note removed: "Pi_nLED_Activity"

Commit message: Schematic cleanup, added logotypes
Connections:
- net labels removed: CDTX_DSI_D3_N, CDTX_DSI_D3_P, CDTX_DSI_D4_N, CDTX_DSI_D4_P, CSI0_PWDN, CSI1_PWDN, SDIO0_CD
Other:
- note added: "B2B connectors"
- note added: "Signal from VIC to be connected:\nSDIO0_CD?"
- note added: "Signals from VIC to be connected:\nCDTX_DSI_D4_N\nCDTX_DSI_D4_P\nCDTX_DSI_D3_N\nCDTX_DSI_D3_P"
- note added: "Signals from VIC to be connected:\nCSI1_PWDN\nCSI0_PWDN"
- note removed: "TBD:"

Commit message: B2B updated
Connections:
- net labels added: CDTX_DSI_D3_N, CDTX_DSI_D3_P, CDTX_DSI_D4_N, CDTX_DSI_D4_P, CSI0_PWDN, CTL5, DSI0_C_N, DSI0_C_P, I2C2_SCL, I2C2_SDA, LED, SD_DAT6, SYNC_IN, SYNC_OUT, VCC_1V8, VCC_3V3
- net labels removed: 1V8_OUT, 3V3_OUT, CAM_GPIO, DSI1_C_N, DSI1_C_P, DSI1_D3_N, DSI1_D3_P, DSI2_D1_N, DSI2_D1_P, I2C0_SCL, I2C0_SDA, PI_nLED_ACT, RUN_PG, SD_DAT2
Other:
- note added: "BCM54210PE PHY \nspecific"
- note added: "Blue annotations: CM pin reference"
- note added: "CAM_GPIO"
- note added: "DSI1_C_N"
- note added: "DSI1_C_P"
- note added: "DSI1_D0_N"
- note added: "DSI1_D0_P"
- note added: "DSI1_D1_N"
- note added: "DSI1_D1_P"
- note added: "DSI1_D2_N"
- note added: "DSI1_D2_P"
- note added: "DSI1_D3_N"
- note added: "DSI1_D3_P"
- note added: "Drive low to power off"
- note added: "ETHERNET_nLED1"
- note added: "Note: signals in cursive are NOT mapped on the SoM"
- note added: "RUN_PG"
- note added: "Uart_RXD"
- note added: "Uart_TXD"
- note added: "Write protection"
- note added: "force SD if to 1.8V\n"
- note added: "nLED_ACT"
- note removed: "Analog inputs of CM4's PMIC\n(Type C power connector)"
- note removed: "Drive low to power off CM4"
- note removed: "ETH_nLED1"
- note removed: "LED replicating status LED from RPi4B"
- note removed: "Low: resets CM4\nOutput: signals Power good (10k pullup)"
- note removed: "RPi_RXD"
- note removed: "RPi_TXD"
- note removed: "SDCARD/eMMC \navailable only on CM4Lite"
- note removed: "SYNC_IN"
- note removed: "SYNC_OUT"
- note removed: "Signal from VIC to be connected:\nSDIO0_CD?"
- note removed: "Signals from VIC to be connected:\nCDTX_DSI_D4_N\nCDTX_DSI_D4_P\nCDTX_DSI_D3_N\nCDTX_DSI_D3_P"
- note removed: "Signals from VIC to be connected:\nCSI1_PWDN\nCSI0_PWDN"
- note removed: "Signals provided by CM4's PHY (BCM54210PE)"
- note removed: "TBD: connect to any free GPIO?"
- note removed: "Write protection TBD"
- note removed: "force SD/eMMC interface to 1.8V, otherwise NC"

Commit message: Added local libraries
Parts:
- J3, J4: footprint antmicro-footprints:HRS_DF40C-100DP-0.4V(51) -> arv-som-footprints:HRS_DF40C-100DP-0.4V(51); symbol antmicroRectangularConnectorsHeadersMalePins:DF40C-100DP-0.4V(51) -> arv-som:DF40C-100DP-0.4V(51)
Changed lines of the file:
@@
 GPIO_VREF
 $Comp
-L power:GND #PWR0224
+L arv-som:GND #PWR0224
 U 1 1 6083430C
 P 3700 7650
@@
 $EndComp
 $Comp
-L power:GND #PWR0225
+L arv-som:GND #PWR0225
 U 1 1 60834719
 P 4900 7650
@@
 $EndComp
 $Comp
-L power:GND #PWR0226
+L arv-som:GND #PWR0226
 U 1 1 608363DA
 P 11075 7625
@@
 $EndComp
 $Comp
-L power:GND #PWR0227
+L arv-som:GND #PWR0227
 U 1 1 6083A5F9
 P 12325 7625
@@
 RESERVED
 $Comp
-L antmicroRectangularConnectorsHeadersMalePins:DF40C-100DP-0.4V(51) J3
+L arv-som:DF40C-100DP-0.4V(51) J3
 U 1 1 60FEF31E
 P 4300 4800
 F 0 "J3" H 4300 7557 50  0000 C CNN
 F 1 "DF40C-100DP-0.4V(51)" H 4300 7466 50  0000 C CNN
-F 2 "antmicro-footprints:HRS_DF40C-100DP-0.4V(51)" H 4300 4800 50  0001 L BNN
+F 2 "arv-som-footprints:HRS_DF40C-100DP-0.4V(51)" H 4300 4800 50  0001 L BNN
 F 3 "" H 4300 4800 50  0001 L BNN
 F 4 "HRS" H 4300 4800 50  0001 L BNN "Manufacturer"
@@
 Connection ~ 3800 6700
 $Comp
-L antmicroRectangularConnectorsHeadersMalePins:DF40C-100DP-0.4V(51) J4
+L arv-som:DF40C-100DP-0.4V(51) J4
 U 1 1 60FFB551
 P 11725 4725
 F 0 "J4" H 11725 7482 50  0000 C CNN
 F 1 "DF40C-100DP-0.4V(51)" H 11725 7391 50  0000 C CNN
-F 2 "antmicro-footprints:HRS_DF40C-100DP-0.4V(51)" H 11725 4725 50  0001 L BNN
+F 2 "arv-som-footprints:HRS_DF40C-100DP-0.4V(51)" H 11725 4725 50  0001 L BNN
 F 3 "" H 11725 4725 50  0001 L BNN
 F 4 "HRS" H 11725 4725 50  0001 L BNN "Manufacturer"

Commit message: Update naming convention
Parts:
- J3, J4: footprint arv-som-footprints:HRS_DF40C-100DP-0.4V(51) -> arvsom-footprints:HRS_DF40C-100DP-0.4V(51); symbol arv-som:DF40C-100DP-0.4V(51) -> arvsom:DF40C-100DP-0.4V(51)
Changed lines of the file:
@@
 GPIO_VREF
 $Comp
-L arv-som:GND #PWR0224
+L arvsom:GND #PWR0224
 U 1 1 6083430C
 P 3700 7650
@@
 $EndComp
 $Comp
-L arv-som:GND #PWR0225
+L arvsom:GND #PWR0225
 U 1 1 60834719
 P 4900 7650
@@
 $EndComp
 $Comp
-L arv-som:GND #PWR0226
+L arvsom:GND #PWR0226
 U 1 1 608363DA
 P 11075 7625
@@
 $EndComp
 $Comp
-L arv-som:GND #PWR0227
+L arvsom:GND #PWR0227
 U 1 1 6083A5F9
 P 12325 7625
@@
 RESERVED
 $Comp
-L arv-som:DF40C-100DP-0.4V(51) J3
+L arvsom:DF40C-100DP-0.4V(51) J3
 U 1 1 60FEF31E
 P 4300 4800
 F 0 "J3" H 4300 7557 50  0000 C CNN
 F 1 "DF40C-100DP-0.4V(51)" H 4300 7466 50  0000 C CNN
-F 2 "arv-som-footprints:HRS_DF40C-100DP-0.4V(51)" H 4300 4800 50  0001 L BNN
+F 2 "arvsom-footprints:HRS_DF40C-100DP-0.4V(51)" H 4300 4800 50  0001 L BNN
 F 3 "" H 4300 4800 50  0001 L BNN
 F 4 "HRS" H 4300 4800 50  0001 L BNN "Manufacturer"
@@
 Connection ~ 3800 6700
 $Comp
-L arv-som:DF40C-100DP-0.4V(51) J4
+L arvsom:DF40C-100DP-0.4V(51) J4
 U 1 1 60FFB551
 P 11725 4725
 F 0 "J4" H 11725 7482 50  0000 C CNN
 F 1 "DF40C-100DP-0.4V(51)" H 11725 7391 50  0000 C CNN
-F 2 "arv-som-footprints:HRS_DF40C-100DP-0.4V(51)" H 11725 4725 50  0001 L BNN
+F 2 "arvsom-footprints:HRS_DF40C-100DP-0.4V(51)" H 11725 4725 50  0001 L BNN
 F 3 "" H 11725 4725 50  0001 L BNN
 F 4 "HRS" H 11725 4725 50  0001 L BNN "Manufacturer"
