File: VIC7100-config.sch (KiCad schematic (older format))
At the start: 10 parts

Commit message: Connected interfaces to VIC to visualise its ball locations (wip, mock purposes)
Parts:
- gave numbers to parts that had none: 9
Changed lines of the file:
@@
 $Descr A4 11693 8268
 encoding utf-8
-Sheet 9 12
+Sheet 8 11
 Title ""
 Date ""
@@
 $EndDescr
 $Comp
-L antmicroMicrocontrollers:VIC7100 U?
+L antmicroMicrocontrollers:VIC7100 U13
 U 12 1 61E58C70
 P 2650 1100
-F 0 "U?" H 3381 -1952 60  0000 L CNN
+F 0 "U13" H 3381 -1952 60  0000 L CNN
 F 1 "VIC7100" H 3381 -2058 60  0000 L CNN
 F 2 "antmicro-footprints:vic7100" H 2850 1150 60  0001 L CNN
@@
 Connection ~ 2650 5900
 $Comp
-L power:GND #PWR?
+L power:GND #PWR0209
 U 1 1 61ECAD23
 P 2475 6125
-F 0 "#PWR?" H 2475 5875 50  0001 C CNN
+F 0 "#PWR0209" H 2475 5875 50  0001 C CNN
 F 1 "GND" H 2480 5952 50  0000 C CNN
 F 2 "" H 2475 6125 50  0001 C CNN
@@
 BOOT_MODE
 $Comp
-L antmicroMicrocontrollers:VIC7100 U?
+L antmicroMicrocontrollers:VIC7100 U13
 U 13 1 61EF0169
 P 5275 1325
-F 0 "U?" H 6506 423 60  0000 L CNN
+F 0 "U13" H 6506 423 60  0000 L CNN
 F 1 "VIC7100" H 6506 317 60  0000 L CNN
 F 2 "antmicro-footprints:vic7100" H 5475 1375 60  0001 L CNN
@@
 ATEMP_VCAL
 $Comp
-L antmicroResistors0402:R_10k_0402 R?
+L antmicroResistors0402:R_10k_0402 R49
 U 1 1 620611F3
 P 4300 2025
-F 0 "R?" V 4255 2095 60  0000 L CNN
+F 0 "R49" V 4255 2095 60  0000 L CNN
 F 1 "R_10k_0402" H 4300 1875 60  0001 C CNN
 F 2 "antmicro-footprints:0402-res" H 4500 2225 60  0001 L CNN
@@
 $EndComp
 $Comp
-L antmicroCapacitorsmisc:C_100n_0201 C?
+L antmicroCapacitorsmisc:C_100n_0201 C171
 U 1 1 62088F55
 P 4150 2025
-F 0 "C?" H 4265 2070 60  0000 L CNN
+F 0 "C171" H 4265 2070 60  0000 L CNN
 F 1 "C_100n_0201" H 4150 1875 60  0001 C CNN
 F 2 "antmicro-footprints:0201-res" H 4350 2225 60  0001 L CNN
@@
 	4150 2175 4150 2225
 $Comp
-L power:GND #PWR?
+L power:GND #PWR0210
 U 1 1 620F475A
 P 4150 2275
-F 0 "#PWR?" H 4150 2025 50  0001 C CNN
+F 0 "#PWR0210" H 4150 2025 50  0001 C CNN
 F 1 "GND" H 4155 2102 50  0000 C CNN
 F 2 "" H 4150 2275 50  0001 C CNN
@@
 	4075 1525 4450 1525
 $Comp
-L antmicroResistors0402:R_10k_0402 R?
+L antmicroResistors0402:R_10k_0402 R50
 U 1 1 6228863D
 P 4450 2025
-F 0 "R?" V 4405 2095 60  0000 L CNN
+F 0 "R50" V 4405 2095 60  0000 L CNN
 F 1 "R_10k_0402" H 4450 1875 60  0001 C CNN
 F 2 "antmicro-footprints:0402-res" H 4650 2225 60  0001 L CNN
@@
 $EndComp
 $Comp
-L antmicroResistors0402:R_10k_0402 R?
+L antmicroResistors0402:R_10k_0402 R51
 U 1 1 62289923
 P 4600 2025
-F 0 "R?" V 4555 2095 60  0000 L CNN
+F 0 "R51" V 4555 2095 60  0000 L CNN
 F 1 "R_10k_0402" H 4600 1875 60  0001 C CNN
 F 2 "antmicro-footprints:0402-res" H 4800 2225 60  0001 L CNN
@@
 	5275 3325 5275 3525
 $Comp
-L power:GND #PWR?
+L power:GND #PWR0211
 U 1 1 623E400A
 P 5275 3525
-F 0 "#PWR?" H 5275 3275 50  0001 C CNN
+F 0 "#PWR0211" H 5275 3275 50  0001 C CNN
 F 1 "GND" H 5280 3352 50  0000 C CNN
 F 2 "" H 5275 3525 50  0001 C CNN
@@
 SYS_RSTN
 $Comp
-L antmicroResistorsmisc:R_0R_0201 R?
+L antmicroResistorsmisc:R_0R_0201 R52
 U 1 1 62480CED
 P 4975 4425
-F 0 "R?" V 4930 4495 60  0000 L CNN
+F 0 "R52" V 4930 4495 60  0000 L CNN
 F 1 "R_0R_0201" H 4975 4275 60  0001 C CNN
 F 2 "antmicro-footprints:0201-res" H 5175 4625 60  0001 L CNN
@@
 $EndComp
 $Comp
-L antmicroResistorsmisc:R_0R_0201 R?
+L antmicroResistorsmisc:R_0R_0201 R53
 U 1 1 6248208B
 P 4975 4825
-F 0 "R?" V 4930 4895 60  0000 L CNN
+F 0 "R53" V 4930 4895 60  0000 L CNN
 F 1 "R_0R_0201" H 4975 4675 60  0001 C CNN
 F 2 "antmicro-footprints:0201-res" H 5175 5025 60  0001 L CNN
@@
 	4975 4200 4975 4275
 $Comp
-L power:GND #PWR?
+L power:GND #PWR0212
 U 1 1 624C90BA
 P 4975 5050
-F 0 "#PWR?" H 4975 4800 50  0001 C CNN
+F 0 "#PWR0212" H 4975 4800 50  0001 C CNN
 F 1 "GND" H 4980 4877 50  0000 C CNN
 F 2 "" H 4975 5050 50  0001 C CNN
@@
 	5875 4200 5875 4275
 $Comp
-L power:GND #PWR?
+L power:GND #PWR0213
 U 1 1 6253E02A
 P 5875 5050
-F 0 "#PWR?" H 5875 4800 50  0001 C CNN
+F 0 "#PWR0213" H 5875 4800 50  0001 C CNN
 F 1 "GND" H 5880 4877 50  0000 C CNN
 F 2 "" H 5875 5050 50  0001 C CNN
@@
 	5875 4625 5875 4675
 $Comp
-L antmicroResistors0402:R_10k_0402 R?
+L antmicroResistors0402:R_10k_0402 R54
 U 1 1 6254985B
 P 5875 4425
-F 0 "R?" V 5830 4495 60  0000 L CNN
+F 0 "R54" V 5830 4495 60  0000 L CNN
 F 1 "R_10k_0402" H 5875 4275 60  0001 C CNN
 F 2 "antmicro-footprints:0402-res" H 6075 4625 60  0001 L CNN
@@
 $EndComp
 $Comp
-L antmicroCapacitors0402:C_10n_0402 C?
+L antmicroCapacitors0402:C_10n_0402 C172
 U 1 1 62549E17
 P 5875 4825
-F 0 "C?" H 5990 4870 60  0000 L CNN
+F 0 "C172" H 5990 4870 60  0000 L CNN
 F 1 "C_10n_0402" H 5875 4675 60  0001 C CNN
 F 2 "antmicro-footprints:0402-cap" H 6075 5025 60  0001 L CNN

Commit message: Schematic cleanup, added logotypes
Parts:
- added C35: C_1u_0402, antmicro-footprints:0402-cap, symbol antmicroCapacitors0402:C_1u_0402
- added C36: C_100n_0201, antmicro-footprints:0201-res, symbol antmicroCapacitorsmisc:C_100n_0201
- added R18, R19, R20, R22, R23, R24: R_33R_0402, antmicro-footprints:0402-res, symbol antmicroResistors0402:R_33R_0402
- added R21: R_4k7_0402, antmicro-footprints:0402-res, symbol antmicroResistors0402:R_4k7_0402
- added U2: GD25LQ256DWIGR, antmicro-footprints:8-WSON-6x5, symbol antmicroMemory:GD25LQ256DWIGR
Connections:
- net labels added: QSPI_CS0_N
- wire segments 48 -> 66
Other:
- note added: "NOR Flash"
- note added: "TODO: replace 33R with 0201 package"
- note added: "VIC7100 configuration"
- moved on the sheet: R52, R53

Commit message: Changes to VIC config after review
Parts:
- removed R52, R53: R_0R_0201, antmicro-footprints:0201-res, symbol antmicroResistorsmisc:R_0R_0201
- added R109, R110, R111, R112, R113, R114, R115, R116, R52, R53: R_10k_0402, antmicro-footprints:0402-res, symbol antmicroResistors0402:R_10k_0402
- added TP13, TP14, TP15, TP16: TP_SMD_0_75MM, antmicro-footprints:Testpoint_smd_0_75mm, symbol antmicroTestPoints:TP_SMD_0_75MM
Connections:
- wire segments 66 -> 94
Other:
- note added: "TBD: which pins should be pulled high/low"
- note added: "Test mode enable for DFT\n(active high)"

Commit message: Added local libraries
Parts:
- C171, C36: footprint antmicro-footprints:0201-res -> arv-som-footprints:0201-res; symbol antmicroCapacitorsmisc:C_100n_0201 -> arv-som:C_100n_0201
- C172: footprint antmicro-footprints:0402-cap -> arv-som-footprints:0402-cap; symbol antmicroCapacitors0402:C_10n_0402 -> arv-som:C_10n_0402
- C35: footprint antmicro-footprints:0402-cap -> arv-som-footprints:0402-cap; symbol antmicroCapacitors0402:C_1u_0402 -> arv-som:C_1u_0402
- R109, R110, R111, R112, R113, R114, R115, R116, R49, R50, R51, R52, R53, R54: footprint antmicro-footprints:0402-res -> arv-som-footprints:0402-res; symbol antmicroResistors0402:R_10k_0402 -> arv-som:R_10k_0402
- R18, R19, R20, R22, R23, R24: footprint antmicro-footprints:0402-res -> arv-som-footprints:0402-res; symbol antmicroResistors0402:R_33R_0402 -> arv-som:R_33R_0402
- R21: footprint antmicro-footprints:0402-res -> arv-som-footprints:0402-res; symbol antmicroResistors0402:R_4k7_0402 -> arv-som:R_4k7_0402
- TP13, TP14, TP15, TP16: footprint antmicro-footprints:Testpoint_smd_0_75mm -> arv-som-footprints:Testpoint_smd_0_75mm; symbol antmicroTestPoints:TP_SMD_0_75MM -> arv-som:TP_SMD_0_75MM
- U13: footprint antmicro-footprints:vic7100 -> arv-som-footprints:vic7100; symbol antmicroMicrocontrollers:VIC7100 -> arv-som:VIC7100
- U2: footprint antmicro-footprints:8-WSON-6x5 -> arv-som-footprints:8-WSON-6x5; symbol antmicroMemory:GD25LQ256DWIGR -> arv-som:GD25LQ256DWIGR

Commit message: Update naming convention
Parts:
- C171, C36: footprint arv-som-footprints:0201-res -> arvsom-footprints:0201-res; symbol arv-som:C_100n_0201 -> arvsom:C_100n_0201
- C172: footprint arv-som-footprints:0402-cap -> arvsom-footprints:0402-cap; symbol arv-som:C_10n_0402 -> arvsom:C_10n_0402
- C35: footprint arv-som-footprints:0402-cap -> arvsom-footprints:0402-cap; symbol arv-som:C_1u_0402 -> arvsom:C_1u_0402
- R109, R110, R111, R112, R113, R114, R115, R116, R49, R50, R51, R52, R53, R54: footprint arv-som-footprints:0402-res -> arvsom-footprints:0402-res; symbol arv-som:R_10k_0402 -> arvsom:R_10k_0402
- R18, R19, R20, R22, R23, R24: footprint arv-som-footprints:0402-res -> arvsom-footprints:0402-res; symbol arv-som:R_33R_0402 -> arvsom:R_33R_0402
- R21: footprint arv-som-footprints:0402-res -> arvsom-footprints:0402-res; symbol arv-som:R_4k7_0402 -> arvsom:R_4k7_0402
- TP13, TP14, TP15, TP16: footprint arv-som-footprints:Testpoint_smd_0_75mm -> arvsom-footprints:Testpoint_smd_0_75mm; symbol arv-som:TP_SMD_0_75MM -> arvsom:TP_SMD_0_75MM
- U13: footprint arv-som-footprints:vic7100 -> arvsom-footprints:vic7100; symbol arv-som:VIC7100 -> arvsom:VIC7100
- U2: footprint arv-som-footprints:8-WSON-6x5 -> arvsom-footprints:8-WSON-6x5; symbol arv-som:GD25LQ256DWIGR -> arvsom:GD25LQ256DWIGR
