File: ethernet.sch (KiCad schematic (older format))
At the start: 44 parts

Commit message: Connected interfaces to VIC to visualise its ball locations (wip, mock purposes)
Parts:
- gave numbers to parts that had none: 44

Commit message: Updated interfaces, CPU and B2B connector connections
Connections:
- net labels added: LED_MODE, RGMII_GTXCLK, RGMII_MDC, RGMII_MDIO, RGMII_RCTL, RGMII_RXCLK, RGMII_RXDV, RGMII_TXEN
- net labels removed: ETH_INT_N, ETH_MDC, RGMII_REF_CLK, RGMII_RX_CLK, RGMII_RX_DV, RGMII_TX_CLK, RGMII_TX_DV
- wire segments 213 -> 212
- no-connect marks 1 -> 2
Other:
- note added: "Can be connected to SYS_RST from PMIC"
Changed lines of the file:
@@
 $Descr A3 16535 11693
 encoding utf-8
-Sheet 5 11
+Sheet 5 10
 Title ""
 Date ""
@@
 $EndDescr
 Text GLabel 7950 9050 0    50   UnSpc ~ 0
-RGMII_RX_DV
+RGMII_RXDV
 Text GLabel 7950 8950 0    50   UnSpc ~ 0
 RGMII_RXD3
@@
 RGMII_RXD1
 Text GLabel 7950 9150 0    50   UnSpc ~ 0
-RGMII_RX_CLK
+RGMII_RXCLK
 Text GLabel 8925 8500 1    50   Input ~ 0
 VCC3V3
 Text GLabel 7950 9250 0    50   UnSpc ~ 0
-RGMII_REF_CLK
+LED_MODE
 Text GLabel 7950 9450 0    50   UnSpc ~ 0
 ETH_MDIO
 Text GLabel 7950 9550 0    50   UnSpc ~ 0
 ETH_~RESET
-Text Label 7150 9650 0    50   ~ 0
-ETH_LED1
-Text Label 7150 9750 0    50   ~ 0
-ETH_LED2
 Wire Wire Line
 	8800 3600 8800 3375
@@
 Wire Wire Line
 	6075 6300 6900 6300
-Wire Wire Line
-	6900 6100 6075 6100
-Text GLabel 6075 6100 0    50   Output ~ 0
-ETH_INT_N
-Text GLabel 6075 6300 0    50   Output ~ 0
-RGMII_REF_CLK
+Text GLabel 6075 6300 0    50   Input ~ 0
+LED_MODE
 Wire Wire Line
 	6650 6400 6650 6450
 Wire Wire Line
 	6650 6450 6075 6450
-Text GLabel 6100 5700 0    50   Output ~ 0
-RGMII_RX_CLK
 Text GLabel 6100 5600 0    50   Output ~ 0
 RGMII_RXD3
@@
 Wire Wire Line
 	6900 5300 6100 5300
-Text GLabel 6100 5000 0    50   Input ~ 0
-RGMII_TX_CLK
 Text GLabel 6100 4900 0    50   Input ~ 0
 RGMII_TXD3
@@
 Text GLabel 6100 4600 0    50   Input ~ 0
 RGMII_TXD0
-Text GLabel 6100 4500 0    50   Input ~ 0
-RGMII_TX_DV
 Wire Wire Line
 	6100 4900 6900 4900
@@
 Wire Wire Line
 	6900 4600 6100 4600
-Text GLabel 6100 4300 0    50   BiDi ~ 0
-ETH_MDIO
-Text GLabel 6100 4200 0    50   Input ~ 0
-ETH_MDC
 Wire Wire Line
 	6100 4200 6900 4200
@@
 	3025 4175 3275 4175
 Text GLabel 6100 5200 0    50   Output ~ 0
-RGMII_RX_DV
+RGMII_RXDV
 Wire Wire Line
 	3575 8725 3750 8725
@@
 P 7100 3800
 F 0 "U11" H 8200 711 50  0000 C CNN
-F 1 "KSZ9031RNXCA" H 8200 620 50  0000 C CNN
+F 1 "KSZ9031RNXCA" H 7500 825 50  0000 C CNN
 F 2 "antmicro-footprints:QFN-48-Microchip-QFN77-48LD-PL-2" H 7100 4300 50  0001 L CNN
 F 3 "http://ww1.microchip.com/downloads/en/DeviceDoc/00002117F.pdf" H 7100 4300 50  0001 L CNN
@@
 Text GLabel 6100 6000 0    50   Input ~ 0
 ETH_LED1
+Text GLabel 6100 4500 0    50   Input ~ 0
+RGMII_TXEN
+Text GLabel 6100 5700 0    50   Output ~ 0
+RGMII_RXCLK
+Text GLabel 6100 5000 0    50   Input ~ 0
+RGMII_GTXCLK
+Text GLabel 6100 4300 0    50   BiDi ~ 0
+RGMII_MDIO
+Text GLabel 6100 4200 0    50   Input ~ 0
+RGMII_MDC
+Text GLabel 7150 9650 0    50   Input ~ 0
+ETH_LED2
+Text GLabel 7150 9750 0    50   Input ~ 0
+ETH_LED1
+NoConn ~ 6900 6100
+Text Notes 5225 6575 0    50   ~ 0
+Can be connected to SYS_RST from PMIC
+Text Label 6325 5200 0    50   ~ 0
+RGMII_RCTL
 $EndSCHEMATC

Commit message: Neatened decoupling labels
Connections:
- wire segments 212 -> 215

Commit message: Added local libraries
Parts:
- C45, C47, C49, C50, C58: footprint antmicro-footprints:0402-cap -> arv-som-footprints:0402-cap; symbol antmicroCapacitors0402:C_4u7_0402 -> arv-som:C_4u7_0402
- C46, C48, C51, C52, C53: footprint antmicro-footprints:0402-cap -> arv-som-footprints:0402-cap; symbol antmicroCapacitors0402:C_470n_0402 -> arv-som:C_470n_0402
- C54: footprint antmicro-footprints:0402-cap -> arv-som-footprints:0402-cap; symbol antmicroCapacitors0402:C_100n_0402 -> arv-som:C_100n_0402
- C55, C56, C57, C59, C60, C61, C62, C63, C64, C65, C66, C67, C68: footprint antmicro-footprints:0402-cap -> arv-som-footprints:0402-cap; symbol antmicroCapacitors0402:C_10n_0402 -> arv-som:C_10n_0402
- C69, C70: footprint antmicro-footprints:0402-cap -> arv-som-footprints:0402-cap; symbol antmicroCapacitors0402:C_22p_0402 -> arv-som:C_22p_0402
- FB2, FB3, FB4: footprint antmicro-footprints:0603 -> arv-som-footprints:0603; symbol antmicroFerriteBeadsandChips:BLM18AG601SN1D -> arv-som:BLM18AG601SN1D
- R29: footprint antmicro-footprints:0402-res -> arv-som-footprints:0402-res; symbol antmicroResistors0402:R_1k_0402 -> arv-som:R_1k_0402
- R30: footprint antmicro-footprints:0402-res -> arv-som-footprints:0402-res; symbol antmicroResistors0402:R_12k1_0402 -> arv-som:R_12k1_0402
- R31, R32, R33, R34, R35, R36, R38, R39, R40: footprint antmicro-footprints:0402-res -> arv-som-footprints:0402-res; symbol antmicroResistors0402:R_10k_0402 -> arv-som:R_10k_0402
- R37: footprint antmicro-footprints:0402-res -> arv-som-footprints:0402-res; symbol antmicroResistors0402:R_4k7_0402 -> arv-som:R_4k7_0402
- R41: footprint antmicro-footprints:0402-res -> arv-som-footprints:0402-res; symbol antmicroResistors0402:R_1M5_0402 -> arv-som:R_1M5_0402
- U11: footprint antmicro-footprints:QFN-48-Microchip-QFN77-48LD-PL-2 -> arv-som-footprints:QFN-48-Microchip-QFN77-48LD-PL-2; symbol antmicroInterfaceControllers:KSZ9031RNXCA -> arv-som:KSZ9031RNXCA
- Y1: footprint antmicro-footprints:KX-7 -> arv-som-footprints:KX-7; symbol antmicroCrystals:ABM8G-25.000MHZ-18-D2Y-T -> arv-som:ABM8G-25.000MHZ-18-D2Y-T

Commit message: Update naming convention
Parts:
- C45, C47, C49, C50, C58: footprint arv-som-footprints:0402-cap -> arvsom-footprints:0402-cap; symbol arv-som:C_4u7_0402 -> arvsom:C_4u7_0402
- C46, C48, C51, C52, C53: footprint arv-som-footprints:0402-cap -> arvsom-footprints:0402-cap; symbol arv-som:C_470n_0402 -> arvsom:C_470n_0402
- C54: footprint arv-som-footprints:0402-cap -> arvsom-footprints:0402-cap; symbol arv-som:C_100n_0402 -> arvsom:C_100n_0402
- C55, C56, C57, C59, C60, C61, C62, C63, C64, C65, C66, C67, C68: footprint arv-som-footprints:0402-cap -> arvsom-footprints:0402-cap; symbol arv-som:C_10n_0402 -> arvsom:C_10n_0402
- C69, C70: footprint arv-som-footprints:0402-cap -> arvsom-footprints:0402-cap; symbol arv-som:C_22p_0402 -> arvsom:C_22p_0402
- FB2, FB3, FB4: footprint arv-som-footprints:0603 -> arvsom-footprints:0603; symbol arv-som:BLM18AG601SN1D -> arvsom:BLM18AG601SN1D
- R29: footprint arv-som-footprints:0402-res -> arvsom-footprints:0402-res; symbol arv-som:R_1k_0402 -> arvsom:R_1k_0402
- R30: footprint arv-som-footprints:0402-res -> arvsom-footprints:0402-res; symbol arv-som:R_12k1_0402 -> arvsom:R_12k1_0402
- R31, R32, R33, R34, R35, R36, R38, R39, R40: footprint arv-som-footprints:0402-res -> arvsom-footprints:0402-res; symbol arv-som:R_10k_0402 -> arvsom:R_10k_0402
- R37: footprint arv-som-footprints:0402-res -> arvsom-footprints:0402-res; symbol arv-som:R_4k7_0402 -> arvsom:R_4k7_0402
- R41: footprint arv-som-footprints:0402-res -> arvsom-footprints:0402-res; symbol arv-som:R_1M5_0402 -> arvsom:R_1M5_0402
- U11: footprint arv-som-footprints:QFN-48-Microchip-QFN77-48LD-PL-2 -> arvsom-footprints:QFN-48-Microchip-QFN77-48LD-PL-2; symbol arv-som:KSZ9031RNXCA -> arvsom:KSZ9031RNXCA
- Y1: footprint arv-som-footprints:KX-7 -> arvsom-footprints:KX-7; symbol arv-som:ABM8G-25.000MHZ-18-D2Y-T -> arvsom:ABM8G-25.000MHZ-18-D2Y-T
