File: expansion-connectors.sch (KiCad schematic (older format))
At the start: 5 parts, among them J1 QSE-020-01-F-D, J2 QSE-020-01-F-D

Commit message: Added local libraries
Parts:
- J1, J2: footprint scalenode-footprints:QSE-020-01-XXX-D-A -> arv-som-footprints:QSE-020-01-XXX-D-A; symbol scalenode:QSE-020-01-F-D -> arv-som:QSE-020-01-F-D
- MP1: footprint scalenode-footprints:mounting-hole-2.2mm -> arv-som-footprints:mounting-hole-2.2mm; symbol scalenode:PCB_Mount_Hole_2.2_4.5 -> arv-som:PCB_Mount_Hole_2.2_4.5
- MP2, MP3: footprint scalenode-footprints:Mount-hole-M2.5 -> arv-som-footprints:Mount-hole-M2.5; symbol scalenode:PCB_Mount_Hole_2.5_6.2 -> arv-som:PCB_Mount_Hole_2.5_6.2
Changed lines of the file:
@@
 HDMI1_HOTPLUG
 $Comp
-L scalenode:QSE-020-01-F-D J1
+L arv-som:QSE-020-01-F-D J1
 U 1 1 600BF3F1
 P 5125 4050
 F 0 "J1" H 5275 4225 50  0000 C CNN
 F 1 "QSE-020-01-F-D" H 5275 4134 50  0000 C CNN
-F 2 "scalenode-footprints:QSE-020-01-XXX-D-A" H 5275 1700 60  0001 L CNN
+F 2 "arv-som-footprints:QSE-020-01-XXX-D-A" H 5275 1700 60  0001 L CNN
 F 3 "https://eu.mouser.com/datasheet/2/527/qse-1370325.pdf" H 6125 3300 60  0001 L CNN
 F 4 "QSE-020-01-F-D" H 4825 1550 60  0001 L CNN "MPN"
@@
 Connection ~ 5625 5200
 $Comp
-L scalenode:GND #PWR01
+L arv-som:GND #PWR01
 U 1 1 601419BB
 P 5275 6400
@@
 SDA0
 $Comp
-L scalenode:GND #PWR02
+L arv-som:GND #PWR02
 U 1 1 601DA6BC
 P 9025 6450
@@
 	8775 5150 8325 5150
 $Comp
-L scalenode:QSE-020-01-F-D J2
+L arv-som:QSE-020-01-F-D J2
 U 1 1 601B8118
 P 8875 4100
 F 0 "J2" H 9025 4275 50  0000 C CNN
 F 1 "QSE-020-01-F-D" H 9025 4184 50  0000 C CNN
-F 2 "scalenode-footprints:QSE-020-01-XXX-D-A" H 9025 1750 60  0001 L CNN
+F 2 "arv-som-footprints:QSE-020-01-XXX-D-A" H 9025 1750 60  0001 L CNN
 F 3 "https://eu.mouser.com/datasheet/2/527/qse-1370325.pdf" H 9875 3350 60  0001 L CNN
 F 4 "QSE-020-01-F-D" H 8575 1600 60  0001 L CNN "MPN"
@@
 VCC5V0
 $Comp
-L scalenode:GND #PWR03
+L arv-som:GND #PWR03
 U 1 1 603380B5
 P 9700 4350
@@
 QSE connector current rating:\n2A per pin (2 pins powered)
 $Comp
-L scalenode:PCB_Mount_Hole_2.2_4.5 MP1
+L arv-som:PCB_Mount_Hole_2.2_4.5 MP1
 U 1 1 603AAAE1
 P 5325 7725
 F 0 "MP1" H 5533 7771 50  0000 L CNN
 F 1 "PCB_Mount_Hole_2.2_4.5" H 5533 7680 50  0000 L CNN
-F 2 "scalenode-footprints:mounting-hole-2.2mm" H 6125 8425 50  0001 C CNN
+F 2 "arv-som-footprints:mounting-hole-2.2mm" H 6125 8425 50  0001 C CNN
 F 3 "" H 6275 8525 50  0001 C CNN
 	1    5325 7725
@@
 3V3_SSD
 $Comp
-L scalenode:PCB_Mount_Hole_2.5_6.2 MP2
+L arv-som:PCB_Mount_Hole_2.5_6.2 MP2
 U 1 1 606358C7
 P 6900 7750
 F 0 "MP2" H 7108 7796 50  0000 L CNN
 F 1 "PCB_Mount_Hole_2.5_6.2" H 7108 7705 50  0000 L CNN
-F 2 "scalenode-footprints:Mount-hole-M2.5" H 7700 8450 50  0001 C CNN
+F 2 "arv-som-footprints:Mount-hole-M2.5" H 7700 8450 50  0001 C CNN
 F 3 "" H 7850 8550 50  0001 C CNN
 	1    6900 7750
@@
 $EndComp
 $Comp
-L scalenode:PCB_Mount_Hole_2.5_6.2 MP3
+L arv-som:PCB_Mount_Hole_2.5_6.2 MP3
 U 1 1 606391B7
 P 8400 7750
 F 0 "MP3" H 8608 7796 50  0000 L CNN
 F 1 "PCB_Mount_Hole_2.5_6.2" H 8608 7705 50  0000 L CNN
-F 2 "scalenode-footprints:Mount-hole-M2.5" H 9200 8450 50  0001 C CNN
+F 2 "arv-som-footprints:Mount-hole-M2.5" H 9200 8450 50  0001 C CNN
 F 3 "" H 9350 8550 50  0001 C CNN
 	1    8400 7750

Commit message: Update naming convention
Parts:
- J1, J2: footprint arv-som-footprints:QSE-020-01-XXX-D-A -> arvsom-footprints:QSE-020-01-XXX-D-A; symbol arv-som:QSE-020-01-F-D -> arvsom:QSE-020-01-F-D
- MP1: footprint arv-som-footprints:mounting-hole-2.2mm -> arvsom-footprints:mounting-hole-2.2mm; symbol arv-som:PCB_Mount_Hole_2.2_4.5 -> arvsom:PCB_Mount_Hole_2.2_4.5
- MP2, MP3: footprint arv-som-footprints:Mount-hole-M2.5 -> arvsom-footprints:Mount-hole-M2.5; symbol arv-som:PCB_Mount_Hole_2.5_6.2 -> arvsom:PCB_Mount_Hole_2.5_6.2
Changed lines of the file:
@@
 HDMI1_HOTPLUG
 $Comp
-L arv-som:QSE-020-01-F-D J1
+L arvsom:QSE-020-01-F-D J1
 U 1 1 600BF3F1
 P 5125 4050
 F 0 "J1" H 5275 4225 50  0000 C CNN
 F 1 "QSE-020-01-F-D" H 5275 4134 50  0000 C CNN
-F 2 "arv-som-footprints:QSE-020-01-XXX-D-A" H 5275 1700 60  0001 L CNN
+F 2 "arvsom-footprints:QSE-020-01-XXX-D-A" H 5275 1700 60  0001 L CNN
 F 3 "https://eu.mouser.com/datasheet/2/527/qse-1370325.pdf" H 6125 3300 60  0001 L CNN
 F 4 "QSE-020-01-F-D" H 4825 1550 60  0001 L CNN "MPN"
@@
 Connection ~ 5625 5200
 $Comp
-L arv-som:GND #PWR01
+L arvsom:GND #PWR01
 U 1 1 601419BB
 P 5275 6400
@@
 SDA0
 $Comp
-L arv-som:GND #PWR02
+L arvsom:GND #PWR02
 U 1 1 601DA6BC
 P 9025 6450
@@
 	8775 5150 8325 5150
 $Comp
-L arv-som:QSE-020-01-F-D J2
+L arvsom:QSE-020-01-F-D J2
 U 1 1 601B8118
 P 8875 4100
 F 0 "J2" H 9025 4275 50  0000 C CNN
 F 1 "QSE-020-01-F-D" H 9025 4184 50  0000 C CNN
-F 2 "arv-som-footprints:QSE-020-01-XXX-D-A" H 9025 1750 60  0001 L CNN
+F 2 "arvsom-footprints:QSE-020-01-XXX-D-A" H 9025 1750 60  0001 L CNN
 F 3 "https://eu.mouser.com/datasheet/2/527/qse-1370325.pdf" H 9875 3350 60  0001 L CNN
 F 4 "QSE-020-01-F-D" H 8575 1600 60  0001 L CNN "MPN"
@@
 VCC5V0
 $Comp
-L arv-som:GND #PWR03
+L arvsom:GND #PWR03
 U 1 1 603380B5
 P 9700 4350
@@
 QSE connector current rating:\n2A per pin (2 pins powered)
 $Comp
-L arv-som:PCB_Mount_Hole_2.2_4.5 MP1
+L arvsom:PCB_Mount_Hole_2.2_4.5 MP1
 U 1 1 603AAAE1
 P 5325 7725
 F 0 "MP1" H 5533 7771 50  0000 L CNN
 F 1 "PCB_Mount_Hole_2.2_4.5" H 5533 7680 50  0000 L CNN
-F 2 "arv-som-footprints:mounting-hole-2.2mm" H 6125 8425 50  0001 C CNN
+F 2 "arvsom-footprints:mounting-hole-2.2mm" H 6125 8425 50  0001 C CNN
 F 3 "" H 6275 8525 50  0001 C CNN
 	1    5325 7725
@@
 3V3_SSD
 $Comp
-L arv-som:PCB_Mount_Hole_2.5_6.2 MP2
+L arvsom:PCB_Mount_Hole_2.5_6.2 MP2
 U 1 1 606358C7
 P 6900 7750
 F 0 "MP2" H 7108 7796 50  0000 L CNN
 F 1 "PCB_Mount_Hole_2.5_6.2" H 7108 7705 50  0000 L CNN
-F 2 "arv-som-footprints:Mount-hole-M2.5" H 7700 8450 50  0001 C CNN
+F 2 "arvsom-footprints:Mount-hole-M2.5" H 7700 8450 50  0001 C CNN
 F 3 "" H 7850 8550 50  0001 C CNN
 	1    6900 7750
@@
 $EndComp
 $Comp
-L arv-som:PCB_Mount_Hole_2.5_6.2 MP3
+L arvsom:PCB_Mount_Hole_2.5_6.2 MP3
 U 1 1 606391B7
 P 8400 7750
 F 0 "MP3" H 8608 7796 50  0000 L CNN
 F 1 "PCB_Mount_Hole_2.5_6.2" H 8608 7705 50  0000 L CNN
-F 2 "arv-som-footprints:Mount-hole-M2.5" H 9200 8450 50  0001 C CNN
+F 2 "arvsom-footprints:Mount-hole-M2.5" H 9200 8450 50  0001 C CNN
 F 3 "" H 9350 8550 50  0001 C CNN
 	1    8400 7750
