File: lpddr4.sch (KiCad schematic (older format))
At the start: 44 parts

Commit message: Connected interfaces to VIC to visualise its ball locations (wip, mock purposes)
Parts:
- gave numbers to parts that had none: 43
Connections:
- net labels added: DDR0_A00, DDR0_A01, DDR0_A02, DDR0_A03, DDR0_A04, DDR0_A05, DDR0_CK0_N, DDR0_CK0_P, DDR0_CK1_N, DDR0_CK1_P, DDR0_CKE0, DDR0_CKE1
- net labels removed: CA2_A, CA3_A, CA4_A, CA5_A, CA_0A, CA_1A, CKE0_A, CK_CA, CK_TA
- wire segments 94 -> 96
Other:
- note added: "TODO: find suitable LPDDR4 (32bit, 2ch, 4die, 1Gb)"

Commit message: Updated interfaces, CPU and B2B connector connections
Parts:
- removed R42: R_10k_0402, antmicro-footprints:0402-res, symbol antmicroResistors0402:R_10k_0402
- added C207, C208, C209, C210, C211, C212, C213, C214, C215, C216, C217, C218, C219, C220, C221, C222, C223, C224, C225, C226, C227, C228, C229, C230, C231, C232, C233, C234, C235, C236, C237, C238, C239, C240, C241: C_100n_0201, antmicro-footprints:0201-res, symbol antmicroCapacitorsmisc:C_100n_0201
- added R100, R102: R_0R_0402, antmicro-footprints:0402-res, symbol antmicroResistors0402:R_0R_0402
- added R101, R103, R104, R105, R106, R107, R108, R92, R93, R94, R95, R96, R98: R_10k_0402, antmicro-footprints:0402-res, symbol antmicroResistors0402:R_10k_0402
- added R42, R97, R99: R_240R_0402, antmicro-footprints:0402-res, symbol antmicroResistors0402:R_240R_0402
- added U1: MT53E256M32D2DS-053, antmicro-footprints:BGA-200_10.0x14.5mm_Layout12x22_P0.80x0.65mm, symbol antmicroMemory:MT53E256M32D2DS-053
Connections:
- net labels added: DDR0_CS0, DDR0_CS1, DDR0_CS2, DDR0_CS3, DDR0_DMI0, DDR0_DMI1, DDR0_DMI2, DDR0_DMI3, DDR0_DQ00, DDR0_DQ01, DDR0_DQ02, DDR0_DQ03, DDR0_DQ04, DDR0_DQ05, DDR0_DQ06, DDR0_DQ07, DDR0_DQ08, DDR0_DQ09, DDR0_DQ10, DDR0_DQ11, DDR0_DQ12, DDR0_DQ13, DDR0_DQ14, DDR0_DQ15, DDR0_DQ16, DDR0_DQ17, DDR0_DQ18, DDR0_DQ19, DDR0_DQ20, DDR0_DQ21, DDR0_DQ22, DDR0_DQ23, DDR0_DQ24, DDR0_DQ25, DDR0_DQ26, DDR0_DQ27, DDR0_DQ28, DDR0_DQ29, DDR0_DQ30, DDR0_DQ31, DDR0_DQS0N, DDR0_DQS0P, DDR0_DQS1N, DDR0_DQS1P, DDR0_DQS2N, DDR0_DQS2P, DDR0_DQS3N, DDR0_DQS3P, DDR0_ODT0, DDR0_ODT1, DDR0_ODT_0, DDR0_ODT_1, DDR0_RSTN, DDR1_A00, DDR1_A01, DDR1_A02, DDR1_A03, DDR1_A04, DDR1_A05, DDR1_CK0_N, DDR1_CK0_P, DDR1_CK1_N, DDR1_CK1_P, DDR1_CKE0, DDR1_CKE1, DDR1_CS0, DDR1_CS1, DDR1_CS2, DDR1_DMI0, DDR1_DMI1, DDR1_DMI2, DDR1_DMI3, DDR1_DQ00, DDR1_DQ01, DDR1_DQ02, DDR1_DQ03, DDR1_DQ04, DDR1_DQ05, DDR1_DQ06, DDR1_DQ07, DDR1_DQ08, DDR1_DQ09, DDR1_DQ10, DDR1_DQ11, DDR1_DQ12, DDR1_DQ13, DDR1_DQ14, DDR1_DQ15, DDR1_DQ16, DDR1_DQ17, DDR1_DQ18, DDR1_DQ19, DDR1_DQ20, DDR1_DQ21, DDR1_DQ22, DDR1_DQ23, DDR1_DQ24, DDR1_DQ25, DDR1_DQ26, DDR1_DQ27, DDR1_DQ28, DDR1_DQ29, DDR1_DQ30, DDR1_DQ31, DDR1_DQS0N, DDR1_DQS0P, DDR1_DQS1N, DDR1_DQS1P, DDR1_DQS2N, DDR1_DQS2P, DDR1_DQS3N, DDR1_DQS3P, DDR1_ODT0, DDR1_ODT1, DDR1_ODT_0, DDR1_ODT_1, DDR1_RSTN, DDR_CS3
- net labels removed: CS0_A, CS0_B, DMI_0A, DMI_1A, DQ00_A, DQ01_A, DQ02_A, DQ03_A, DQ04_A, DQ05_A, DQ06_A, DQ07_A, DQ08_A, DQ09_A, DQ10_A, DQ11_A, DQ12_A, DQ13_A, DQ14_A, DQ15_A, DQ_S0_CA, DQ_S0_TA, DQ_S1_CA, DQ_S1_TA, OTD_CA_A, RESET_N
- wire segments 96 -> 244

Commit message: Updated DDR MPN
Parts:
- removed U1, U12: MT53E256M32D2DS-053, antmicro-footprints:BGA-200_10.0x14.5mm_Layout12x22_P0.80x0.65mm, symbol antmicroMemory:MT53E256M32D2DS-053
- added U? (x4): MT53D1024M32D4DT-053, antmicro-footprints:BGA-200_10.0x14.5mm_Layout12x22_P0.80x0.65mm, symbol antmicroMemory:MT53D1024M32D4DT-053
Changed lines of the file:
@@
 Wire Wire Line
 	3650 6025 3875 6025
-$Comp
-L antmicroMemory:MT53E256M32D2DS-053 U12
-U 2 1 60A69CAC
-P 2850 7025
-F 0 "U12" H 2350 8375 50  0000 C CNN
-F 1 "MT53E256M32D2DS-053" H 3550 8475 50  0001 C CNN
-F 2 "antmicro-footprints:BGA-200_10.0x14.5mm_Layout12x22_P0.80x0.65mm" H 2900 5125 50  0001 C CNN
-F 3 "" H 2750 5825 50  0001 C CNN
-F 4 "Micron" H 3325 5675 50  0000 C CNN "Manufacturer"
-F 5 "MT53E256M32D2DS-053 WT:B" H 3775 5575 50  0000 C CNN "MPN"
-	2    2850 7025
-	1    0    0    -1
-$EndComp
 Wire Wire Line
 	3625 1850 3800 1850
@@
 	3625 3450 3900 3450
 $Comp
-L antmicroMemory:MT53E256M32D2DS-053 U12
-U 1 1 60A63E27
-P 2825 3050
-F 0 "U12" H 2325 4425 50  0000 C CNN
-F 1 "MT53E256M32D2DS-053" H 3525 4500 50  0001 C CNN
-F 2 "antmicro-footprints:BGA-200_10.0x14.5mm_Layout12x22_P0.80x0.65mm" H 2875 1150 50  0001 C CNN
-F 3 "" H 2725 1850 50  0001 C CNN
-F 4 "Micron" H 3300 1700 50  0000 C CNN "Manufacturer"
-F 5 "MT53E256M32D2DS-053 WT:B" H 3750 1625 50  0000 C CNN "MPN"
-	1    2825 3050
-	1    0    0    -1
-$EndComp
-$Comp
 L antmicroResistors0402:R_10k_0402 R43
 U 1 1 60AAAA68
@@
 	11750 3900 12025 3900
 $Comp
-L antmicroMemory:MT53E256M32D2DS-053 U1
-U 1 1 616DD63E
-P 10950 3500
-F 0 "U1" H 10425 4850 50  0000 C CNN
-F 1 "MT53E256M32D2DS-053" H 11650 4950 50  0001 C CNN
-F 2 "antmicro-footprints:BGA-200_10.0x14.5mm_Layout12x22_P0.80x0.65mm" H 11000 1600 50  0001 C CNN
-F 3 "" H 10850 2300 50  0001 C CNN
-F 4 "Micron" H 11450 2150 50  0000 C CNN "Manufacturer"
-F 5 "MT53E256M32D2DS-053 WT:B" H 11900 2075 50  0000 C CNN "MPN"
-	1    10950 3500
-	1    0    0    -1
-$EndComp
-$Comp
 L antmicroResistors0402:R_10k_0402 R98
 U 1 1 616DD647
@@
 	0    1    1    0
 $EndComp
-$Comp
-L antmicroMemory:MT53E256M32D2DS-053 U1
-U 2 1 616DD62A
-P 10975 7375
-F 0 "U1" H 10450 8725 50  0000 C CNN
-F 1 "MT53E256M32D2DS-053" H 11675 8825 50  0001 C CNN
-F 2 "antmicro-footprints:BGA-200_10.0x14.5mm_Layout12x22_P0.80x0.65mm" H 11025 5475 50  0001 C CNN
-F 3 "" H 10875 6175 50  0001 C CNN
-F 4 "Micron" H 11475 6025 50  0000 C CNN "Manufacturer"
-F 5 "MT53E256M32D2DS-053 WT:B" H 11925 5950 50  0000 C CNN "MPN"
-	2    10975 7375
-	1    0    0    -1
-$EndComp
 Wire Wire Line
 	11775 6375 12000 6375
@@
 	1    0    0    -1
 $EndComp
+$Comp
+L antmicroMemory:MT53D1024M32D4DT-053 U?
+U 1 1 62E16A15
+P 2825 3050
+F 0 "U?" H 2625 1575 50  0000 C CNN
+F 1 "MT53D1024M32D4DT-053" H 3525 4500 50  0001 C CNN
+F 2 "antmicro-footprints:BGA-200_10.0x14.5mm_Layout12x22_P0.80x0.65mm" H 2875 1150 50  0001 C CNN
+F 3 "" H 2725 1850 50  0001 C CNN
+F 4 "Micron" H 2825 1370 50  0001 C CNN "Manufacturer"
+F 5 "MT53D1024M32D4DT-053 WT:D" H 2100 1675 50  0000 C CNN "MPN"
+	1    2825 3050
+	1    0    0    -1
+$EndComp
+$Comp
+L antmicroMemory:MT53D1024M32D4DT-053 U?
+U 2 1 62E1B568
+P 2850 7025
+F 0 "U?" H 2650 5550 50  0000 C CNN
+F 1 "MT53D1024M32D4DT-053" H 3550 8475 50  0001 C CNN
+F 2 "antmicro-footprints:BGA-200_10.0x14.5mm_Layout12x22_P0.80x0.65mm" H 2900 5125 50  0001 C CNN
+F 3 "" H 2750 5825 50  0001 C CNN
+F 4 "Micron" H 2850 5345 50  0001 C CNN "Manufacturer"
+F 5 "MT53D1024M32D4DT-053 WT:D" H 2150 5650 50  0000 C CNN "MPN"
+	2    2850 7025
+	1    0    0    -1
+$EndComp
+$Comp
+L antmicroMemory:MT53D1024M32D4DT-053 U?
+U 1 1 62E53070
+P 10950 3500
+F 0 "U?" H 10750 2025 50  0000 C CNN
+F 1 "MT53D1024M32D4DT-053" H 11650 4950 50  0001 C CNN
+F 2 "antmicro-footprints:BGA-200_10.0x14.5mm_Layout12x22_P0.80x0.65mm" H 11000 1600 50  0001 C CNN
+F 3 "" H 10850 2300 50  0001 C CNN
+F 4 "Micron" H 10950 1820 50  0001 C CNN "Manufacturer"
+F 5 "MT53D1024M32D4DT-053 WT:D" H 10225 2125 50  0000 C CNN "MPN"
+	1    10950 3500
+	1    0    0    -1
+$EndComp
+$Comp
+L antmicroMemory:MT53D1024M32D4DT-053 U?
+U 2 1 62E7500A
+P 10975 7375
+F 0 "U?" H 10775 5925 50  0000 C CNN
+F 1 "MT53D1024M32D4DT-053" H 11675 8825 50  0001 C CNN
+F 2 "antmicro-footprints:BGA-200_10.0x14.5mm_Layout12x22_P0.80x0.65mm" H 11025 5475 50  0001 C CNN
+F 3 "" H 10875 6175 50  0001 C CNN
+F 4 "Micron" H 10975 5695 50  0001 C CNN "Manufacturer"
+F 5 "MT53D1024M32D4DT-053 WT:D" H 10275 6025 50  0000 C CNN "MPN"
+	2    10975 7375
+	1    0    0    -1
+$EndComp

Commit message: Added title block settings
Parts:
- gave numbers to parts that had none: 2
Changed lines of the file:
@@
 encoding utf-8
 Sheet 5 10
-Title ""
+Title "LPDDR4"
 Date ""
-Rev ""
-Comp ""
-Comment1 ""
+Rev "1.0.0"
+Comp "Antmicro ltd"
+Comment1 "http://antmicro.com"
 Comment2 ""
 Comment3 ""
@@
 $EndComp
 $Comp
-L antmicroMemory:MT53D1024M32D4DT-053 U?
+L antmicroMemory:MT53D1024M32D4DT-053 U1
 U 1 1 62E16A15
 P 2825 3050
-F 0 "U?" H 2625 1575 50  0000 C CNN
+F 0 "U1" H 2625 1575 50  0000 C CNN
 F 1 "MT53D1024M32D4DT-053" H 3525 4500 50  0001 C CNN
 F 2 "antmicro-footprints:BGA-200_10.0x14.5mm_Layout12x22_P0.80x0.65mm" H 2875 1150 50  0001 C CNN
@@
 $EndComp
 $Comp
-L antmicroMemory:MT53D1024M32D4DT-053 U?
+L antmicroMemory:MT53D1024M32D4DT-053 U1
 U 2 1 62E1B568
 P 2850 7025
-F 0 "U?" H 2650 5550 50  0000 C CNN
+F 0 "U1" H 2650 5550 50  0000 C CNN
 F 1 "MT53D1024M32D4DT-053" H 3550 8475 50  0001 C CNN
 F 2 "antmicro-footprints:BGA-200_10.0x14.5mm_Layout12x22_P0.80x0.65mm" H 2900 5125 50  0001 C CNN
@@
 $EndComp
 $Comp
-L antmicroMemory:MT53D1024M32D4DT-053 U?
+L antmicroMemory:MT53D1024M32D4DT-053 U3
 U 1 1 62E53070
 P 10950 3500
-F 0 "U?" H 10750 2025 50  0000 C CNN
+F 0 "U3" H 10750 2025 50  0000 C CNN
 F 1 "MT53D1024M32D4DT-053" H 11650 4950 50  0001 C CNN
 F 2 "antmicro-footprints:BGA-200_10.0x14.5mm_Layout12x22_P0.80x0.65mm" H 11000 1600 50  0001 C CNN
@@
 $EndComp
 $Comp
-L antmicroMemory:MT53D1024M32D4DT-053 U?
+L antmicroMemory:MT53D1024M32D4DT-053 U3
 U 2 1 62E7500A
 P 10975 7375
-F 0 "U?" H 10775 5925 50  0000 C CNN
+F 0 "U3" H 10775 5925 50  0000 C CNN
 F 1 "MT53D1024M32D4DT-053" H 11675 8825 50  0001 C CNN
 F 2 "antmicro-footprints:BGA-200_10.0x14.5mm_Layout12x22_P0.80x0.65mm" H 11025 5475 50  0001 C CNN

Commit message: Added local libraries
Parts:
- C100, C101, C102, C103, C104, C105, C207, C208, C209, C210, C211, C212, C213, C214, C215, C216, C217, C218, C219, C220, C221, C222, C223, C224, C225, C226, C227, C228, C229, C230, C231, C232, C233, C234, C235, C236, C237, C238, C239, C240, C241, C71, C72, C73, C74, C75, C76, C77, C78, C79, C80, C81, C82, C83, C84, C85, C86, C87, C88, C89, C90, C91, C92, C93, C94, C95, C96, C97, C98, C99: footprint antmicro-footprints:0201-res -> arv-som-footprints:0201-res; symbol antmicroCapacitorsmisc:C_100n_0201 -> arv-som:C_100n_0201
- R100, R102, R46, R48: footprint antmicro-footprints:0402-res -> arv-som-footprints:0402-res; symbol antmicroResistors0402:R_0R_0402 -> arv-som:R_0R_0402
- R101, R103, R104, R105, R106, R107, R108, R43, R44, R47, R92, R93, R94, R95, R96, R98: footprint antmicro-footprints:0402-res -> arv-som-footprints:0402-res; symbol antmicroResistors0402:R_10k_0402 -> arv-som:R_10k_0402
- R42, R45, R97, R99: footprint antmicro-footprints:0402-res -> arv-som-footprints:0402-res; symbol antmicroResistors0402:R_240R_0402 -> arv-som:R_240R_0402
- U1, U3: footprint antmicro-footprints:BGA-200_10.0x14.5mm_Layout12x22_P0.80x0.65mm -> arv-som-footprints:BGA-200_10.0x14.5mm_Layout12x22_P0.80x0.65mm; symbol antmicroMemory:MT53D1024M32D4DT-053 -> arv-som:MT53D1024M32D4DT-053

Commit message: Update naming convention
Parts:
- C100, C101, C102, C103, C104, C105, C207, C208, C209, C210, C211, C212, C213, C214, C215, C216, C217, C218, C219, C220, C221, C222, C223, C224, C225, C226, C227, C228, C229, C230, C231, C232, C233, C234, C235, C236, C237, C238, C239, C240, C241, C71, C72, C73, C74, C75, C76, C77, C78, C79, C80, C81, C82, C83, C84, C85, C86, C87, C88, C89, C90, C91, C92, C93, C94, C95, C96, C97, C98, C99: footprint arv-som-footprints:0201-res -> arvsom-footprints:0201-res; symbol arv-som:C_100n_0201 -> arvsom:C_100n_0201
- R100, R102, R46, R48: footprint arv-som-footprints:0402-res -> arvsom-footprints:0402-res; symbol arv-som:R_0R_0402 -> arvsom:R_0R_0402
- R101, R103, R104, R105, R106, R107, R108, R43, R44, R47, R92, R93, R94, R95, R96, R98: footprint arv-som-footprints:0402-res -> arvsom-footprints:0402-res; symbol arv-som:R_10k_0402 -> arvsom:R_10k_0402
- R42, R45, R97, R99: footprint arv-som-footprints:0402-res -> arvsom-footprints:0402-res; symbol arv-som:R_240R_0402 -> arvsom:R_240R_0402
- U1, U3: footprint arv-som-footprints:BGA-200_10.0x14.5mm_Layout12x22_P0.80x0.65mm -> arvsom-footprints:BGA-200_10.0x14.5mm_Layout12x22_P0.80x0.65mm; symbol arv-som:MT53D1024M32D4DT-053 -> arvsom:MT53D1024M32D4DT-053
