File: VIC7100-DDR.sch (KiCad schematic (older format))
At the start: 14 parts

Commit message: Connected interfaces to VIC to visualise its ball locations (wip, mock purposes)
Parts:
- gave numbers to parts that had none: 13
Changed lines of the file:
@@
 $Descr A3 16535 11693
 encoding utf-8
-Sheet 11 12
+Sheet 10 11
 Title ""
 Date ""
@@
 $EndDescr
 $Comp
-L antmicroMicrocontrollers:VIC7100 U?
+L antmicroMicrocontrollers:VIC7100 U13
 U 5 1 613A4303
 P 4200 2250
-F 0 "U?" H 4475 2500 60  0000 L CNN
+F 0 "U13" H 4475 2500 60  0000 L CNN
 F 1 "VIC7100" H 4800 2425 60  0000 L CNN
 F 2 "antmicro-footprints:vic7100" H 4400 2300 60  0001 L CNN
@@
 $EndComp
 $Comp
-L antmicroMicrocontrollers:VIC7100 U?
+L antmicroMicrocontrollers:VIC7100 U13
 U 6 1 613ABB1B
 P 9575 2250
-F 0 "U?" H 9825 2575 60  0000 L CNN
+F 0 "U13" H 9825 2575 60  0000 L CNN
 F 1 "VIC7100" H 10200 2475 60  0000 L CNN
 F 2 "antmicro-footprints:vic7100" H 9775 2300 60  0001 L CNN
@@
 NoConn ~ 4200 5550
 $Comp
-L antmicroResistors0402:R_240R_0402 R?
+L antmicroResistors0402:R_240R_0402 R89
 U 1 1 615EA23C
 P 3900 5850
-F 0 "R?" H 3900 6063 60  0000 C CNN
+F 0 "R89" H 3900 6063 60  0000 C CNN
 F 1 "R_240R_0402" H 3900 5700 60  0001 C CNN
 F 2 "antmicro-footprints:0402-res" H 4100 6050 60  0001 L CNN
@@
 	4200 5850 4050 5850
 $Comp
-L antmicroResistors0402:R_10k_0402 R?
+L antmicroResistors0402:R_10k_0402 R88
 U 1 1 615F0DBD
 P 3700 5950
-F 0 "R?" H 3700 6163 60  0000 C CNN
+F 0 "R88" H 3700 6163 60  0000 C CNN
 F 1 "R_10k_0402" H 3700 5800 60  0001 C CNN
 F 2 "antmicro-footprints:0402-res" H 3900 6150 60  0001 L CNN
@@
 	3550 5950 3425 5950
 $Comp
-L power:GND #PWR?
+L power:GND #PWR0222
 U 1 1 615F7BC0
 P 3425 5850
-F 0 "#PWR?" H 3425 5600 50  0001 C CNN
+F 0 "#PWR0222" H 3425 5600 50  0001 C CNN
 F 1 "GND" V 3430 5722 50  0000 R CNN
 F 2 "" H 3425 5850 50  0001 C CNN
@@
 	4200 7750 3525 7750
 $Comp
-L antmicroTestPoints:TP_SMD1MM TP?
+L antmicroTestPoints:TP_SMD1MM TP5
 U 1 1 61630E41
 P 3225 7150
-F 0 "TP?" H 3175 7197 50  0000 R CNN
+F 0 "TP5" H 3175 7197 50  0000 R CNN
 F 1 "TP_SMD1MM" H 3225 7050 50  0001 C CNN
 F 2 "antmicro-footprints:Testpoint_smd_1mm" H 3425 7350 60  0001 L CNN
@@
 $EndComp
 $Comp
-L antmicroTestPoints:TP_SMD1MM TP?
+L antmicroTestPoints:TP_SMD1MM TP6
 U 1 1 61631802
 P 3325 7150
-F 0 "TP?" H 3275 7197 50  0000 R CNN
+F 0 "TP6" H 3275 7197 50  0000 R CNN
 F 1 "TP_SMD1MM" H 3325 7050 50  0001 C CNN
 F 2 "antmicro-footprints:Testpoint_smd_1mm" H 3525 7350 60  0001 L CNN
@@
 $EndComp
 $Comp
-L antmicroTestPoints:TP_SMD1MM TP?
+L antmicroTestPoints:TP_SMD1MM TP7
 U 1 1 6163202C
 P 3425 7150
-F 0 "TP?" H 3375 7197 50  0000 R CNN
+F 0 "TP7" H 3375 7197 50  0000 R CNN
 F 1 "TP_SMD1MM" H 3425 7050 50  0001 C CNN
 F 2 "antmicro-footprints:Testpoint_smd_1mm" H 3625 7350 60  0001 L CNN
@@
 $EndComp
 $Comp
-L antmicroTestPoints:TP_SMD1MM TP?
+L antmicroTestPoints:TP_SMD1MM TP8
 U 1 1 61632781
 P 3525 7150
-F 0 "TP?" H 3475 7197 50  0000 R CNN
+F 0 "TP8" H 3475 7197 50  0000 R CNN
 F 1 "TP_SMD1MM" H 3525 7050 50  0001 C CNN
 F 2 "antmicro-footprints:Testpoint_smd_1mm" H 3725 7350 60  0001 L CNN
@@
 NoConn ~ 9575 5550
 $Comp
-L antmicroResistors0402:R_240R_0402 R?
+L antmicroResistors0402:R_240R_0402 R91
 U 1 1 6170D5ED
 P 9275 5850
-F 0 "R?" H 9275 6063 60  0000 C CNN
+F 0 "R91" H 9275 6063 60  0000 C CNN
 F 1 "R_240R_0402" H 9275 5700 60  0001 C CNN
 F 2 "antmicro-footprints:0402-res" H 9475 6050 60  0001 L CNN
@@
 	9575 5850 9425 5850
 $Comp
-L antmicroResistors0402:R_10k_0402 R?
+L antmicroResistors0402:R_10k_0402 R90
 U 1 1 6170D5F7
 P 9075 5950
-F 0 "R?" H 9075 6163 60  0000 C CNN
+F 0 "R90" H 9075 6163 60  0000 C CNN
 F 1 "R_10k_0402" H 9075 5800 60  0001 C CNN
 F 2 "antmicro-footprints:0402-res" H 9275 6150 60  0001 L CNN
@@
 	8925 5950 8800 5950
 $Comp
-L power:GND #PWR?
+L power:GND #PWR0223
 U 1 1 6170D600
 P 8800 5850
-F 0 "#PWR?" H 8800 5600 50  0001 C CNN
+F 0 "#PWR0223" H 8800 5600 50  0001 C CNN
 F 1 "GND" V 8805 5722 50  0000 R CNN
 F 2 "" H 8800 5850 50  0001 C CNN
@@
 	9575 7750 8900 7750
 $Comp
-L antmicroTestPoints:TP_SMD1MM TP?
+L antmicroTestPoints:TP_SMD1MM TP9
 U 1 1 6170D617
 P 8600 7150
-F 0 "TP?" H 8550 7197 50  0000 R CNN
+F 0 "TP9" H 8550 7197 50  0000 R CNN
 F 1 "TP_SMD1MM" H 8600 7050 50  0001 C CNN
 F 2 "antmicro-footprints:Testpoint_smd_1mm" H 8800 7350 60  0001 L CNN
@@
 $EndComp
 $Comp
-L antmicroTestPoints:TP_SMD1MM TP?
+L antmicroTestPoints:TP_SMD1MM TP10
 U 1 1 6170D61D
 P 8700 7150
-F 0 "TP?" H 8650 7197 50  0000 R CNN
+F 0 "TP10" H 8650 7197 50  0000 R CNN
 F 1 "TP_SMD1MM" H 8700 7050 50  0001 C CNN
 F 2 "antmicro-footprints:Testpoint_smd_1mm" H 8900 7350 60  0001 L CNN
@@
 $EndComp
 $Comp
-L antmicroTestPoints:TP_SMD1MM TP?
+L antmicroTestPoints:TP_SMD1MM TP11
 U 1 1 6170D623
 P 8800 7150
-F 0 "TP?" H 8750 7197 50  0000 R CNN
+F 0 "TP11" H 8750 7197 50  0000 R CNN
 F 1 "TP_SMD1MM" H 8800 7050 50  0001 C CNN
 F 2 "antmicro-footprints:Testpoint_smd_1mm" H 9000 7350 60  0001 L CNN
@@
 $EndComp
 $Comp
-L antmicroTestPoints:TP_SMD1MM TP?
+L antmicroTestPoints:TP_SMD1MM TP12
 U 1 1 6170D629
 P 8900 7150
-F 0 "TP?" H 8850 7197 50  0000 R CNN
+F 0 "TP12" H 8850 7197 50  0000 R CNN
 F 1 "TP_SMD1MM" H 8900 7050 50  0001 C CNN
 F 2 "antmicro-footprints:Testpoint_smd_1mm" H 9100 7350 60  0001 L CNN

Commit message: Schematic cleanup, added logotypes
Other:
- note added: "VIC7100 DDR"

Commit message: Added local libraries
Parts:
- R88, R90: footprint antmicro-footprints:0402-res -> arv-som-footprints:0402-res; symbol antmicroResistors0402:R_10k_0402 -> arv-som:R_10k_0402
- R89, R91: footprint antmicro-footprints:0402-res -> arv-som-footprints:0402-res; symbol antmicroResistors0402:R_240R_0402 -> arv-som:R_240R_0402
- TP10, TP11, TP12, TP5, TP6, TP7, TP8, TP9: footprint antmicro-footprints:Testpoint_smd_1mm -> arv-som-footprints:Testpoint_smd_1mm; symbol antmicroTestPoints:TP_SMD1MM -> arv-som:TP_SMD1MM
- U13: footprint antmicro-footprints:vic7100 -> arv-som-footprints:vic7100; symbol antmicroMicrocontrollers:VIC7100 -> arv-som:VIC7100
Changed lines of the file:
@@
 $EndDescr
 $Comp
-L antmicroMicrocontrollers:VIC7100 U13
+L arv-som:VIC7100 U13
 U 5 1 613A4303
 P 4200 2250
 F 0 "U13" H 4400 2425 60  0000 L CNN
 F 1 "VIC7100" H 4800 2425 60  0000 L CNN
-F 2 "antmicro-footprints:vic7100" H 4400 2300 60  0001 L CNN
+F 2 "arv-som-footprints:vic7100" H 4400 2300 60  0001 L CNN
 F 3 "" H 4400 2100 60  0001 L CNN
 F 4 "VIC7100" H 5275 2450 50  0001 L CNN "MPN"
@@
 $EndComp
 $Comp
-L antmicroMicrocontrollers:VIC7100 U13
+L arv-som:VIC7100 U13
 U 6 1 613ABB1B
 P 9575 2250
 F 0 "U13" H 9775 2425 60  0000 L CNN
 F 1 "VIC7100" H 10200 2425 60  0000 L CNN
-F 2 "antmicro-footprints:vic7100" H 9775 2300 60  0001 L CNN
+F 2 "arv-som-footprints:vic7100" H 9775 2300 60  0001 L CNN
 F 3 "" H 9775 2100 60  0001 L CNN
 F 4 "VIC7100" H 10575 2500 50  0001 L CNN "MPN"
@@
 NoConn ~ 4200 5550
 $Comp
-L antmicroResistors0402:R_240R_0402 R89
+L arv-som:R_240R_0402 R89
 U 1 1 615EA23C
 P 3900 5850
 F 0 "R89" H 3700 5900 60  0000 C CNN
 F 1 "R_240R_0402" H 3900 5700 60  0001 C CNN
-F 2 "antmicro-footprints:0402-res" H 4100 6050 60  0001 L CNN
+F 2 "arv-som-footprints:0402-res" H 4100 6050 60  0001 L CNN
 F 3 "" H 3900 5850 50  0001 C CNN
 F 4 "PANASONIC" H 4100 6250 60  0001 L CNN "Manufacturer"
@@
 	4200 5850 4050 5850
 $Comp
-L antmicroResistors0402:R_10k_0402 R88
+L arv-som:R_10k_0402 R88
 U 1 1 615F0DBD
 P 3700 5950
 F 0 "R88" H 3500 6000 60  0000 C CNN
 F 1 "R_10k_0402" H 3700 5800 60  0001 C CNN
-F 2 "antmicro-footprints:0402-res" H 3900 6150 60  0001 L CNN
+F 2 "arv-som-footprints:0402-res" H 3900 6150 60  0001 L CNN
 F 3 "" H 3700 5950 50  0001 C CNN
 F 4 "VISHAY" H 3900 6350 60  0001 L CNN "Manufacturer"
@@
 	3550 5950 3425 5950
 $Comp
-L power:GND #PWR0222
+L arv-som:GND #PWR0222
 U 1 1 615F7BC0
 P 3425 5850
@@
 	4200 7750 3525 7750
 $Comp
-L antmicroTestPoints:TP_SMD1MM TP5
+L arv-som:TP_SMD1MM TP5
 U 1 1 61630E41
 P 3225 7150
 F 0 "TP5" V 3225 7075 50  0000 R CNN
 F 1 "TP_SMD1MM" H 3225 7050 50  0001 C CNN
-F 2 "antmicro-footprints:Testpoint_smd_1mm" H 3425 7350 60  0001 L CNN
+F 2 "arv-som-footprints:Testpoint_smd_1mm" H 3425 7350 60  0001 L CNN
 F 3 "" H 3425 7450 60  0001 L CNN
 	1    3225 7150
@@
 $EndComp
 $Comp
-L antmicroTestPoints:TP_SMD1MM TP6
+L arv-som:TP_SMD1MM TP6
 U 1 1 61631802
 P 3325 7150
 F 0 "TP6" V 3325 7075 50  0000 R CNN
 F 1 "TP_SMD1MM" H 3325 7050 50  0001 C CNN
-F 2 "antmicro-footprints:Testpoint_smd_1mm" H 3525 7350 60  0001 L CNN
+F 2 "arv-som-footprints:Testpoint_smd_1mm" H 3525 7350 60  0001 L CNN
 F 3 "" H 3525 7450 60  0001 L CNN
 	1    3325 7150
@@
 $EndComp
 $Comp
-L antmicroTestPoints:TP_SMD1MM TP7
+L arv-som:TP_SMD1MM TP7
 U 1 1 6163202C
 P 3425 7150
 F 0 "TP7" V 3425 7075 50  0000 R CNN
 F 1 "TP_SMD1MM" H 3425 7050 50  0001 C CNN
-F 2 "antmicro-footprints:Testpoint_smd_1mm" H 3625 7350 60  0001 L CNN
+F 2 "arv-som-footprints:Testpoint_smd_1mm" H 3625 7350 60  0001 L CNN
 F 3 "" H 3625 7450 60  0001 L CNN
 	1    3425 7150
@@
 $EndComp
 $Comp
-L antmicroTestPoints:TP_SMD1MM TP8
+L arv-som:TP_SMD1MM TP8
 U 1 1 61632781
 P 3525 7150
 F 0 "TP8" V 3525 7075 50  0000 R CNN
 F 1 "TP_SMD1MM" H 3525 7050 50  0001 C CNN
-F 2 "antmicro-footprints:Testpoint_smd_1mm" H 3725 7350 60  0001 L CNN
+F 2 "arv-som-footprints:Testpoint_smd_1mm" H 3725 7350 60  0001 L CNN
 F 3 "" H 3725 7450 60  0001 L CNN
 	1    3525 7150
@@
 NoConn ~ 9575 5550
 $Comp
-L antmicroResistors0402:R_240R_0402 R91
+L arv-som:R_240R_0402 R91
 U 1 1 6170D5ED
 P 9275 5850
 F 0 "R91" H 9075 5900 60  0000 C CNN
 F 1 "R_240R_0402" H 9275 5700 60  0001 C CNN
-F 2 "antmicro-footprints:0402-res" H 9475 6050 60  0001 L CNN
+F 2 "arv-som-footprints:0402-res" H 9475 6050 60  0001 L CNN
 F 3 "" H 9275 5850 50  0001 C CNN
 F 4 "PANASONIC" H 9475 6250 60  0001 L CNN "Manufacturer"
@@
 	9575 5850 9425 5850
 $Comp
-L antmicroResistors0402:R_10k_0402 R90
+L arv-som:R_10k_0402 R90
 U 1 1 6170D5F7
 P 9075 5950
 F 0 "R90" H 8875 6000 60  0000 C CNN
 F 1 "R_10k_0402" H 9075 5800 60  0001 C CNN
-F 2 "antmicro-footprints:0402-res" H 9275 6150 60  0001 L CNN
+F 2 "arv-som-footprints:0402-res" H 9275 6150 60  0001 L CNN
 F 3 "" H 9075 5950 50  0001 C CNN
 F 4 "VISHAY" H 9275 6350 60  0001 L CNN "Manufacturer"
@@
 	8925 5950 8800 5950
 $Comp
-L power:GND #PWR0223
+L arv-som:GND #PWR0223
 U 1 1 6170D600
 P 8800 5850
@@
 	9575 7750 8900 7750
 $Comp
-L antmicroTestPoints:TP_SMD1MM TP9
+L arv-som:TP_SMD1MM TP9
 U 1 1 6170D617
 P 8600 7150
 F 0 "TP9" V 8600 7075 50  0000 R CNN
 F 1 "TP_SMD1MM" H 8600 7050 50  0001 C CNN
-F 2 "antmicro-footprints:Testpoint_smd_1mm" H 8800 7350 60  0001 L CNN
+F 2 "arv-som-footprints:Testpoint_smd_1mm" H 8800 7350 60  0001 L CNN
 F 3 "" H 8800 7450 60  0001 L CNN
 	1    8600 7150
@@
 $EndComp
 $Comp
-L antmicroTestPoints:TP_SMD1MM TP10
+L arv-som:TP_SMD1MM TP10
 U 1 1 6170D61D
 P 8700 7150
 F 0 "TP10" V 8700 7075 50  0000 R CNN
 F 1 "TP_SMD1MM" H 8700 7050 50  0001 C CNN
-F 2 "antmicro-footprints:Testpoint_smd_1mm" H 8900 7350 60  0001 L CNN
+F 2 "arv-som-footprints:Testpoint_smd_1mm" H 8900 7350 60  0001 L CNN
 F 3 "" H 8900 7450 60  0001 L CNN
 	1    8700 7150
@@
 $EndComp
 $Comp
-L antmicroTestPoints:TP_SMD1MM TP11
+L arv-som:TP_SMD1MM TP11
 U 1 1 6170D623
 P 8800 7150
 F 0 "TP11" V 8800 7075 50  0000 R CNN
 F 1 "TP_SMD1MM" H 8800 7050 50  0001 C CNN
-F 2 "antmicro-footprints:Testpoint_smd_1mm" H 9000 7350 60  0001 L CNN
+F 2 "arv-som-footprints:Testpoint_smd_1mm" H 9000 7350 60  0001 L CNN
 F 3 "" H 9000 7450 60  0001 L CNN
 	1    8800 7150
@@
 $EndComp
 $Comp
-L antmicroTestPoints:TP_SMD1MM TP12
+L arv-som:TP_SMD1MM TP12
 U 1 1 6170D629
 P 8900 7150
 F 0 "TP12" V 8900 7075 50  0000 R CNN
 F 1 "TP_SMD1MM" H 8900 7050 50  0001 C CNN
-F 2 "antmicro-footprints:Testpoint_smd_1mm" H 9100 7350 60  0001 L CNN
+F 2 "arv-som-footprints:Testpoint_smd_1mm" H 9100 7350 60  0001 L CNN
 F 3 "" H 9100 7450 60  0001 L CNN
 	1    8900 7150

Commit message: Update naming convention
Parts:
- R88, R90: footprint arv-som-footprints:0402-res -> arvsom-footprints:0402-res; symbol arv-som:R_10k_0402 -> arvsom:R_10k_0402
- R89, R91: footprint arv-som-footprints:0402-res -> arvsom-footprints:0402-res; symbol arv-som:R_240R_0402 -> arvsom:R_240R_0402
- TP10, TP11, TP12, TP5, TP6, TP7, TP8, TP9: footprint arv-som-footprints:Testpoint_smd_1mm -> arvsom-footprints:Testpoint_smd_1mm; symbol arv-som:TP_SMD1MM -> arvsom:TP_SMD1MM
- U13: footprint arv-som-footprints:vic7100 -> arvsom-footprints:vic7100; symbol arv-som:VIC7100 -> arvsom:VIC7100
Changed lines of the file:
@@
 $EndDescr
 $Comp
-L arv-som:VIC7100 U13
+L arvsom:VIC7100 U13
 U 5 1 613A4303
 P 4200 2250
 F 0 "U13" H 4400 2425 60  0000 L CNN
 F 1 "VIC7100" H 4800 2425 60  0000 L CNN
-F 2 "arv-som-footprints:vic7100" H 4400 2300 60  0001 L CNN
+F 2 "arvsom-footprints:vic7100" H 4400 2300 60  0001 L CNN
 F 3 "" H 4400 2100 60  0001 L CNN
 F 4 "VIC7100" H 5275 2450 50  0001 L CNN "MPN"
@@
 $EndComp
 $Comp
-L arv-som:VIC7100 U13
+L arvsom:VIC7100 U13
 U 6 1 613ABB1B
 P 9575 2250
 F 0 "U13" H 9775 2425 60  0000 L CNN
 F 1 "VIC7100" H 10200 2425 60  0000 L CNN
-F 2 "arv-som-footprints:vic7100" H 9775 2300 60  0001 L CNN
+F 2 "arvsom-footprints:vic7100" H 9775 2300 60  0001 L CNN
 F 3 "" H 9775 2100 60  0001 L CNN
 F 4 "VIC7100" H 10575 2500 50  0001 L CNN "MPN"
@@
 NoConn ~ 4200 5550
 $Comp
-L arv-som:R_240R_0402 R89
+L arvsom:R_240R_0402 R89
 U 1 1 615EA23C
 P 3900 5850
 F 0 "R89" H 3700 5900 60  0000 C CNN
 F 1 "R_240R_0402" H 3900 5700 60  0001 C CNN
-F 2 "arv-som-footprints:0402-res" H 4100 6050 60  0001 L CNN
+F 2 "arvsom-footprints:0402-res" H 4100 6050 60  0001 L CNN
 F 3 "" H 3900 5850 50  0001 C CNN
 F 4 "PANASONIC" H 4100 6250 60  0001 L CNN "Manufacturer"
@@
 	4200 5850 4050 5850
 $Comp
-L arv-som:R_10k_0402 R88
+L arvsom:R_10k_0402 R88
 U 1 1 615F0DBD
 P 3700 5950
 F 0 "R88" H 3500 6000 60  0000 C CNN
 F 1 "R_10k_0402" H 3700 5800 60  0001 C CNN
-F 2 "arv-som-footprints:0402-res" H 3900 6150 60  0001 L CNN
+F 2 "arvsom-footprints:0402-res" H 3900 6150 60  0001 L CNN
 F 3 "" H 3700 5950 50  0001 C CNN
 F 4 "VISHAY" H 3900 6350 60  0001 L CNN "Manufacturer"
@@
 	3550 5950 3425 5950
 $Comp
-L arv-som:GND #PWR0222
+L arvsom:GND #PWR0222
 U 1 1 615F7BC0
 P 3425 5850
@@
 	4200 7750 3525 7750
 $Comp
-L arv-som:TP_SMD1MM TP5
+L arvsom:TP_SMD1MM TP5
 U 1 1 61630E41
 P 3225 7150
 F 0 "TP5" V 3225 7075 50  0000 R CNN
 F 1 "TP_SMD1MM" H 3225 7050 50  0001 C CNN
-F 2 "arv-som-footprints:Testpoint_smd_1mm" H 3425 7350 60  0001 L CNN
+F 2 "arvsom-footprints:Testpoint_smd_1mm" H 3425 7350 60  0001 L CNN
 F 3 "" H 3425 7450 60  0001 L CNN
 	1    3225 7150
@@
 $EndComp
 $Comp
-L arv-som:TP_SMD1MM TP6
+L arvsom:TP_SMD1MM TP6
 U 1 1 61631802
 P 3325 7150
 F 0 "TP6" V 3325 7075 50  0000 R CNN
 F 1 "TP_SMD1MM" H 3325 7050 50  0001 C CNN
-F 2 "arv-som-footprints:Testpoint_smd_1mm" H 3525 7350 60  0001 L CNN
+F 2 "arvsom-footprints:Testpoint_smd_1mm" H 3525 7350 60  0001 L CNN
 F 3 "" H 3525 7450 60  0001 L CNN
 	1    3325 7150
@@
 $EndComp
 $Comp
-L arv-som:TP_SMD1MM TP7
+L arvsom:TP_SMD1MM TP7
 U 1 1 6163202C
 P 3425 7150
 F 0 "TP7" V 3425 7075 50  0000 R CNN
 F 1 "TP_SMD1MM" H 3425 7050 50  0001 C CNN
-F 2 "arv-som-footprints:Testpoint_smd_1mm" H 3625 7350 60  0001 L CNN
+F 2 "arvsom-footprints:Testpoint_smd_1mm" H 3625 7350 60  0001 L CNN
 F 3 "" H 3625 7450 60  0001 L CNN
 	1    3425 7150
@@
 $EndComp
 $Comp
-L arv-som:TP_SMD1MM TP8
+L arvsom:TP_SMD1MM TP8
 U 1 1 61632781
 P 3525 7150
 F 0 "TP8" V 3525 7075 50  0000 R CNN
 F 1 "TP_SMD1MM" H 3525 7050 50  0001 C CNN
-F 2 "arv-som-footprints:Testpoint_smd_1mm" H 3725 7350 60  0001 L CNN
+F 2 "arvsom-footprints:Testpoint_smd_1mm" H 3725 7350 60  0001 L CNN
 F 3 "" H 3725 7450 60  0001 L CNN
 	1    3525 7150
@@
 NoConn ~ 9575 5550
 $Comp
-L arv-som:R_240R_0402 R91
+L arvsom:R_240R_0402 R91
 U 1 1 6170D5ED
 P 9275 5850
 F 0 "R91" H 9075 5900 60  0000 C CNN
 F 1 "R_240R_0402" H 9275 5700 60  0001 C CNN
-F 2 "arv-som-footprints:0402-res" H 9475 6050 60  0001 L CNN
+F 2 "arvsom-footprints:0402-res" H 9475 6050 60  0001 L CNN
 F 3 "" H 9275 5850 50  0001 C CNN
 F 4 "PANASONIC" H 9475 6250 60  0001 L CNN "Manufacturer"
@@
 	9575 5850 9425 5850
 $Comp
-L arv-som:R_10k_0402 R90
+L arvsom:R_10k_0402 R90
 U 1 1 6170D5F7
 P 9075 5950
 F 0 "R90" H 8875 6000 60  0000 C CNN
 F 1 "R_10k_0402" H 9075 5800 60  0001 C CNN
-F 2 "arv-som-footprints:0402-res" H 9275 6150 60  0001 L CNN
+F 2 "arvsom-footprints:0402-res" H 9275 6150 60  0001 L CNN
 F 3 "" H 9075 5950 50  0001 C CNN
 F 4 "VISHAY" H 9275 6350 60  0001 L CNN "Manufacturer"
@@
 	8925 5950 8800 5950
 $Comp
-L arv-som:GND #PWR0223
+L arvsom:GND #PWR0223
 U 1 1 6170D600
 P 8800 5850
@@
 	9575 7750 8900 7750
 $Comp
-L arv-som:TP_SMD1MM TP9
+L arvsom:TP_SMD1MM TP9
 U 1 1 6170D617
 P 8600 7150
 F 0 "TP9" V 8600 7075 50  0000 R CNN
 F 1 "TP_SMD1MM" H 8600 7050 50  0001 C CNN
-F 2 "arv-som-footprints:Testpoint_smd_1mm" H 8800 7350 60  0001 L CNN
+F 2 "arvsom-footprints:Testpoint_smd_1mm" H 8800 7350 60  0001 L CNN
 F 3 "" H 8800 7450 60  0001 L CNN
 	1    8600 7150
@@
 $EndComp
 $Comp
-L arv-som:TP_SMD1MM TP10
+L arvsom:TP_SMD1MM TP10
 U 1 1 6170D61D
 P 8700 7150
 F 0 "TP10" V 8700 7075 50  0000 R CNN
 F 1 "TP_SMD1MM" H 8700 7050 50  0001 C CNN
-F 2 "arv-som-footprints:Testpoint_smd_1mm" H 8900 7350 60  0001 L CNN
+F 2 "arvsom-footprints:Testpoint_smd_1mm" H 8900 7350 60  0001 L CNN
 F 3 "" H 8900 7450 60  0001 L CNN
 	1    8700 7150
@@
 $EndComp
 $Comp
-L arv-som:TP_SMD1MM TP11
+L arvsom:TP_SMD1MM TP11
 U 1 1 6170D623
 P 8800 7150
 F 0 "TP11" V 8800 7075 50  0000 R CNN
 F 1 "TP_SMD1MM" H 8800 7050 50  0001 C CNN
-F 2 "arv-som-footprints:Testpoint_smd_1mm" H 9000 7350 60  0001 L CNN
+F 2 "arvsom-footprints:Testpoint_smd_1mm" H 9000 7350 60  0001 L CNN
 F 3 "" H 9000 7450 60  0001 L CNN
 	1    8800 7150
@@
 $EndComp
 $Comp
-L arv-som:TP_SMD1MM TP12
+L arvsom:TP_SMD1MM TP12
 U 1 1 6170D629
 P 8900 7150
 F 0 "TP12" V 8900 7075 50  0000 R CNN
 F 1 "TP_SMD1MM" H 8900 7050 50  0001 C CNN
-F 2 "arv-som-footprints:Testpoint_smd_1mm" H 9100 7350 60  0001 L CNN
+F 2 "arvsom-footprints:Testpoint_smd_1mm" H 9100 7350 60  0001 L CNN
 F 3 "" H 9100 7450 60  0001 L CNN
 	1    8900 7150
