File: VIC7100-power.sch (KiCad schematic (older format))
At the start: 70 parts

Commit message: Connected interfaces to VIC to visualise its ball locations (wip, mock purposes)
Parts:
- gave numbers to parts that had none: 67

Commit message: Schematic cleanup, added logotypes
Other:
- note added: "VIC7100 power"

Commit message: Added local libraries
Parts:
- C106, C107, C112, C113, C117, C119, C123, C127, C128, C129, C130, C131, C132, C133, C134, C136, C137, C138, C140, C141, C142, C144, C145, C146, C147, C148, C149, C150, C151, C152, C153, C154, C155, C156, C157, C158, C159, C162, C164, C165, C166, C167, C168, C169: footprint antmicro-footprints:0201-res -> arv-som-footprints:0201-res; symbol antmicroCapacitorsmisc:C_100n_0201 -> arv-som:C_100n_0201
- C108, C124, C125, C126, C143: footprint antmicro-footprints:0402-cap -> arv-som-footprints:0402-cap; symbol antmicroCapacitors0402:C_1u_0402 -> arv-som:C_1u_0402
- C109, C110, C111, C116, C135: footprint antmicro-footprints:0603-cap -> arv-som-footprints:0603-cap; symbol antmicroCapacitors0603:C_22u_0603 -> arv-som:C_22u_0603
- C114, C115, C118, C120, C121, C122, C139: footprint antmicro-footprints:0402-cap -> arv-som-footprints:0402-cap; symbol antmicroCapacitors0402:C_10u_0402 -> arv-som:C_10u_0402
- C160, C161, C163, C170: footprint antmicro-footprints:0402-res -> arv-som-footprints:0402-res; symbol antmicroCapacitors0402:C_1n_0402 -> arv-som:C_1n_0402
- FB5: footprint antmicro-footprints:0402-res -> arv-som-footprints:0402-res; symbol antmicroFerriteBeadsandChips:BLM15PD121SN1D -> arv-som:BLM15PD121SN1D
- U13: footprint antmicro-footprints:vic7100 -> arv-som-footprints:vic7100; symbol antmicroMicrocontrollers:VIC7100 -> arv-som:VIC7100

Commit message: Update naming convention
Parts:
- C106, C107, C112, C113, C117, C119, C123, C127, C128, C129, C130, C131, C132, C133, C134, C136, C137, C138, C140, C141, C142, C144, C145, C146, C147, C148, C149, C150, C151, C152, C153, C154, C155, C156, C157, C158, C159, C162, C164, C165, C166, C167, C168, C169: footprint arv-som-footprints:0201-res -> arvsom-footprints:0201-res; symbol arv-som:C_100n_0201 -> arvsom:C_100n_0201
- C108, C124, C125, C126, C143: footprint arv-som-footprints:0402-cap -> arvsom-footprints:0402-cap; symbol arv-som:C_1u_0402 -> arvsom:C_1u_0402
- C109, C110, C111, C116, C135: footprint arv-som-footprints:0603-cap -> arvsom-footprints:0603-cap; symbol arv-som:C_22u_0603 -> arvsom:C_22u_0603
- C114, C115, C118, C120, C121, C122, C139: footprint arv-som-footprints:0402-cap -> arvsom-footprints:0402-cap; symbol arv-som:C_10u_0402 -> arvsom:C_10u_0402
- C160, C161, C163, C170: footprint arv-som-footprints:0402-res -> arvsom-footprints:0402-res; symbol arv-som:C_1n_0402 -> arvsom:C_1n_0402
- FB5: footprint arv-som-footprints:0402-res -> arvsom-footprints:0402-res; symbol arv-som:BLM15PD121SN1D -> arvsom:BLM15PD121SN1D
- U13: footprint arv-som-footprints:vic7100 -> arvsom-footprints:vic7100; symbol arv-som:VIC7100 -> arvsom:VIC7100
